File: sensors.kicad_sch (KiCad schematic)
At the start: 0 parts

Commit message: Copy over sensor designs
Parts:
- added C22, C23, C24, C25, C26, C28: 0.1u, Capacitor_SMD:C_0603_1608Metric, symbol Device:C
- added C27: 10u, Capacitor_SMD:C_0805_2012Metric, symbol Device:C
- added C29: 220n, Capacitor_SMD:C_0603_1608Metric, symbol Device:C
- added R11, R12: 1K, Resistor_SMD:R_0603_1608Metric, symbol Device:R
- added U5: BMI088, LRI_partlib:PQFN50P450X300X100-16N, symbol LRI_partlib:BMI088
- added U6: TMP117xxDRV, Package_SON:WSON-6-1EP_2x2mm_P0.65mm_EP1x1.6mm, symbol Sensor_Temperature:TMP117xxDRV
- added U7: LIS2MDL, Package_LGA:LGA-12_2x2mm_P0.5mm, symbol Sensor_Magnetic:LIS2MDL
- added U9: MS5611-01BA, Package_LGA:LGA-8_3x5mm_P1.25mm, symbol Sensor_Pressure:MS5611-01BA
Connections:
- new net: U7.6 (GND), U7.8 (GND)
- new net +3V3: C22.1, C22.2, C23.1, C23.2, C24.1, C24.2, C28.1, C28.2, R11.1, R12.1, U5.10 (SDO2), U5.11 (VDDIO), U5.15 (SDO1), U5.3 (VDD), U5.4 (GNDA), U5.6 (GNDIO), U5.7 (PS), U6.2 (GND), U6.4 (ADD0), U6.5 (V+), U9.1 (VDD), U9.2 (PS), U9.3 (GND), U9.4 (CSB), U9.5 (CSB)
- new net SENSOR_SCL: R11.2, U5.8 (SCL/SCK), U6.1 (SCL), U9.8 (SCLK)
- new net SENSOR_SDA: R12.2, U5.9 (SDA/SDI), U6.6 (SDA), U9.7 (SDI/SDA)
- no-connect marks 0 -> 9
Other:
- note added: "Barometer I2C Addr: 0x77"
- note added: "Bus pull-up resistors"
- note added: "I2C Addr: 0x90"
- note added: "IMU Accel. I2C Addr: 0x18 Gyro. I2C Addr: 0x68"
- note added: "Magnetometer I2C Addr: 0x1E"
- note added: "Temperature"

Commit message: the beginnings of a footprint
Parts:
- removed U6: TMP117xxDRV, Package_SON:WSON-6-1EP_2x2mm_P0.65mm_EP1x1.6mm, symbol Sensor_Temperature:TMP117xxDRV
- added U8: SHT4x, Sensor_Humidity:Sensirion_DFN-4_1.5x1.5mm_P0.8mm_SHT4x_NoCentralPad, symbol Sensor_Humidity:SHT4x
Connections:
- net SENSOR_SCL is gone; now on net I2C0_SCL: R11.2, U5.8 (SCL/SCK), U9.8 (SCLK)
- net SENSOR_SDA is gone; now on net I2C0_SDA: R12.2, U5.9 (SDA/SDI), U9.7 (SDI/SDA)
- net +3V3: now also U8.3 (VDD); no longer C22.1, C23.1, C24.1, C28.2, U5.10 (SDO2), U5.15 (SDO1), U5.4 (GNDA), U5.6 (GNDIO), U9.3 (GND), U9.4 (CSB), U9.5 (CSB)
- net I2C0_SCL: now reaches U7.1 (SCL/SPC)
- net I2C0_SCL: now also U8.2 (SCL)
- net I2C0_SDA: now reaches U7.4 (SDA/SDI/SDO)
- net I2C0_SDA: now also U8.1 (SDA)
- net GND: now reaches U7.6 (GND), U7.8 (GND)
- net GND: now also C22.1, C23.1, C24.1, C28.2, U5.10 (SDO2), U5.15 (SDO1), U5.4 (GNDA), U5.6 (GNDIO), U9.3 (GND), U9.4 (CSB), U9.5 (CSB), U8.4 (VSS)
- no-connect marks 9 -> 8
Other:
- moved on the sheet: C24, C28, U9

Commit message: created project lib
Other:
- note added: "ICM-42688-P MISSING"
- moved on the sheet: R11, R12
Changed lines of the file:
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@@
 	)
 	(rectangle
-		(start 198.12 29.21)
-		(end 255.27 63.5)
+		(start 208.28 36.83)
+		(end 265.43 71.12)
 		(stroke
 			(width 0)
@@
 		)
 	)
+	(text "ICM-42688-P MISSING"
+		(exclude_from_sim no)
+		(at 108.966 165.354 0)
+		(effects
+			(font
+				(size 3.81 3.81)
+			)
+		)
+	)
 	(text "Bus pull-up resistors"
 		(exclude_from_sim no)
-		(at 227.076 27.178 0)
+		(at 237.236 34.798 0)
 		(effects
 			(font
@@
 	)
 	(junction
-		(at 240.03 40.64)
+		(at 250.19 48.26)
 		(diameter 0)
 		(color 0 0 0 0)
@@
 	(wire
 		(pts
-			(xy 236.22 40.64) (xy 236.22 43.18)
-		)
-		(stroke
-			(width 0)
-			(type default)
-		)
-	)
-	(wire
-		(pts
-			(xy 240.03 40.64) (xy 236.22 40.64)
+			(xy 245.11 48.26) (xy 245.11 50.8)
+		)
+		(stroke
+			(width 0)
+			(type default)
+		)
+	)
+	(wire
+		(pts
+			(xy 250.19 48.26) (xy 245.11 48.26)
 		)
 		(stroke
@@
 	(wire
 		(pts
-			(xy 243.84 43.18) (xy 243.84 40.64)
-		)
-		(stroke
-			(width 0)
-			(type default)
-		)
-	)
-	(wire
-		(pts
-			(xy 217.17 53.34) (xy 236.22 53.34)
+			(xy 255.27 50.8) (xy 255.27 48.26)
+		)
+		(stroke
+			(width 0)
+			(type default)
+		)
+	)
+	(wire
+		(pts
+			(xy 227.33 60.96) (xy 245.11 60.96)
 		)
 		(stroke
@@
 	(wire
 		(pts
-			(xy 240.03 39.37) (xy 240.03 40.64)
+			(xy 250.19 46.99) (xy 250.19 48.26)
 		)
 		(stroke
@@
 	(wire
 		(pts
-			(xy 236.22 50.8) (xy 236.22 53.34)
-		)
-		(stroke
-			(width 0)
-			(type default)
-		)
-	)
-	(wire
-		(pts
-			(xy 243.84 40.64) (xy 240.03 40.64)
+			(xy 245.11 58.42) (xy 245.11 60.96)
+		)
+		(stroke
+			(width 0)
+			(type default)
+		)
+	)
+	(wire
+		(pts
+			(xy 255.27 48.26) (xy 250.19 48.26)
 		)
 		(stroke
@@
 	(wire
 		(pts
-			(xy 217.17 55.88) (xy 243.84 55.88)
-		)
-		(stroke
-			(width 0)
-			(type default)
-		)
-	)
-	(wire
-		(pts
-			(xy 243.84 50.8) (xy 243.84 55.88)
+			(xy 227.33 64.77) (xy 255.27 64.77)
+		)
+		(stroke
+			(width 0)
+			(type default)
+		)
+	)
+	(wire
+		(pts
+			(xy 255.27 58.42) (xy 255.27 64.77)
 		)
 		(stroke
@@
 	(hierarchical_label "I2C0_SDA"
 		(shape bidirectional)
-		(at 217.17 55.88 180)
+		(at 227.33 64.77 180)
 		(effects
 			(font
@@
 	(hierarchical_label "I2C0_SCL"
 		(shape bidirectional)
-		(at 217.17 53.34 180)
+		(at 227.33 60.96 180)
 		(effects
 			(font
@@
 	(symbol
 		(lib_id "Device:R")
-		(at 236.22 46.99 0)
+		(at 245.11 54.61 0)
 		(unit 1)
 		(exclude_from_sim no)
@@
 		(dnp no)
 		(property "Reference" "R11"
-			(at 237.236 45.212 0)
+			(at 246.888 52.832 0)
 			(effects
 				(font
@@
 		)
 		(property "Value" "1K"
-			(at 237.236 46.99 0)
+			(at 246.888 55.372 0)
 			(effects
 				(font
@@
 		)
 		(property "Footprint" "Resistor_SMD:R_0603_1608Metric"
-			(at 234.442 46.99 90)
+			(at 243.332 54.61 90)
 			(effects
 				(font
@@
 		)
 		(property "Datasheet" "~"
-			(at 236.22 46.99 0)
+			(at 245.11 54.61 0)
 			(effects
 				(font
@@
 		)
 		(property "Description" "Resistor"
-			(at 236.22 46.99 0)
+			(at 245.11 54.61 0)
 			(effects
 				(font
@@
 	(symbol
 		(lib_id "power:+3V3")
-		(at 240.03 39.37 0)
+		(at 250.19 46.99 0)
 		(unit 1)
 		(exclude_from_sim no)
@@
 		(fields_autoplaced yes)
 		(property "Reference" "#PWR036"
-			(at 240.03 43.18 0)
+			(at 250.19 50.8 0)
 			(effects
 				(font
@@
 		)
 		(property "Value" "+3V3"
-			(at 240.03 34.29 0)
+			(at 250.19 41.91 0)
 			(effects
 				(font
@@
 		)
 		(property "Footprint" ""
-			(at 240.03 39.37 0)
+			(at 250.19 46.99 0)
 			(effects
 				(font
@@
 		)
 		(property "Datasheet" ""
-			(at 240.03 39.37 0)
+			(at 250.19 46.99 0)
 			(effects
 				(font
@@
 		)
 		(property "Description" "Power symbol creates a global label with name \"+3V3\""
-			(at 240.03 39.37 0)
+			(at 250.19 46.99 0)
 			(effects
 				(font
@@
 	(symbol
 		(lib_id "Device:R")
-		(at 243.84 46.99 0)
+		(at 255.27 54.61 0)
 		(unit 1)
 		(exclude_from_sim no)
@@
 		(dnp no)
 		(property "Reference" "R12"
-			(at 244.856 45.212 0)
+			(at 257.048 52.832 0)
 			(effects
 				(font
@@
 		)
 		(property "Value" "1K"
-			(at 244.856 46.99 0)
+			(at 257.048 55.372 0)
 			(effects
 				(font
@@
 		)
 		(property "Footprint" "Resistor_SMD:R_0603_1608Metric"
-			(at 242.062 46.99 90)
+			(at 253.492 54.61 90)
 			(effects
 				(font
@@
 		)
 		(property "Datasheet" "~"
-			(at 243.84 46.99 0)
+			(at 255.27 54.61 0)
 			(effects
 				(font
@@
 		)
 		(property "Description" "Resistor"
-			(at 243.84 46.99 0)
-			(effects
-				(font
+			(at 255.27 54.61 0)
+			(effects
+				(font

Commit message: added gitignore
Parts:
- renumbered U9 to U6
Changed lines of the file:
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@@
 		(on_board yes)
 		(dnp no)
-		(property "Reference" "U9"
+		(property "Reference" "U6"
 			(at 58.674 128.778 0)
 			(effects
@@
 			(project "flight-computer-one"
 				(path "/2b49a1e7-3a95-411d-8c49-438ba0d49dde/f69b98ff-ab10-4478-a5d1-a0199723a258"
-					(reference "U9")
+					(reference "U6")
 					(unit 1)
 				)

Commit message: Fixed BMI088 footprint and readme
Parts:
- U5: footprint LRI_partlib:PQFN50P450X300X100-16N -> LRI_partlib:QFN_BMI085_BOS
Other:
- note added: "Backup IMU Accel. I2C Addr: 0x18 Gyro. I2C Addr: 0x68"
- note added: "Temperature & humidity I2C Addr: 0x90"
- note removed: "I2C Addr: 0x90"
- note removed: "IMU Accel. I2C Addr: 0x18 Gyro. I2C Addr: 0x68"
- note removed: "Temperature"

Commit message: nearly completed schematic, partial layout
Parts:
- added C35: 4.7u, Capacitor_SMD:C_0805_2012Metric, symbol Device:C
- added C36: 0.1u, Capacitor_SMD:C_0603_1608Metric, symbol Device:C
- added C37: 10n, Capacitor_SMD:C_0603_1608Metric, symbol Device:C
- added U16: ICM-42688-P, LRI_partlib:IIM42352, symbol LRI_partlib:ICM-42688-P
Connections:
- net +3V3: now also C25.2, C26.1, C27.2, U7.10 (Vdd_IO), U7.9 (Vdd), C35.1, C36.2, C37.1, U16.5 (VDDIO), U16.8 (VDD)
- net GND: now also C25.1, C26.2, C27.1, C29.2, C35.2, C36.1, C37.2, U16.11 (RESV_11), U16.6 (GND), U16.7 (RESV_7)
- net at C29.1: now also U7.5 (C1)
- no-connect marks 8 -> 13
Other:
- note removed: "ICM-42688-P MISSING"
- moved on the sheet: C22, C23, C24, C25, C26, C28, C29, R11, R12, U5, U6, U7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

Commit message: schematic + prelim layout nearly complete
Connections:
- net SPI0_MISO: now reaches U16.1 (AP_SDO/AP_AD0)
- net CS_IMU_MAIN: now reaches U16.12 (AP_CS)
- net SPI0_SCK: now reaches U16.13 (AP_SCL/AP_SCLK)
- net SPI0_MOSI: now reaches U16.14 (AP_SDA/AP_SDIO/AP_SDI)
- net IMU_MAIN_INT: now reaches U16.4 (INT1/INT)
- no-connect marks 13 -> 14
Other:
- note added: "Main IMU SPI, active w CS_IMU_MAIN"
- moved on the sheet: C35, C36, C37, U16

Commit message: Schematic tentatively complete
Parts:
- C35: footprint Capacitor_SMD:C_0805_2012Metric -> Capacitor_SMD:C_0402_1005Metric
Changed lines of the file:
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@@
 			)
 		)
-		(property "Footprint" "Capacitor_SMD:C_0805_2012Metric"
+		(property "Footprint" "Capacitor_SMD:C_0402_1005Metric"
 			(at 98.7552 127 0)
 			(effects
