File: sensors.kicad_sch (KiCad schematic)
At the start: 18 parts, among them U16 ICM-42688-P, U5 BMI088, U6 MS5611-01BA, U7 LIS2MDL, U8 SHT4x

Commit message: schematic tentatively finished
Parts:
- removed R11, R12: 1K, Resistor_SMD:R_0603_1608Metric, symbol Device:R
Other:
- note removed: "Bus pull-up resistors"
- moved on the sheet: C28, C35, C36, C37, U16, U8

Commit message: same51 wired, near completion
Parts:
- C20: renamed from C35; footprint Capacitor_SMD:C_0402_1005Metric -> Capacitor_SMD:C_0603_1608Metric
- U10: renamed from U8; value SHT4x -> SHT40
- renumbered C24 to C17, C22 to C18, C23 to C19, C36 to C21, C37 to C22, C27 to C23, C29 to C24, C26 to C25, C25 to C26, C28 to C27, U5 to U6, U6 to U7, U7 to U8, U16 to U9

Commit message: Moved ICM to I2C
Connections:
- net CS_IMU_MAIN is gone; now on net +3V3: U9.12 (AP_CS)
- net SPI0_MISO is gone; now on net +3V3: U9.1 (AP_SDO/AP_AD0)
- net SPI0_MOSI is gone; now on net I2C0_SDA: U9.14 (AP_SDA/AP_SDIO/AP_SDI)
- net SPI0_SCK is gone; now on net I2C0_SCL: U9.13 (AP_SCL/AP_SCLK)
Other:
- note added: "Main IMU I2C Address: 0x69"
- note removed: "Main IMU SPI, active w CS_IMU_MAIN"
Changed lines of the file:
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@@
 		)
 	)
-	(text "Main IMU\nSPI, active w CS_IMU_MAIN"
+	(text "Main IMU\nI2C Address: 0x69"
 		(exclude_from_sim no)
 		(at 164.338 94.234 0)
@@
 	)
 	(junction
+		(at 144.78 132.08)
+		(diameter 0)
+		(color 0 0 0 0)
+	)
+	(junction
 		(at 53.34 102.87)
 		(diameter 0)
@@
 	(wire
 		(pts
+			(xy 142.24 129.54) (xy 146.05 129.54)
+		)
+		(stroke
+			(width 0)
+			(type default)
+		)
+	)
+	(wire
+		(pts
 			(xy 116.84 109.22) (xy 116.84 107.95)
 		)
@@
 	(wire
 		(pts
-			(xy 138.43 129.54) (xy 146.05 129.54)
-		)
-		(stroke
-			(width 0)
-			(type default)
-		)
-	)
-	(wire
-		(pts
 			(xy 53.34 101.6) (xy 53.34 102.87)
 		)
@@
 	(wire
 		(pts
+			(xy 146.05 124.46) (xy 144.78 124.46)
+		)
+		(stroke
+			(width 0)
+			(type default)
+		)
+	)
+	(wire
+		(pts
 			(xy 72.39 67.31) (xy 72.39 69.85)
 		)
@@
 	(wire
 		(pts
+			(xy 144.78 124.46) (xy 144.78 132.08)
+		)
+		(stroke
+			(width 0)
+			(type default)
+		)
+	)
+	(wire
+		(pts
 			(xy 66.04 125.73) (xy 53.34 125.73)
 		)
@@
 	(wire
 		(pts
+			(xy 144.78 133.35) (xy 144.78 132.08)
+		)
+		(stroke
+			(width 0)
+			(type default)
+		)
+	)
+	(wire
+		(pts
 			(xy 66.04 119.38) (xy 66.04 125.73)
 		)
@@
 	(wire
 		(pts
+			(xy 142.24 127) (xy 146.05 127)
+		)
+		(stroke
+			(width 0)
+			(type default)
+		)
+	)
+	(wire
+		(pts
 			(xy 116.84 118.11) (xy 129.54 118.11)
 		)
@@
 	(wire
 		(pts
-			(xy 138.43 127) (xy 146.05 127)
-		)
-		(stroke
-			(width 0)
-			(type default)
-		)
-	)
-	(wire
-		(pts
 			(xy 77.47 49.53) (xy 77.47 52.07)
 		)
@@
 	(wire
 		(pts
-			(xy 138.43 132.08) (xy 146.05 132.08)
-		)
-		(stroke
-			(width 0)
-			(type default)
-		)
-	)
-	(wire
-		(pts
-			(xy 138.43 124.46) (xy 146.05 124.46)
-		)
-		(stroke
-			(width 0)
-			(type default)
-		)
-	)
-	(wire
-		(pts
 			(xy 116.84 106.68) (xy 116.84 107.95)
 		)
@@
 		(pts
 			(xy 199.39 132.08) (xy 199.39 134.62)
+		)
+		(stroke
+			(width 0)
+			(type default)
+		)
+	)
+	(wire
+		(pts
+			(xy 144.78 132.08) (xy 146.05 132.08)
 		)
 		(stroke
@@
 			)
 			(justify right bottom)
-		)
-	)
-	(hierarchical_label "SPI0_MOSI"
-		(shape input)
-		(at 138.43 129.54 180)
-		(effects
-			(font
-				(size 1.27 1.27)
-			)
-			(justify right)
 		)
 	)
@@
 		)
 	)
-	(hierarchical_label "CS_IMU_MAIN"
-		(shape input)
-		(at 138.43 124.46 180)
-		(effects
-			(font
-				(size 1.27 1.27)
-			)
-			(justify right)
-		)
-	)
-	(hierarchical_label "SPI0_MISO"
-		(shape output)
-		(at 138.43 132.08 180)
-		(effects
-			(font
-				(size 1.27 1.27)
-			)
-			(justify right)
-		)
-	)
-	(hierarchical_label "SPI0_SCK"
-		(shape input)
-		(at 138.43 127 180)
+	(hierarchical_label "I2C0_SDA"
+		(shape bidirectional)
+		(at 142.24 129.54 180)
 		(effects
 			(font
@@
 		(shape bidirectional)
 		(at 125.73 57.15 180)
+		(effects
+			(font
+				(size 1.27 1.27)
+			)
+			(justify right)
+		)
+	)
+	(hierarchical_label "I2C0_SCL"
+		(shape input)
+		(at 142.24 127 180)
 		(effects
 			(font
@@
 					(unit 1)
 				)
+			)
+		)
+	)
+	(symbol
+		(lib_id "power:+3V3")
+		(at 144.78 133.35 180)
+		(unit 1)
+		(exclude_from_sim no)
+		(in_bom yes)
+		(on_board yes)
+		(dnp no)
+		(fields_autoplaced yes)
+		(property "Reference" "#PWR0101"
+			(at 144.78 129.54 0)
+			(effects
+				(font
+					(size 1.27 1.27)
+				)
+				(hide yes)
+			)
+		)
+		(property "Value" "+3V3"
+			(at 144.78 138.43 0)
+			(effects
+				(font
+					(size 1.27 1.27)
+				)
+			)
+		)
+		(property "Footprint" ""
+			(at 144.78 133.35 0)
+			(effects
+				(font
+					(size 1.27 1.27)
+				)
+				(hide yes)
+			)
+		)
+		(property "Datasheet" ""
+			(at 144.78 133.35 0)
+			(effects
+				(font
+					(size 1.27 1.27)
+				)
+				(hide yes)
+			)
+		)
+		(property "Description" "Power symbol creates a global label with name \"+3V3\""
+			(at 144.78 133.35 0)
+			(effects
+				(font
+					(size 1.27 1.27)
+				)
+				(hide yes)
+			)
+		)
+		(pin "1"
+		)
+		(instances
+			(project "flight-computer-one"
+				(path "/2b49a1e7-3a95-411d-8c49-438ba0d49dde/f69b98ff-ab10-4478-a5d1-a0199723a258"
+					(reference "#PWR0101")
+					(unit 1)
+				)

Commit message: Final schematic changes
Connections:
- net +3V3: no longer U9.1 (AP_SDO/AP_AD0), U9.12 (AP_CS)
- net I2C0_SCL: no longer U9.13 (AP_SCL/AP_SCLK)
- net I2C0_SDA: no longer U9.14 (AP_SDA/AP_SDIO/AP_SDI)
- new net CS_ICM: U9.12 (AP_CS)
- new net SPI0_MISO: U9.1 (AP_SDO/AP_AD0)
- new net SPI0_MOSI: U9.14 (AP_SDA/AP_SDIO/AP_SDI)
- new net SPI0_SCK: U9.13 (AP_SCL/AP_SCLK)
Changed lines of the file:
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@@
-	)
-	(junction
-		(at 144.78 132.08)
-		(diameter 0)
-		(color 0 0 0 0)
 	)
 	(junction
@@
 	(wire
 		(pts
+			(xy 142.24 129.54) (xy 146.05 129.54)
+		)
+		(stroke
+			(width 0)
+			(type default)
+		)
+	)
+	(wire
+		(pts
 			(xy 161.29 34.29) (xy 161.29 33.02)
 		)
@@
 	(wire
 		(pts
-			(xy 142.24 129.54) (xy 146.05 129.54)
-		)
-		(stroke
-			(width 0)
-			(type default)
-		)
-	)
-	(wire
-		(pts
 			(xy 116.84 109.22) (xy 116.84 107.95)
 		)
@@
 	(wire
 		(pts
-			(xy 146.05 124.46) (xy 144.78 124.46)
-		)
-		(stroke
-			(width 0)
-			(type default)
-		)
-	)
-	(wire
-		(pts
 			(xy 72.39 67.31) (xy 72.39 69.85)
 		)
@@
 	(wire
 		(pts
+			(xy 142.24 124.46) (xy 146.05 124.46)
+		)
+		(stroke
+			(width 0)
+			(type default)
+		)
+	)
+	(wire
+		(pts
 			(xy 53.34 125.73) (xy 53.34 127)
 		)
@@
 	(wire
 		(pts
+			(xy 142.24 127) (xy 146.05 127)
+		)
+		(stroke
+			(width 0)
+			(type default)
+		)
+	)
+	(wire
+		(pts
 			(xy 140.97 109.22) (xy 140.97 107.95)
 		)
@@
 	(wire
 		(pts
+			(xy 142.24 132.08) (xy 146.05 132.08)
+		)
+		(stroke
+			(width 0)
+			(type default)
+		)
+	)
+	(wire
+		(pts
 			(xy 140.97 41.91) (xy 140.97 43.18)
 		)
@@
 	(wire
 		(pts
-			(xy 144.78 124.46) (xy 144.78 132.08)
-		)
-		(stroke
-			(width 0)
-			(type default)
-		)
-	)
-	(wire
-		(pts
 			(xy 66.04 125.73) (xy 53.34 125.73)
 		)
@@
 	(wire
 		(pts
-			(xy 144.78 133.35) (xy 144.78 132.08)
-		)
-		(stroke
-			(width 0)
-			(type default)
-		)
-	)
-	(wire
-		(pts
 			(xy 66.04 119.38) (xy 66.04 125.73)
 		)
@@
 	(wire
 		(pts
-			(xy 142.24 127) (xy 146.05 127)
-		)
-		(stroke
-			(width 0)
-			(type default)
-		)
-	)
-	(wire
-		(pts
 			(xy 116.84 118.11) (xy 129.54 118.11)
 		)
@@
 		(pts
 			(xy 199.39 132.08) (xy 199.39 134.62)
-		)
-		(stroke
-			(width 0)
-			(type default)
-		)
-	)
-	(wire
-		(pts
-			(xy 144.78 132.08) (xy 146.05 132.08)
 		)
 		(stroke
@@
 			)
 			(justify right bottom)
+		)
+	)
+	(hierarchical_label "SPI0_MOSI"
+		(shape output)
+		(at 142.24 129.54 180)
+		(effects
+			(font
+				(size 1.27 1.27)
+			)
+			(justify right)
 		)
 	)
@@
 		)
 	)
+	(hierarchical_label "SPI0_MISO"
+		(shape output)
+		(at 142.24 132.08 180)
+		(effects
+			(font
+				(size 1.27 1.27)
+			)
+			(justify right)
+		)
+	)
 	(hierarchical_label "I2C0_SDA"
 		(shape bidirectional)
@@
 	(hierarchical_label "I2C0_SDA"
 		(shape bidirectional)
-		(at 142.24 129.54 180)
+		(at 217.17 59.69 180)
 		(effects
 			(font
@@
 		)
 	)
-	(hierarchical_label "I2C0_SDA"
-		(shape bidirectional)
-		(at 217.17 59.69 180)
+	(hierarchical_label "CS_ICM"
+		(shape output)
+		(at 142.24 124.46 180)
 		(effects
 			(font
@@
 	(hierarchical_label "I2C0_SCL"
 		(shape input)
-		(at 142.24 127 180)
-		(effects
-			(font
-				(size 1.27 1.27)
-			)
-			(justify right)
-		)
-	)
-	(hierarchical_label "I2C0_SCL"
-		(shape input)
 		(at 217.17 54.61 180)
 		(effects
@@
 		(shape bidirectional)
 		(at 31.75 59.69 180)
+		(effects
+			(font
+				(size 1.27 1.27)
+			)
+			(justify right)
+		)
+	)
+	(hierarchical_label "SPI0_SCK"
+		(shape input)
+		(at 142.24 127 180)
 		(effects
 			(font
@@
 					(unit 1)
 				)
-			)
-		)
-	)
-	(symbol
-		(lib_id "power:+3V3")
-		(at 144.78 133.35 180)
-		(unit 1)
-		(exclude_from_sim no)
-		(in_bom yes)
-		(on_board yes)
-		(dnp no)
-		(fields_autoplaced yes)
-		(property "Reference" "#PWR0101"
-			(at 144.78 129.54 0)
-			(effects
-				(font
-					(size 1.27 1.27)
-				)
-				(hide yes)
-			)
-		)
-		(property "Value" "+3V3"
-			(at 144.78 138.43 0)
-			(effects
-				(font
-					(size 1.27 1.27)
-				)
-			)
-		)
-		(property "Footprint" ""
-			(at 144.78 133.35 0)
-			(effects
-				(font
-					(size 1.27 1.27)
-				)
-				(hide yes)
-			)
-		)
-		(property "Datasheet" ""
-			(at 144.78 133.35 0)
-			(effects
-				(font
-					(size 1.27 1.27)
-				)
-				(hide yes)
-			)
-		)
-		(property "Description" "Power symbol creates a global label with name \"+3V3\""
-			(at 144.78 133.35 0)
-			(effects
-				(font
-					(size 1.27 1.27)
-				)
-				(hide yes)
-			)
-		)
-		(pin "1"
-		)
-		(instances
-			(project "flight-computer-one"
-				(path "/2b49a1e7-3a95-411d-8c49-438ba0d49dde/f69b98ff-ab10-4478-a5d1-a0199723a258"
-					(reference "#PWR0101")
-					(unit 1)
-				)

Commit message: final production files
Parts:
- U10: DK Part (none) -> https://www.digikey.com/en/products/detail/sensirion-ag/SHT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
- U7: DK Part (none) -> https://www.digikey.com/en/products/detail/te-connectivity-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
Changed lines of the file:
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@@
+			)
+		)
+		(property "DK Part" "https://www.digikey.com/en/products/detail/sensirion-ag/SHT40-AD1B-R2/13532084"
+			(at 227.33 57.15 0)
+			(effects
+				(font
+					(size 1.27 1.27)
+				)
+				(hide yes)
 			)
 		)
@@
 			(at 53.34 114.3 0)
 			(effects
+				(font
+					(size 1.27 1.27)
+				)
+				(hide yes)
+			)
+		)
+		(property "DK Part" "https://www.digikey.com/en/products/detail/te-connectivity-measurement-specialties/MS561101BA03-50/5277445"
+			(at 53.34 114.3 0)
+			(effects
