File: compute.kicad_sch (KiCad schematic)
At the start: 0 parts

Commit message: Copied over completed compute page
Parts:
- added C1, C19, C5: 10u, Capacitor_SMD:C_0805_2012Metric, symbol Device:C
- added C10, C6, C7, C9: 4.7u, Capacitor_SMD:C_0805_2012Metric, symbol Device:C
- added C11, C12, C13, C14, C15, C16, C17, C18, C2, C20, C21, C8: 100n, Capacitor_SMD:C_0603_1608Metric, symbol Device:C
- added C3, C4: 15p, Capacitor_SMD:C_0603_1608Metric, symbol Device:C
- added J1: USB_C_Receptacle_USB2.0_16P, Connector_USB:USB_C_Receptacle_GCT_USB4110, symbol Connector:USB_C_Receptacle_USB2.0_16P
- added L1: 3.3u, RP2350_80QFN_minimal:L_pol_2016, symbol Device:L
- added R1, R9: DNF, Resistor_SMD:R_0402_1005Metric, symbol Device:R
- added R10: 0, Resistor_SMD:R_0402_1005Metric, symbol Device:R
- added R13: 5k1, Capacitor_SMD:C_0603_1608Metric, symbol Device:R
- added R2, R4, R6: 1k, Resistor_SMD:R_0402_1005Metric, symbol Device:R
- added R3: 33, Resistor_SMD:R_0402_1005Metric, symbol Device:R
- added R5: 5k1, symbol Device:R
- added R7, R8: 27, Resistor_SMD:R_0402_1005Metric, symbol Device:R
- added SW1, SW2: SW_Push, Button_Switch_SMD:SW_Push_1P1T_NO_Vertical_Wuerth_434133025816, symbol Switch:SW_Push
- added U1: RP2350_80QFN, Package_DFN_QFN:QFN-80-1EP_10x10mm_P0.4mm_EP3.4x3.4mm_ThermalVias, symbol MCU_RaspberryPi_RP2350:RP2350_80QFN
- added U2: NCP1117-3.3_SOT223, Package_TO_SOT_SMD:SOT-223-3_TabPin2, symbol Regulator_Linear:NCP1117-3.3_SOT223
- added U3: W25Q128JVS, Package_SO:SOIC-8_5.23x5.23mm_P1.27mm, symbol Memory_Flash:W25Q128JVS
- added Y1: ABM8-272-T3, Crystal:Crystal_SMD_3225-4Pin_3.2x2.5mm, symbol Device:Crystal_GND24
Connections:
- new net: C4.1, R2.2, Y1.3
- new net: R7.2, U1.67 (USB_DP)
- new net: R8.2, U1.66 (USB_DM)
- new net: R4.1, SW2.1
- new net: J1.B5 (CC2), R13.1
- new net: J1.A5 (CC1), R5.1
- new net +1V1: C10.1, C11.1, C7.1, C8.1, L1.1, U1.10 (DVDD), U1.32 (DVDD), U1.51 (DVDD), U1.64 (VREG_VIN), U1.65 (VREG_FB)
- new net +3V3: C12.1, C13.1, C14.1, C15.1, C16.1, C17.1, C18.1, C19.1, C2.1, C20.1, C21.1, C5.1, C6.1, R1.1, R3.1, U1.15 (IOVDD), U1.24 (IOVDD), U1.29 (IOVDD), U1.41 (IOVDD), U1.5 (IOVDD), U1.50 (IOVDD), U1.59 (ADC_AVDD), U1.60 (IOVDD), U1.68 (USB_OTP_VDD), U1.69 (QSPI_IOVDD), U1.76 (IOVDD), U2.2 (VO), U3.8 (VCC)
- new net FLASH_SS: R1.2, R10.2, R9.2, U3.1 (~{CS})
- new net GND: C1.2, C10.2, C11.2, C12.2, C13.2, C14.2, C15.2, C16.2, C17.2, C18.2, C19.2, C2.2, C20.2, C21.2, C3.2, C4.2, C5.2, C6.2, C7.2, C8.2, C9.2, J1.A1 (GND), J1.A12 (GND), J1.B1 (GND), J1.B12 (GND), J1.S1 (SHIELD), R13.2, R4.2, R5.2, SW1.1, U1.62 (VREG_PGND), U1.81 (GND), U2.1 (GND), U3.4 (GND), Y1.2, Y1.4
- new net GPIO0: R9.1, U1.77 (GPIO0)
- new net GPIO1: U1.78 (GPIO1)
- new net GPIO10: U1.8 (GPIO10)
- new net GPIO11: U1.9 (GPIO11)
- new net GPIO12: U1.11 (GPIO12)
- new net GPIO13: U1.12 (GPIO13)
- new net GPIO14: U1.13 (GPIO14)
- new net GPIO15: U1.14 (GPIO15)
- new net GPIO16: U1.16 (GPIO16)
- new net GPIO17: U1.17 (GPIO17)
- new net GPIO18: U1.18 (GPIO18)
- new net GPIO19: U1.19 (GPIO19)
- new net GPIO2: U1.79 (GPIO2)
- new net GPIO20: U1.20 (GPIO20)
- new net GPIO21: U1.21 (GPIO21)
- new net GPIO22: U1.22 (GPIO22)
- new net GPIO23: U1.23 (GPIO23)
- new net GPIO24: U1.25 (GPIO24)
- new net GPIO25: U1.26 (GPIO25)
- new net GPIO26: U1.27 (GPIO26)
- new net GPIO27: U1.28 (GPIO27)
- new net GPIO28: U1.36 (GPIO28)
- new net GPIO29: U1.37 (GPIO29)
- new net GPIO3: U1.80 (GPIO3)
- new net GPIO30: U1.38 (GPIO30)
- new net GPIO31: U1.39 (GPIO31)
- new net GPIO32: U1.40 (GPIO32)
- new net GPIO33: U1.42 (GPIO33)
- new net GPIO34: U1.43 (GPIO34)
- new net GPIO35: U1.44 (GPIO35)
- new net GPIO36: U1.45 (GPIO36)
- new net GPIO37: U1.46 (GPIO37)
- new net GPIO38: U1.47 (GPIO38)
- new net GPIO39: U1.48 (GPIO39)
- new net GPIO4: U1.1 (GPIO4)
- new net GPIO40_ADC0: U1.49 (GPIO40_ADC0)
- new net GPIO41_ADC1: U1.52 (GPIO41_ADC1)
- new net GPIO42_ADC2: U1.53 (GPIO42_ADC2)
- new net GPIO43_ADC3: U1.54 (GPIO43_ADC3)
- new net GPIO44_ADC4: U1.55 (GPIO44_ADC4)
- new net GPIO45_ADC5: U1.56 (GPIO45_ADC5)
- new net GPIO46_ADC6: U1.57 (GPIO46_ADC6)
- new net GPIO47_ADC7: U1.58 (GPIO47_ADC7)
- new net GPIO5: U1.2 (GPIO5)
- new net GPIO6: U1.3 (GPIO6)
- new net GPIO7: U1.4 (GPIO7)
- new net GPIO8: U1.6 (GPIO8)
- new net GPIO9: U1.7 (GPIO9)
- new net QSPI_SCLK: U1.71 (QSPI_SCLK), U3.6 (CLK)
- new net QSPI_SD0: U1.72 (QSPI_SD0), U3.5 (DI(IO0))
- new net QSPI_SD1: U1.74 (QSPI_SD1), U3.2 (DO(IO1))
- new net QSPI_SD2: U1.73 (QSPI_SD2), U3.3 (IO2)
- new net QSPI_SD3: U1.70 (QSPI_SD3), U3.7 (IO3)
- new net QSPI_SS: R10.1, R6.1, U1.75 (QSPI_SS)
- new net RUN: SW2.2, U1.35 (RUN)
- new net SWCLK: U1.33 (SWCLK)
- new net SWD: U1.34 (SWD)
- new net USB_D+: J1.A7 (D-), J1.B7 (D-), R7.1
- new net USB_D-: J1.A6 (D+), J1.B6 (D+), R8.1
- new net VBUS: C1.1, J1.A4 (VBUS), J1.A9 (VBUS), J1.B4 (VBUS), J1.B9 (VBUS), U2.3 (VI)
- new net VREG_AVDD: C9.1, R3.2, U1.61 (VREG_AVDD)
- new net VREG_LX: L1.2, U1.63 (VREG_LX)
- new net XIN: C3.1, U1.30 (XIN), Y1.1
- new net XOUT: R2.1, U1.31 (XOUT)
- new net ~{USB_BOOT}: R6.2, SW1.2
- no-connect marks 0 -> 2
Other:
- note added: "12MHz Crystal"
- note added: "Power"
- note added: "QSPI Flash"

Commit message: the beginnings of a footprint
Parts:
- removed U3: W25Q128JVS, Package_SO:SOIC-8_5.23x5.23mm_P1.27mm, symbol Memory_Flash:W25Q128JVS
- added U10: USBLC6-2SC6, Package_TO_SOT_SMD:SOT-23-6, symbol Power_Protection:USBLC6-2SC6
- added U3: W25Q32JVSS, Package_SO:SOIC-8_5.3x5.3mm_P1.27mm, symbol Memory_Flash:W25Q32JVSS
- C11, C12, C13, C14, C15, C16, C17, C18, C2, C20, C21, C8: value 100n -> 0.1u
- L1: value 3.3u -> 3.3uH; footprint RP2350_80QFN_minimal:L_pol_2016 -> Inductor_SMD:L_Murata_DFE201610P
- R5: footprint (none) -> Resistor_SMD:R_0603_1608Metric
Connections:
- net +3V3: now also U3.8 (VCC)
- net FLASH_SS: now also U3.1 (~{CS})
- net GND: now also U3.4 (GND)
- net QSPI_SCLK: now also U3.6 (CLK)
- net QSPI_SD0: now also U3.5 (DI/IO_{0})
- net QSPI_SD1: now also U3.2 (DO/IO_{1})
- net QSPI_SD2: now also U3.3 (~{WP}/IO_{2})
- net QSPI_SD3: now also U3.7 (~{HOLD}/~{RESET}/IO_{3})
Other:
- moved on the sheet: C2, R1, R10, R9

Commit message: created project lib
Parts:
- removed C1, C19, C5: 10u, Capacitor_SMD:C_0805_2012Metric, symbol Device:C
- removed J1: USB_C_Receptacle_USB2.0_16P, Connector_USB:USB_C_Receptacle_GCT_USB4110, symbol Connector:USB_C_Receptacle_USB2.0_16P
- removed R13: 5k1, Capacitor_SMD:C_0603_1608Metric, symbol Device:R
- removed R5: 5k1, Resistor_SMD:R_0603_1608Metric, symbol Device:R
- removed U10: USBLC6-2SC6, Package_TO_SOT_SMD:SOT-23-6, symbol Power_Protection:USBLC6-2SC6
- removed U2: NCP1117-3.3_SOT223, Package_TO_SOT_SMD:SOT-223-3_TabPin2, symbol Regulator_Linear:NCP1117-3.3_SOT223
- removed U3: W25Q32JVSS, Package_SO:SOIC-8_5.3x5.3mm_P1.27mm, symbol Memory_Flash:W25Q32JVSS
- added J4: Micro_SD_Card_Det2, Connector_Card:microSD_HC_Hirose_DM3AT-SF-PEJM5, symbol Connector:Micro_SD_Card_Det2
- added TP1: TestPoint, TestPoint:TestPoint_Pad_D1.0mm, symbol Connector:TestPoint
- added U3: W25Q32JVZP, Package_SON:WSON-8-1EP_6x5mm_P1.27mm_EP3.4x4.3mm, symbol Memory_Flash:W25Q32JVZP
- SW1: value SW_Push -> BOOTSEL
- SW2: value SW_Push -> USER
Connections:
- net +3V3: now also J4.4 (VDD), U3.8 (VCC)
- net FLASH_SS: now also U3.1 (~{CS})
- net GND: now also J4.11 (SHIELD), J4.6 (VSS), U3.4 (GND), U3.9 (EP)
- net QSPI_SCLK: now also U3.6 (CLK)
- net QSPI_SD0: now also U3.5 (DI/IO_{0})
- net QSPI_SD1: now also U3.2 (DO/IO_{1})
- net QSPI_SD2: now also U3.3 (~{WP}/IO_{2})
- net QSPI_SD3: now also U3.7 (~{HOLD}/~{RESET}/IO_{3})
- net RUN: now also TP1.1; no longer SW2.2
- no-connect marks 2 -> 0
Other:
- note removed: "Power"
- moved on the sheet: C2, R1, R10, R4, R9, SW2

Commit message: added gitignore
Parts:
- removed R1: DNF, Resistor_SMD:R_0402_1005Metric, symbol Device:R
- added J7: Conn_01x03_Pin, Connector_JST:JST_SH_BM03B-SRSS-TB_1x03-1MP_P1.00mm_Vertical, symbol Connector:Conn_01x03_Pin
- added R13: 100K, Resistor_SMD:R_0603_1608Metric, symbol Device:R
- R1: renamed from R6; value 1k -> 1K; footprint Resistor_SMD:R_0402_1005Metric -> Resistor_SMD:R_0603_1608Metric
- R10: value 0 -> 100; footprint Resistor_SMD:R_0402_1005Metric -> Resistor_SMD:R_0603_1608Metric
- R2: value 1k -> 1K; footprint Resistor_SMD:R_0402_1005Metric -> Resistor_SMD:R_0603_1608Metric
- R3, R7, R8: footprint Resistor_SMD:R_0402_1005Metric -> Resistor_SMD:R_0603_1608Metric
- R4: value 1k -> 100K; footprint Resistor_SMD:R_0402_1005Metric -> Resistor_SMD:R_0603_1608Metric
- R9: value DNF -> 100; footprint Resistor_SMD:R_0402_1005Metric -> Resistor_SMD:R_0603_1608Metric; now fitted
- renumbered U3 to U2
Connections:
- net +3V3: now also R4.1, R13.1
- net GND: now also J4.9 (DET_B), SW2.1, J7.2 (Pin_2); no longer R4.2
- net GPIO0: no longer R9.1
- net QSPI_SS: now also U2.1 (~{CS}); no longer R10.1
- net SWCLK: now also R9.1, J7.3 (Pin_3); no longer U1.33 (SWCLK)
- net DAT2: now reaches J4.1 (DAT2)
- net CARD_DET: now reaches J4.10 (DET_A)
- net CARD_DET: now also R13.2
- net DAT3/CS: now reaches J4.2 (DAT3/CD)
- net CMD/MOSI: now reaches J4.3 (CMD)
- net SD_CLK: now reaches J4.5 (CLK)
- net DAT0/MISO: now reaches J4.7 (DAT0)
- net DAT1: now reaches J4.8 (DAT1)
- net at SW2.2: now also R4.2
- removed net FLASH_SS: R10.2, R9.2, U2.1 (~{CS})
- net SWD: no longer names the net of U1.34 (SWD)
- net SWD: now also R10.2
- new net: R9.2, U1.33 (SWCLK)
- new net SWDIO: J7.1 (Pin_1), R10.1
Other:
- note added: "SWD header"
- moved on the sheet: R4, R7, R8, SW2

Commit message: progress, particularly on power
Parts:
- U2: value W25Q32JVZP -> W25Q32RVXHJQ; footprint Package_SON:WSON-8-1EP_6x5mm_P1.27mm_EP3.4x4.3mm -> Package_SON:Winbond_USON-8-1EP_3x2mm_P0.5mm_EP0.2x1.6mm
Other:
- moved on the sheet: C2, J4, J7, R13, R4, SW2, U2

Commit message: schematic + prelim layout nearly complete
Parts:
- TP1: value TestPoint -> RUN
Connections:
- net USER_BTN: now reaches R4.2, SW2.2
Changed lines of the file:
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@@
 	(generator_version "9.0")
 	(paper "A4")
+	(rectangle
+		(start 15.24 143.51)
+		(end 73.66 180.34)
+		(stroke
+			(width 0)
+			(type dash)
+		)
+		(fill
+			(type none)
+		)
+	)
+	(rectangle
+		(start 219.71 104.14)
+		(end 280.67 158.75)
+		(stroke
+			(width 0)
+			(type dash)
+		)
+		(fill
+			(type none)
+		)
+	)
 	(circle
 		(center 44.45 51.435)
@@
 	(wire
 		(pts
-			(xy 191.77 129.54) (xy 200.66 129.54)
-		)
-		(stroke
-			(width 0)
-			(type default)
-		)
-	)
-	(wire
-		(pts
 			(xy 45.72 48.26) (xy 45.72 49.53)
 		)
@@
 	(wire
 		(pts
+			(xy 186.69 129.54) (xy 200.66 129.54)
+		)
+		(stroke
+			(width 0)
+			(type default)
+		)
+	)
+	(wire
+		(pts
 			(xy 161.29 31.75) (xy 161.29 33.02)
 		)
@@
 		)
 	)
+	(label "USER_BTN"
+		(at 186.69 129.54 0)
+		(effects
+			(font
+				(size 1.27 1.27)
+			)
+			(justify left bottom)
+		)
+	)
 	(label "SWDIO"
 		(at 40.64 120.65 180)
@@
 			)
 		)
-		(property "Value" "TestPoint"
+		(property "Value" "RUN"
 			(at 50.038 107.95 90)
 			(effects

Commit message: Schematic tentatively complete
Parts:
- added D2: Red 5mA, LED_SMD:LED_0603_1608Metric, symbol Device:LED
- added R38: 634, Resistor_SMD:R_0603_1608Metric, symbol Device:R
- C10, C6, C7, C9: footprint Capacitor_SMD:C_0805_2012Metric -> Capacitor_SMD:C_0402_1005Metric
- R3: footprint Resistor_SMD:R_0603_1608Metric -> Resistor_SMD:R_0402_1005Metric
Connections:
- net +1V1: no longer U1.64 (VREG_VIN)
- net +3V3: now also U1.64 (VREG_VIN)
- net GND: now also R38.2
- new net: D2.1 (K), R38.1
- new net USER_LED: D2.2 (A)
Other:
- moved on the sheet: R4, SW2

Commit message: schematic tentatively finished
Changed lines of the file:
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@@
 	(wire
 		(pts
-			(xy 160.02 46.99) (xy 171.45 46.99)
+			(xy 160.02 46.99) (xy 167.64 46.99)
 		)
 		(stroke
@@
 	(wire
 		(pts
-			(xy 160.02 49.53) (xy 171.45 49.53)
+			(xy 160.02 49.53) (xy 167.64 49.53)
 		)
 		(stroke
@@
 		)
 	)
-	(label "GPIO40_ADC0"
-		(at 160.02 161.29 180)
-		(effects
-			(font
-				(size 1.27 1.27)
-			)
-			(justify right bottom)
-		)
-	)
 	(label "GPIO9"
 		(at 160.02 80.01 180)
@@
 		)
 	)
-	(label "USB_D-"
-		(at 171.45 49.53 180)
-		(effects
-			(font
-				(size 1.27 1.27)
-			)
-			(justify right bottom)
-		)
-	)
 	(label "GPIO6"
 		(at 160.02 72.39 180)
@@
 		)
 	)
-	(label "USB_D+"
-		(at 171.45 46.99 180)
-		(effects
-			(font
-				(size 1.27 1.27)
-			)
-			(justify right bottom)
-		)
-	)
 	(label "QSPI_SCLK"
 		(at 62.23 83.82 0)
@@
 		)
 	)
+	(hierarchical_label "SERVO4_CTL"
+		(shape output)
+		(at 172.72 80.01 0)
+		(effects
+			(font
+				(size 1.27 1.27)
+			)
+			(justify left)
+		)
+	)
+	(hierarchical_label "SERVO1_CTL"
+		(shape output)
+		(at 172.72 72.39 0)
+		(effects
+			(font
+				(size 1.27 1.27)
+			)
+			(justify left)
+		)
+	)
+	(hierarchical_label "SPI0_MOSI"
+		(shape output)
+		(at 168.91 97.79 0)
+		(effects
+			(font
+				(size 1.27 1.27)
+			)
+			(justify left)
+		)
+	)
+	(hierarchical_label "TCAN_STB"
+		(shape output)
+		(at 172.72 64.77 0)
+		(effects
+			(font
+				(size 1.27 1.27)
+			)
+			(justify left)
+		)
+	)
+	(hierarchical_label "SERVO2_CTL"
+		(shape output)
+		(at 172.72 74.93 0)
+		(effects
+			(font
+				(size 1.27 1.27)
+			)
+			(justify left)
+		)
+	)
+	(hierarchical_label "USB_D-"
+		(shape bidirectional)
+		(at 167.64 49.53 0)
+		(effects
+			(font
+				(size 1.27 1.27)
+			)
+			(justify left)
+		)
+	)
+	(hierarchical_label "I2C0_SDA"
+		(shape bidirectional)
+		(at 170.18 86.36 0)
+		(effects
+			(font
+				(size 1.27 1.27)
+			)
+			(justify left)
+		)
+	)
+	(hierarchical_label "SERVO3_CTL"
+		(shape output)
+		(at 172.72 77.47 0)
+		(effects
+			(font
+				(size 1.27 1.27)
+			)
+			(justify left)
+		)
+	)
+	(hierarchical_label "SPI0_MISO"
+		(shape input)
+		(at 168.91 100.33 0)
+		(effects
+			(font
+				(size 1.27 1.27)
+			)
+			(justify left)
+		)
+	)
+	(hierarchical_label "CS_CANXC"
+		(shape output)
+		(at 168.91 109.22 0)
+		(effects
+			(font
+				(size 1.27 1.27)
+			)
+			(justify left)
+		)
+	)
+	(hierarchical_label "SPI0_SCK"
+		(shape output)
+		(at 168.91 95.25 0)
+		(effects
+			(font
+				(size 1.27 1.27)
+			)
+			(justify left)
+		)
+	)
+	(hierarchical_label "CS_RADIO"
+		(shape output)
+		(at 168.91 106.68 0)
+		(effects
+			(font
+				(size 1.27 1.27)
+			)
+			(justify left)
+		)
+	)
+	(hierarchical_label "BUZZER_CTL"
+		(shape output)
+		(at 172.72 67.31 0)
+		(effects
+			(font
+				(size 1.27 1.27)
+			)
+			(justify left)
+		)
+	)
+	(hierarchical_label "GPIO40_ADC0"
+		(shape bidirectional)
+		(at 160.02 161.29 0)
+		(effects
+			(font
+				(size 1.27 1.27)
+			)
+			(justify left)
+		)
+	)
+	(hierarchical_label "I2C0_SCL"
+		(shape output)
+		(at 170.18 88.9 0)
+		(effects
+			(font
+				(size 1.27 1.27)
+			)
+			(justify left)
+		)
+	)
+	(hierarchical_label "USB_D+"
+		(shape bidirectional)
+		(at 167.64 46.99 0)
+		(effects
+			(font
+				(size 1.27 1.27)
+			)
+			(justify left)
+		)
+	)
+	(hierarchical_label "CS_IMU_MAIN"
+		(shape output)
+		(at 168.91 104.14 0)
+		(effects
+			(font
+				(size 1.27 1.27)
+			)
+			(justify left)
+		)
+	)
