File: compute.kicad_sch (KiCad schematic)
At the start: 38 parts, among them J4 Micro_SD_Card_Det2, J7 Conn_01x03_Pin, SW1 BOOTSEL, SW2 USER, U1 RP2350_80QFN, U2 W25Q32RVXHJQ, Y1 ABM8-272-T3

Commit message: swapped POR chip for TPS2121
Connections:
- net GPIO33 is gone; now on net USER_LED: U1.42 (GPIO33)
- net GPIO36 is gone; now on net SERVO1_CTL: U1.45 (GPIO36)
- net GPIO37 is gone; now on net SERVO2_CTL: U1.46 (GPIO37)
- net GPIO38 is gone; now on net SERVO3_CTL: U1.47 (GPIO38)
- net GPIO39 is gone; now on net SERVO4_CTL: U1.48 (GPIO39)
Changed lines of the file:
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@@
 	(wire
 		(pts
-			(xy 144.78 140.97) (xy 160.02 140.97)
+			(xy 144.78 140.97) (xy 171.45 140.97)
 		)
 		(stroke
@@
 		)
 	)
-	(label "GPIO36"
-		(at 160.02 148.59 180)
-		(effects
-			(font
-				(size 1.27 1.27)
-			)
-			(justify right bottom)
-		)
-	)
 	(label "GPIO23"
 		(at 160.02 115.57 180)
@@
 		)
 	)
-	(label "GPIO39"
-		(at 160.02 156.21 180)
-		(effects
-			(font
-				(size 1.27 1.27)
-			)
-			(justify right bottom)
-		)
-	)
 	(label "GPIO43_ADC3"
 		(at 160.02 168.91 180)
@@
 		)
 	)
+	(label "USER_LED"
+		(at 171.45 140.97 180)
+		(effects
+			(font
+				(size 1.27 1.27)
+			)
+			(justify right bottom)
+		)
+	)
 	(label "QSPI_SD0"
 		(at 224.79 134.62 0)
@@
 		)
 	)
-	(label "GPIO37"
-		(at 160.02 151.13 180)
-		(effects
-			(font
-				(size 1.27 1.27)
-			)
-			(justify right bottom)
-		)
-	)
-	(label "GPIO38"
-		(at 160.02 153.67 180)
-		(effects
-			(font
-				(size 1.27 1.27)
-			)
-			(justify right bottom)
-		)
-	)
 	(label "GPIO10"
 		(at 160.02 82.55 180)
@@
 		)
 	)
-	(label "GPIO33"
-		(at 160.02 140.97 180)
-		(effects
-			(font
-				(size 1.27 1.27)
-			)
-			(justify right bottom)
-		)
-	)
 	(label "QSPI_SD2"
 		(at 224.79 139.7 0)
@@
 		)
 	)
+	(hierarchical_label "SERVO2_CTL"
+		(shape output)
+		(at 160.02 151.13 0)
+		(effects
+			(font
+				(size 1.27 1.27)
+			)
+			(justify left)
+		)
+	)
+	(hierarchical_label "SPI0_MOSI"
+		(shape output)
+		(at 168.91 96.52 0)
+		(effects
+			(font
+				(size 1.27 1.27)
+			)
+			(justify left)
+		)
+	)
+	(hierarchical_label "TCAN_STB"
+		(shape output)
+		(at 168.91 64.77 0)
+		(effects
+			(font
+				(size 1.27 1.27)
+			)
+			(justify left)
+		)
+	)
 	(hierarchical_label "SERVO4_CTL"
 		(shape output)
-		(at 172.72 80.01 0)
+		(at 160.02 156.21 0)
+		(effects
+			(font
+				(size 1.27 1.27)
+			)
+			(justify left)
+		)
+	)
+	(hierarchical_label "I2C0_SDA"
+		(shape bidirectional)
+		(at 168.91 85.09 0)
+		(effects
+			(font
+				(size 1.27 1.27)
+			)
+			(justify left)
+		)
+	)
+	(hierarchical_label "SPI0_MISO"
+		(shape input)
+		(at 168.91 99.06 0)
+		(effects
+			(font
+				(size 1.27 1.27)
+			)
+			(justify left)
+		)
+	)
+	(hierarchical_label "CS_CANXC"
+		(shape output)
+		(at 168.91 106.68 0)
+		(effects
+			(font
+				(size 1.27 1.27)
+			)
+			(justify left)
+		)
+	)
+	(hierarchical_label "SPI0_SCK"
+		(shape output)
+		(at 168.91 93.98 0)
+		(effects
+			(font
+				(size 1.27 1.27)
+			)
+			(justify left)
+		)
+	)
+	(hierarchical_label "CS_RADIO"
+		(shape output)
+		(at 168.91 104.14 0)
+		(effects
+			(font
+				(size 1.27 1.27)
+			)
+			(justify left)
+		)
+	)
+	(hierarchical_label "BUZZER_CTL"
+		(shape output)
+		(at 168.91 67.31 0)
+		(effects
+			(font
+				(size 1.27 1.27)
+			)
+			(justify left)
+		)
+	)
+	(hierarchical_label "GPIO40_ADC0"
+		(shape bidirectional)
+		(at 160.02 161.29 0)
 		(effects
 			(font
@@
 	(hierarchical_label "SERVO1_CTL"
 		(shape output)
-		(at 172.72 72.39 0)
+		(at 160.02 148.59 0)
 		(effects
 			(font
@@
 		)
 	)
-	(hierarchical_label "SPI0_MOSI"
+	(hierarchical_label "USB_D+"
+		(shape bidirectional)
+		(at 167.64 46.99 0)
+		(effects
+			(font
+				(size 1.27 1.27)
+			)
+			(justify left)
+		)
+		(property "Netclass" "USB_DIFF"
+			(at 177.038 46.99 0)
+			(effects
+				(font
+					(size 1.27 1.27)
+					(italic yes)
+				)
+				(justify left)
+			)
+		)
+	)
+	(hierarchical_label "SERVO3_CTL"
 		(shape output)
-		(at 168.91 97.79 0)
+		(at 160.02 153.67 0)
 		(effects
 			(font
@@
 		)
 	)
-	(hierarchical_label "TCAN_STB"
+	(hierarchical_label "I2C0_SCL"
 		(shape output)
-		(at 172.72 64.77 0)
-		(effects
-			(font
-				(size 1.27 1.27)
-			)
-			(justify left)
-		)
-	)
-	(hierarchical_label "SERVO2_CTL"
-		(shape output)
-		(at 172.72 74.93 0)
+		(at 168.91 87.63 0)
 		(effects
 			(font
@@
 			(justify left)
 		)
-	)
-	(hierarchical_label "I2C0_SDA"
-		(shape bidirectional)
-		(at 170.18 86.36 0)
-		(effects
-			(font
-				(size 1.27 1.27)
-			)
-			(justify left)
-		)
-	)
-	(hierarchical_label "SERVO3_CTL"
-		(shape output)
-		(at 172.72 77.47 0)
-		(effects
-			(font
-				(size 1.27 1.27)
-			)
-			(justify left)
-		)
-	)
-	(hierarchical_label "SPI0_MISO"
-		(shape input)
-		(at 168.91 100.33 0)
-		(effects
-			(font
-				(size 1.27 1.27)
-			)
-			(justify left)
-		)
-	)
-	(hierarchical_label "CS_CANXC"
-		(shape output)
-		(at 168.91 109.22 0)
-		(effects
-			(font
-				(size 1.27 1.27)
-			)
-			(justify left)
-		)
-	)
-	(hierarchical_label "SPI0_SCK"
-		(shape output)
-		(at 168.91 95.25 0)
-		(effects
-			(font
-				(size 1.27 1.27)
-			)
-			(justify left)
-		)
-	)
-	(hierarchical_label "CS_RADIO"
-		(shape output)
-		(at 168.91 106.68 0)
-		(effects
-			(font
-				(size 1.27 1.27)
-			)
-			(justify left)
-		)
-	)
-	(hierarchical_label "BUZZER_CTL"
-		(shape output)
-		(at 172.72 67.31 0)
-		(effects
-			(font
-				(size 1.27 1.27)
-			)
-			(justify left)
-		)
-	)
-	(hierarchical_label "GPIO40_ADC0"
-		(shape bidirectional)
-		(at 160.02 161.29 0)
-		(effects
-			(font
-				(size 1.27 1.27)
-			)
-			(justify left)
-		)
-	)
-	(hierarchical_label "I2C0_SCL"
-		(shape output)
-		(at 170.18 88.9 0)
-		(effects
-			(font
-				(size 1.27 1.27)
-			)
-			(justify left)
-		)
-	)
-	(hierarchical_label "USB_D+"
-		(shape bidirectional)
-		(at 167.64 46.99 0)
-		(effects
-			(font
-				(size 1.27 1.27)
-			)
-			(justify left)
+		(property "Netclass" "USB_DIFF"
+			(at 177.038 49.53 0)
+			(effects
+				(font
+					(size 1.27 1.27)
+					(italic yes)
+				)
+				(justify left)
+			)
 		)
 	)
 	(hierarchical_label "CS_IMU_MAIN"
 		(shape output)
-		(at 168.91 104.14 0)
-		(effects
-			(font
+		(at 168.91 101.6 0)
+		(effects
+			(font

Commit message: preliminary change to SAME51
Parts:
- removed C10, C9: 4.7u, Capacitor_SMD:C_0402_1005Metric, symbol Device:C
- removed C11, C17, C18, C2, C20, C21, C8: 0.1u, Capacitor_SMD:C_0603_1608Metric, symbol Device:C
- removed J7: Conn_01x03_Pin, Connector_JST:JST_SH_BM03B-SRSS-TB_1x03-1MP_P1.00mm_Vertical, symbol Connector:Conn_01x03_Pin
- removed L1: 3.3uH, Inductor_SMD:L_Murata_DFE201610P, symbol Device:L
- removed R10: 100, Resistor_SMD:R_0603_1608Metric, symbol Device:R
- removed R2: 1K, Resistor_SMD:R_0603_1608Metric, symbol Device:R
- removed R3: 33, Resistor_SMD:R_0402_1005Metric, symbol Device:R
- removed R7, R8: 27, Resistor_SMD:R_0603_1608Metric, symbol Device:R
- removed TP1: RUN, TestPoint:TestPoint_Pad_D1.0mm, symbol Connector:TestPoint
- removed U1: RP2350_80QFN, Package_DFN_QFN:QFN-80-1EP_10x10mm_P0.4mm_EP3.4x3.4mm_ThermalVias, symbol MCU_RaspberryPi_RP2350:RP2350_80QFN
- removed U2: W25Q32RVXHJQ, Package_SON:Winbond_USON-8-1EP_3x2mm_P0.5mm_EP0.2x1.6mm, symbol Memory_Flash:W25Q32JVZP
- added J7: Conn_02x05_Counter_Clockwise, Connector_PinSocket_1.27mm:PinSocket_2x05_P1.27mm_Vertical_SMD, symbol Connector_Generic:Conn_02x05_Counter_Clockwise
- added U13: ATSAME51J19A-M, Package_DFN_QFN:QFN-64-1EP_9x9mm_P0.5mm_EP4.7x4.7mm, symbol MCU_Microchip_SAMD:ATSAMD51J19A-M
- C6: value 4.7u -> 10u; footprint Capacitor_SMD:C_0402_1005Metric -> Capacitor_SMD:C_0603_1608Metric
- C7: value 4.7u -> 0.1u; footprint Capacitor_SMD:C_0402_1005Metric -> Capacitor_SMD:C_0603_1608Metric
- D2: value Red 5mA -> Green 5mA
- R1: value 1K -> 10K
- R9: value 100 -> 1K
- SW1: value BOOTSEL -> RESET
- Y1: footprint Crystal:Crystal_SMD_3225-4Pin_3.2x2.5mm -> Crystal:Crystal_SMD_2520-4Pin_2.5x2.0mm
Connections:
- net QSPI_SS is gone; now on net +3V3: R1.1
- net ~{USB_BOOT} is gone; now on net ~{RESET}: R1.2, SW1.2
- net +3V3: now also U13.21 (VDDIOB), U13.34 (VDDIO), U13.48 (VDDIO), U13.56 (VDDIO), U13.8 (VDDANA); no longer C6.1
- net GND: now also C6.1, U13.22 (GND), U13.33 (GND), U13.47 (GND), U13.54 (GND), U13.65 (GND), U13.7 (GNDANA); no longer C6.2
- net X2: now reaches C4.1, Y1.3
- net X2: now also U13.2 (PA01)
- net +1V1 renamed ~{RESET}
- net ~{RESET}: now also U13.52 (~{RESET})
- net XIN renamed X1
- net X1: now also U13.1 (PA00)
- new net: C6.2, U13.53 (VDDCORE)
- no-connect marks 0 -> 1
Other:
- note added: "1 USB pair (2 pins) 2 SPI (6 pins) 1 I2C (2 pins) 8 digital 5 pwm 1 analog in"
- note added: "32.768 kHz crystal"
- note added: "Surprisingly, this generates the system clk"
- note removed: "12MHz Crystal"
- note removed: "QSPI Flash"
- moved on the sheet: C12, C13, C14, C15, C16, C3, C4, C6, C7, R1, R9, SW1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

Commit message: same51 wired, near completion
Parts:
- removed C3, C4: 15p, Capacitor_SMD:C_0603_1608Metric, symbol Device:C
- removed Y1: ABM8-272-T3, Crystal:Crystal_SMD_2520-4Pin_2.5x2.0mm, symbol Device:Crystal_GND24
- added C9: 0.1u, Capacitor_SMD:C_0603_1608Metric, symbol Device:C
- added Y1: SiT8008BI-11-33N-20.000000, Oscillator:Oscillator_SMD_SiT_PQFN-4Pin_2.5x2.0mm, symbol Oscillator:SiT8008xx-1x-xxN
- J4: renamed from J7; value Conn_02x05_Counter_Clockwise -> SWD; footprint Connector_PinSocket_1.27mm:PinSocket_2x05_P1.27mm_Vertical_SMD -> Connector_PinHeader_1.27mm:PinHeader_2x05_P1.27mm_Vertical_SMD
- renumbered C7 to C10, C6 to C11, D2 to D3, J4 to J5, R9 to R14, R1 to R15, R13 to R16, R4 to R17, R38 to R18, U13 to U1
Connections:
- net +3V3: now also J4.1 (Pin_1), R14.1, C9.1, Y1.4 (Vdd)
- net BUZZER_CTL: now also U1.18 (PA09)
- net CARD_DET: now also U1.40 (PB17)
- net CMD/MOSI: now also U1.38 (PA19)
- net DAT0/MISO: now also U1.35 (PA16)
- net DAT3/CS: now also U1.37 (PA18)
- net GND: now also J4.2 (Pin_2), J4.3 (Pin_3), J4.5 (Pin_5), C9.2, Y1.2 (GND)
- net GPIO40_ADC0: now also U1.19 (PA10)
- net SD_CLK: now also U1.36 (PA17)
- net SERVO1_CTL: now also U1.28 (PB15)
- net SERVO2_CTL: now also U1.27 (PB14)
- net SERVO3_CTL: now also U1.26 (PB13)
- net SERVO4_CTL: now also U1.25 (PB12)
- net SWCLK: now also J4.9 (Pin_9), R14.2, U1.57 (PA30); no longer R14.1
- net SWDIO: now also J4.10 (Pin_10), U1.58 (PA31)
- net USB_D+: now also U1.46 (PA25)
- net USB_D-: now also U1.45 (PA24)
- net USER_BTN: now also U1.24 (PB11)
- net USER_LED: now also U1.39 (PB16)
- net ~{RESET}: now also J4.6 (Pin_6)
- net SWO: now reaches J4.8 (Pin_8)
- net SWO: now also U1.59 (PB30)
- net XIN: now reaches U1.31 (PA14)
- net XIN: now also Y1.3 (OUT)
- net XOUT: now reaches U1.32 (PA15)
- net TXCAN: now reaches U1.43 (PA22)
- net RXCAN: now reaches U1.44 (PA23)
- net X1: no longer names the net of U1.1 (PA00)
- net X2: no longer names the net of U1.2 (PA01)
- no-connect marks 1 -> 9
Other:
- note added: "20 MHz oscillator"
- note added: "CAN0"
- note added: "SERCOM3"
- note removed: "1 USB pair (2 pins) 2 SPI (6 pins) 1 I2C (2 pins) 8 digital 5 pwm 1 analog in"
- note removed: "32.768 kHz crystal"
- note removed: "Surprisingly, this generates the system clk"
- moved on the sheet: R14

Commit message: completed layout for Rev.A
Connections:
- net CS_IMU_MAIN: now also U1.61 (PB00)
- net CS_RADIO: now also U1.1 (PA00)
- net I2C0_SCL: now also U1.11 (PB08)
- net I2C0_SDA: now also U1.12 (PB09)
- net SPI0_MISO: now also U1.62 (PB01)
- net SPI0_MOSI: now also U1.63 (PB02)
- net SPI0_SCK: now also U1.64 (PB03)
- net TCAN_STB: now also U1.15 (PA06)
Other:
- note added: "SERCOM5"
Changed lines of the file:
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@@
+		)
+	)
+	(text "SERCOM5"
+		(exclude_from_sim no)
+		(at 177.038 61.468 90)
+		(effects
+			(font
+				(size 1.27 1.27)
+			)
 		)
 	)
@@
 	(wire
 		(pts
+			(xy 130.81 73.66) (xy 134.62 73.66)
+		)
+		(stroke
+			(width 0)
+			(type default)
+		)
+	)
+	(wire
+		(pts
 			(xy 46.99 154.94) (xy 46.99 157.48)
 		)
@@
 	(wire
 		(pts
+			(xy 130.81 55.88) (xy 134.62 55.88)
+		)
+		(stroke
+			(width 0)
+			(type default)
+		)
+	)
+	(wire
+		(pts
 			(xy 198.12 132.08) (xy 198.12 134.62)
 		)
@@
 	(wire
 		(pts
+			(xy 90.17 50.8) (xy 95.25 50.8)
+		)
+		(stroke
+			(width 0)
+			(type default)
+		)
+	)
+	(wire
+		(pts
 			(xy 132.08 35.56) (xy 132.08 36.83)
 		)
@@
 	(wire
 		(pts
+			(xy 130.81 58.42) (xy 134.62 58.42)
+		)
+		(stroke
+			(width 0)
+			(type default)
+		)
+	)
+	(wire
+		(pts
 			(xy 41.91 52.07) (xy 41.91 53.34)
 		)
@@
 	(wire
 		(pts
+			(xy 130.81 76.2) (xy 134.62 76.2)
+		)
+		(stroke
+			(width 0)
+			(type default)
+		)
+	)
+	(wire
+		(pts
 			(xy 22.86 93.98) (xy 25.4 93.98)
 		)
@@
 	(wire
 		(pts
+			(xy 130.81 53.34) (xy 134.62 53.34)
+		)
+		(stroke
+			(width 0)
+			(type default)
+		)
+	)
+	(wire
+		(pts
 			(xy 115.57 132.08) (xy 115.57 133.35)
 		)
@@
 	(wire
 		(pts
+			(xy 130.81 60.96) (xy 134.62 60.96)
+		)
+		(stroke
+			(width 0)
+			(type default)
+		)
+	)
+	(wire
+		(pts
 			(xy 96.52 35.56) (xy 93.98 35.56)
 		)
@@
 		(pts
 			(xy 154.94 26.67) (xy 166.37 26.67)
+		)
+		(stroke
+			(width 0)
+			(type default)
+		)
+	)
+	(wire
+		(pts
+			(xy 87.63 66.04) (xy 95.25 66.04)
 		)
 		(stroke
@@
 	(hierarchical_label "SPI0_MOSI"
 		(shape output)
-		(at 77.47 60.96 180)
-		(effects
-			(font
-				(size 1.27 1.27)
-			)
-			(justify right)
+		(at 134.62 58.42 0)
+		(effects
+			(font
+				(size 1.27 1.27)
+			)
+			(justify left)
 		)
 	)
 	(hierarchical_label "TCAN_STB"
 		(shape output)
-		(at 143.51 66.04 0)
-		(effects
-			(font
-				(size 1.27 1.27)
-			)
-			(justify left)
+		(at 87.63 66.04 180)
+		(effects
+			(font
+				(size 1.27 1.27)
+			)
+			(justify right)
 		)
 	)
@@
 	(hierarchical_label "I2C0_SDA"
 		(shape bidirectional)
-		(at 160.02 55.88 0)
+		(at 134.62 76.2 0)
 		(effects
 			(font
@@
 	(hierarchical_label "SPI0_MISO"
 		(shape input)
-		(at 77.47 68.58 180)
-		(effects
-			(font
-				(size 1.27 1.27)
-			)
-			(justify right)
+		(at 134.62 55.88 0)
+		(effects
+			(font
+				(size 1.27 1.27)
+			)
+			(justify left)
 		)
 	)
@@
 	(hierarchical_label "SPI0_SCK"
 		(shape output)
-		(at 92.71 63.5 180)
-		(effects
-			(font
-				(size 1.27 1.27)
-			)
-			(justify right)
+		(at 134.62 60.96 0)
+		(effects
+			(font
+				(size 1.27 1.27)
+			)
+			(justify left)
 		)
 	)
 	(hierarchical_label "CS_RADIO"
 		(shape output)
-		(at 77.47 49.53 180)
+		(at 90.17 50.8 180)
 		(effects
 			(font
@@
 	(hierarchical_label "I2C0_SCL"
 		(shape output)
-		(at 160.02 58.42 0)
+		(at 134.62 73.66 0)
 		(effects
 			(font
@@
 	(hierarchical_label "CS_IMU_MAIN"
 		(shape output)
-		(at 92.71 66.04 180)
-		(effects
-			(font
-				(size 1.27 1.27)
-			)
-			(justify right)
-		)
-	)
+		(at 134.62 53.34 0)
+		(effects
+			(font
+				(size 1.27 1.27)
+			)
+			(justify left)
+		)
+	)

Commit message: Moved ICM to I2C
Connections:
- net CS_IMU_MAIN: no longer names the net of U1.61 (PB00)
Changed lines of the file:
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@@
-	(wire
-		(pts
-			(xy 130.81 53.34) (xy 134.62 53.34)
-		)
-		(stroke
-			(width 0)
-			(type default)
-		)
-	)
 	(wire
 		(pts
@@
 		(effects
 			(font
-				(size 1.27 1.27)
-			)
-			(justify left)
-		)
-	)
-	(hierarchical_label "CS_IMU_MAIN"
-		(shape output)
-		(at 134.62 53.34 0)
-		(effects
-			(font

Commit message: Removed unecessary HSE
Parts:
- removed C9: 0.1u, Capacitor_SMD:C_0603_1608Metric, symbol Device:C
- removed Y1: SiT8008BI-11-33N-20.000000, Oscillator:Oscillator_SMD_SiT_PQFN-4Pin_2.5x2.0mm, symbol Oscillator:SiT8008xx-1x-xxN
Connections:
- net XIN: no longer names the net of U1.31 (PA14)
- net XOUT: no longer names the net of U1.32 (PA15)
Other:
- note removed: "20 MHz oscillator"

Commit message: Moved SD card to SPI
Connections:
- net CMD/MOSI: no longer J5.3 (CMD)
- net DAT0/MISO: no longer J5.7 (DAT0)
- net DAT3/CS: no longer J5.2 (DAT3/CD)
- net SD_CLK: no longer J5.5 (CLK)
- net DAT1: no longer names the net of J5.8 (DAT1)
- net DAT2: no longer names the net of J5.1 (DAT2)
- new net SD_CS: J5.2 (DAT3/CD)
- new net SPI_MISO: J5.7 (DAT0)
- new net SPI_MOSI: J5.3 (CMD)
- new net SPI_SCK: J5.5 (CLK)
- no-connect marks 9 -> 11
Changed lines of the file:
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@@
+	)
+	(no_connect
+		(at 226.06 60.96)
 	)
 	(no_connect
@@
 	)
 	(no_connect
+		(at 226.06 78.74)
+	)
+	(no_connect
 		(at 95.25 116.84)
 	)
@@
 	(wire
 		(pts
-			(xy 208.28 78.74) (xy 226.06 78.74)
-		)
-		(stroke
-			(width 0)
-			(type default)
-		)
-	)
-	(wire
-		(pts
 			(xy 110.49 40.64) (xy 110.49 35.56)
 		)
@@
 		(pts
 			(xy 87.63 76.2) (xy 95.25 76.2)
-		)
-		(stroke
-			(width 0)
-			(type default)
-		)
-	)
-	(wire
-		(pts
-			(xy 208.28 60.96) (xy 226.06 60.96)
 		)
 		(stroke
@@
 		)
 	)
-	(label "CMD{slash}MOSI"
+	(label "SPI_MOSI"
 		(at 208.28 66.04 0)
 		(effects
@@
 		)
 	)
-	(label "DAT0{slash}MISO"
+	(label "SPI_MISO"
 		(at 208.28 76.2 0)
 		(effects
@@
 		)
 	)
-	(label "DAT2"
-		(at 208.28 60.96 0)
-		(effects
-			(font
-				(size 1.27 1.27)
-			)
-			(justify left bottom)
-		)
-	)
 	(label "USER_BTN"
 		(at 184.15 134.62 0)
@@
 		)
 	)
-	(label "SD_CLK"
+	(label "SPI_SCK"
 		(at 208.28 71.12 0)
 		(effects
@@
 		)
 	)
-	(label "DAT3{slash}CS"
+	(label "SD_CS"
 		(at 208.28 63.5 0)
 		(effects
@@
 		)
 	)
-	(label "DAT1"
-		(at 208.28 78.74 0)
-		(effects
-			(font
-				(size 1.27 1.27)
-			)
-			(justify left bottom)
-		)
-	)

Commit message: Final schematic changes
Connections:
- net CMD/MOSI is gone; now on net SD_CS: U1.38 (PA19)
- net SPI_MISO is gone; now on net SD_MISO: J5.7 (DAT0)
- net SPI_MOSI is gone; now on net SD_MOSI: J5.3 (CMD)
- net SPI_SCK is gone; now on net SD_SCK: J5.5 (CLK)
- net CS_RADIO: now also U1.60 (PB31); no longer U1.1 (PA00)
- net I2C0_SCL: now also U1.12 (PB09); no longer U1.11 (PB08)
- net I2C0_SDA: now also U1.11 (PB08); no longer U1.12 (PB09)
- net PYRO2_FIRE: now reaches U1.13 (PA04)
- net PYRO2_PRESENT: now reaches U1.14 (PA05)
- net PYRO1_FIRE: now reaches U1.2 (PA01)
- net PYRO1_PRESENT: now reaches U1.3 (PA02)
- net PYRO2_ARM: now reaches U1.4 (PA03)
- net CS_ICM: now reaches U1.61 (PB00)
- net DAT0/MISO renamed SD_SCK
- net DAT3/CS renamed SD_MISO
- net SD_CLK renamed SD_MOSI
- new net PYRO1_ARM: U1.1 (PA00)
- no-connect marks 11 -> 10
