File: compute.kicad_sch (KiCad schematic)
At the start: 18 parts, among them J4 SWD, J5 Micro_SD_Card_Det2, SW1 RESET, SW2 USER, U1 ATSAME51J19A-M

Commit message: Moved power monitor to seperate I2C bus for easier routing
Connections:
- net I2C1_SDA: now reaches U1.29 (PA12)
- net I2C1_SCL: now reaches U1.30 (PA13)
Other:
- note added: "SERCOM2"
Changed lines of the file:
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@@
+		)
+	)
+	(text "SERCOM2"
+		(exclude_from_sim no)
+		(at 75.692 83.312 90)
+		(effects
+			(font
+				(size 1.27 1.27)
+			)
 		)
 	)
@@
 	(wire
 		(pts
+			(xy 87.63 83.82) (xy 95.25 83.82)
+		)
+		(stroke
+			(width 0)
+			(type default)
+		)
+	)
+	(wire
+		(pts
 			(xy 132.08 26.67) (xy 143.51 26.67)
 		)
@@
 		(pts
 			(xy 113.03 40.64) (xy 113.03 35.56)
+		)
+		(stroke
+			(width 0)
+			(type default)
+		)
+	)
+	(wire
+		(pts
+			(xy 87.63 81.28) (xy 95.25 81.28)
 		)
 		(stroke
@@
 		(effects
 			(font
+				(size 1.27 1.27)
+			)
+			(justify right)
+		)
+	)
+	(hierarchical_label "I2C1_SDA"
+		(shape bidirectional)
+		(at 87.63 81.28 180)
+		(effects
+			(font
+				(size 1.27 1.27)
+			)
+			(justify right)
+		)
+	)
+	(hierarchical_label "I2C1_SCL"
+		(shape output)
+		(at 87.63 83.82 180)
+		(effects
+			(font

Commit message: new routing
Connections:
- net PYRO1_ARM: now also U1.6 (PB05); no longer U1.1 (PA00)
- net PYRO1_FIRE: now also U1.5 (PB04); no longer U1.2 (PA01)
- net PYRO1_PRESENT: now also U1.4 (PA03); no longer U1.3 (PA02)
- net PYRO2_ARM: now also U1.3 (PA02); no longer U1.4 (PA03)
- net PYRO2_FIRE: now also U1.2 (PA01); no longer U1.13 (PA04)
- net PYRO2_PRESENT: now also U1.1 (PA00); no longer U1.14 (PA05)
- no-connect marks 10 -> 20
Changed lines of the file:
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@@
+	)
+	(no_connect
+		(at 95.25 68.58)
+	)
+	(no_connect
+		(at 95.25 78.74)
+	)
+	(no_connect
+		(at 95.25 60.96)
 	)
 	(no_connect
@@
 	)
 	(no_connect
+		(at 130.81 78.74)
+	)
+	(no_connect
 		(at 130.81 101.6)
 	)
 	(no_connect
+		(at 95.25 71.12)
+	)
+	(no_connect
+		(at 130.81 71.12)
+	)
+	(no_connect
+		(at 130.81 68.58)
+	)
+	(no_connect
+		(at 95.25 88.9)
+	)
+	(no_connect
+		(at 95.25 86.36)
+	)
+	(no_connect
 		(at 95.25 104.14)
 	)
@@
 	)
 	(no_connect
+		(at 95.25 63.5)
+	)
+	(no_connect
 		(at 95.25 116.84)
 	)
@@
 	(wire
 		(pts
-			(xy 87.63 63.5) (xy 95.25 63.5)
-		)
-		(stroke
-			(width 0)
-			(type default)
-		)
-	)
-	(wire
-		(pts
 			(xy 22.86 91.44) (xy 22.86 93.98)
 		)
@@
 	(wire
 		(pts
+			(xy 87.63 58.42) (xy 95.25 58.42)
+		)
+		(stroke
+			(width 0)
+			(type default)
+		)
+	)
+	(wire
+		(pts
 			(xy 87.63 83.82) (xy 95.25 83.82)
 		)
@@
 	(wire
 		(pts
+			(xy 87.63 50.8) (xy 95.25 50.8)
+		)
+		(stroke
+			(width 0)
+			(type default)
+		)
+	)
+	(wire
+		(pts
 			(xy 87.63 109.22) (xy 95.25 109.22)
 		)
@@
 	(wire
 		(pts
+			(xy 25.4 99.06) (xy 22.86 99.06)
+		)
+		(stroke
+			(width 0)
+			(type default)
+		)
+	)
+	(wire
+		(pts
+			(xy 34.29 156.21) (xy 34.29 157.48)
+		)
+		(stroke
+			(width 0)
+			(type default)
+		)
+	)
+	(wire
+		(pts
+			(xy 130.81 93.98) (xy 158.75 93.98)
+		)
+		(stroke
+			(width 0)
+			(type default)
+		)
+	)
+	(wire
+		(pts
+			(xy 82.55 127) (xy 95.25 127)
+		)
+		(stroke
+			(width 0)
+			(type default)
+		)
+	)
+	(wire
+		(pts
+			(xy 208.28 106.68) (xy 208.28 109.22)
+		)
+		(stroke
+			(width 0)
+			(type default)
+		)
+	)
+	(wire
+		(pts
+			(xy 115.57 133.35) (xy 113.03 133.35)
+		)
+		(stroke
+			(width 0)
+			(type default)
+		)
+	)
+	(wire
+		(pts
+			(xy 130.81 58.42) (xy 134.62 58.42)
+		)
+		(stroke
+			(width 0)
+			(type default)
+		)
+	)
+	(wire
+		(pts
 			(xy 87.63 53.34) (xy 95.25 53.34)
 		)
@@
 	(wire
 		(pts
-			(xy 25.4 99.06) (xy 22.86 99.06)
-		)
-		(stroke
-			(width 0)
-			(type default)
-		)
-	)
-	(wire
-		(pts
-			(xy 34.29 156.21) (xy 34.29 157.48)
-		)
-		(stroke
-			(width 0)
-			(type default)
-		)
-	)
-	(wire
-		(pts
-			(xy 130.81 93.98) (xy 158.75 93.98)
-		)
-		(stroke
-			(width 0)
-			(type default)
-		)
-	)
-	(wire
-		(pts
-			(xy 82.55 127) (xy 95.25 127)
-		)
-		(stroke
-			(width 0)
-			(type default)
-		)
-	)
-	(wire
-		(pts
-			(xy 208.28 106.68) (xy 208.28 109.22)
-		)
-		(stroke
-			(width 0)
-			(type default)
-		)
-	)
-	(wire
-		(pts
-			(xy 115.57 133.35) (xy 113.03 133.35)
-		)
-		(stroke
-			(width 0)
-			(type default)
-		)
-	)
-	(wire
-		(pts
-			(xy 130.81 58.42) (xy 134.62 58.42)
-		)
-		(stroke
-			(width 0)
-			(type default)
-		)
-	)
-	(wire
-		(pts
 			(xy 177.8 36.83) (xy 177.8 39.37)
 		)
@@
 	(wire
 		(pts
+			(xy 130.81 63.5) (xy 134.62 63.5)
+		)
+		(stroke
+			(width 0)
+			(type default)
+		)
+	)
+	(wire
+		(pts
 			(xy 87.63 106.68) (xy 95.25 106.68)
 		)
@@
 	(wire
 		(pts
-			(xy 87.63 60.96) (xy 95.25 60.96)
+			(xy 87.63 55.88) (xy 95.25 55.88)
 		)
 		(stroke
@@
 	(wire
 		(pts
-			(xy 87.63 55.88) (xy 95.25 55.88)
-		)
-		(stroke
-			(width 0)
-			(type default)
-		)
-	)
-	(wire
-		(pts
 			(xy 96.52 35.56) (xy 93.98 35.56)
 		)
@@
 	(wire
 		(pts
-			(xy 87.63 58.42) (xy 95.25 58.42)
+			(xy 130.81 66.04) (xy 134.62 66.04)
 		)
 		(stroke
@@
 		(pts
 			(xy 177.8 27.94) (xy 177.8 26.67)
-		)
-		(stroke
-			(width 0)
-			(type default)
-		)
-	)
-	(wire
-		(pts
-			(xy 87.63 50.8) (xy 95.25 50.8)
 		)
 		(stroke
@@
 	(hierarchical_label "PYRO1_FIRE"
 		(shape output)
-		(at 87.63 53.34 180)
-		(effects
-			(font
-				(size 1.27 1.27)
-			)
-			(justify right)
+		(at 134.62 63.5 0)
+		(effects
+			(font
+				(size 1.27 1.27)
+			)
+			(justify left)
 		)
 	)
@@
 	(hierarchical_label "PYRO2_FIRE"
 		(shape output)
-		(at 87.63 60.96 180)
+		(at 87.63 53.34 180)
 		(effects
 			(font
@@
 	(hierarchical_label "PYRO2_PRESENT"
 		(shape output)
-		(at 87.63 63.5 180)
+		(at 87.63 50.8 180)
 		(effects
 			(font
@@
 	(hierarchical_label "PYRO2_ARM"
 		(shape output)
-		(at 87.63 58.42 180)
+		(at 87.63 55.88 180)
 		(effects
 			(font
@@
 	(hierarchical_label "PYRO1_ARM"
 		(shape output)
-		(at 87.63 50.8 180)
-		(effects
-			(font
-				(size 1.27 1.27)
-			)
-			(justify right)
+		(at 134.62 66.04 0)
+		(effects
+			(font
+				(size 1.27 1.27)
+			)
+			(justify left)
 		)
 	)
@@
 	(hierarchical_label "PYRO1_PRESENT"
 		(shape output)
-		(at 87.63 55.88 180)
-		(effects
-			(font
+		(at 87.63 58.42 180)
+		(effects
+			(font

Commit message: final production files
Parts:
- J4: DK Item (none) -> https://www.digikey.com/en/products/detail/molex/0015910100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
- SW1, SW2: DK Part (none) -> https://www.digikey.com/en/products/detail/w%C3%BCrth-elekt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
Changed lines of the file:
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@@
+			)
+		)
+		(property "DK Item" "https://www.digikey.com/en/products/detail/molex/0015910100/614775"
+			(at 30.48 99.06 0)
+			(effects
+				(font
+					(size 1.27 1.27)
+				)
+				(hide yes)
 			)
 		)
@@
 			)
 		)
+		(property "DK Part" "https://www.digikey.com/en/products/detail/w%C3%BCrth-elektronik/434133025816/9950810?s=N4IgTCBcDaIOwEYAMBaALAZjQjGlgFYAOBANhAF0BfIA"
+			(at 198.12 140.97 90)
+			(effects
+				(font
+					(size 1.27 1.27)
+				)
+				(hide yes)
+			)
+		)
 		(pin "1"
 		)
@@
 			(effects
 				(font
+					(size 1.27 1.27)
+				)
+				(hide yes)
+			)
+		)
+		(property "DK Part" "https://www.digikey.com/en/products/detail/w%C3%BCrth-elektronik/434133025816/9950810?s=N4IgTCBcDaIOwEYAMBaALAZjQjGlgFYAOBANhAF0BfIA"
+			(at 34.29 151.13 90)
+			(effects
+				(font

Commit message: oopsies fixed I2C
Connections:
- net BUZZER_CTL: now also U1.20 (PA11); no longer U1.18 (PA09)
- net I2C0_SCL: now also U1.18 (PA09); no longer U1.12 (PB09)
- net I2C0_SDA: now also U1.17 (PA08); no longer U1.11 (PB08)
Other:
- note added: "SERCOM0"
Changed lines of the file:
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@@
 	(text "SERCOM2"
 		(exclude_from_sim no)
-		(at 75.692 83.312 90)
+		(at 71.628 84.328 0)
 		(effects
 			(font
@@
 		)
 	)
+	(text "SERCOM0"
+		(exclude_from_sim no)
+		(at 70.358 72.39 0)
+		(effects
+			(font
+				(size 1.27 1.27)
+			)
+		)
+	)
 	(text "SERCOM3"
 		(exclude_from_sim no)
@@
 	)
 	(no_connect
-		(at 95.25 78.74)
-	)
-	(no_connect
 		(at 95.25 60.96)
 	)
@@
 	)
 	(no_connect
-		(at 95.25 71.12)
+		(at 130.81 73.66)
 	)
 	(no_connect
@@
 	)
 	(no_connect
+		(at 130.81 76.2)
+	)
+	(no_connect
 		(at 95.25 86.36)
 	)
@@
 	(wire
 		(pts
+			(xy 87.63 71.12) (xy 95.25 71.12)
+		)
+		(stroke
+			(width 0)
+			(type default)
+		)
+	)
+	(wire
+		(pts
 			(xy 186.69 106.68) (xy 198.12 106.68)
 		)
@@
 	(wire
 		(pts
+			(xy 87.63 73.66) (xy 95.25 73.66)
+		)
+		(stroke
+			(width 0)
+			(type default)
+		)
+	)
+	(wire
+		(pts
 			(xy 38.1 93.98) (xy 58.42 93.98)
 		)
@@
 	(wire
 		(pts
-			(xy 130.81 73.66) (xy 134.62 73.66)
-		)
-		(stroke
-			(width 0)
-			(type default)
-		)
-	)
-	(wire
-		(pts
 			(xy 22.86 93.98) (xy 25.4 93.98)
 		)
@@
 	(wire
 		(pts
-			(xy 130.81 76.2) (xy 134.62 76.2)
-		)
-		(stroke
-			(width 0)
-			(type default)
-		)
-	)
-	(wire
-		(pts
 			(xy 110.49 40.64) (xy 110.49 35.56)
 		)
@@
 	(wire
 		(pts
+			(xy 87.63 78.74) (xy 95.25 78.74)
+		)
+		(stroke
+			(width 0)
+			(type default)
+		)
+	)
+	(wire
+		(pts
 			(xy 205.74 106.68) (xy 208.28 106.68)
 		)
@@
 		(pts
 			(xy 130.81 66.04) (xy 134.62 66.04)
-		)
-		(stroke
-			(width 0)
-			(type default)
-		)
-	)
-	(wire
-		(pts
-			(xy 87.63 73.66) (xy 95.25 73.66)
 		)
 		(stroke
@@
 	(hierarchical_label "I2C0_SDA"
 		(shape bidirectional)
-		(at 134.62 73.66 0)
-		(effects
-			(font
-				(size 1.27 1.27)
-			)
-			(justify left)
+		(at 87.63 71.12 180)
+		(effects
+			(font
+				(size 1.27 1.27)
+			)
+			(justify right)
 		)
 	)
@@
 	(hierarchical_label "BUZZER_CTL"
 		(shape output)
-		(at 87.63 73.66 180)
+		(at 87.63 78.74 180)
 		(effects
 			(font
@@
 	(hierarchical_label "I2C0_SCL"
 		(shape output)
-		(at 134.62 76.2 0)
-		(effects
-			(font
-				(size 1.27 1.27)
-			)
-			(justify left)
-		)
-	)
+		(at 87.63 73.66 180)
+		(effects
+			(font
+				(size 1.27 1.27)
+			)
+			(justify right)
+		)
+	)
