File: flight-computer-one.kicad_pcb (KiCad board)
At the start: 4 copper layers, 50 x 100 mm, 100 parts, among them J1 Screw_Terminal_01x08, J2 Screw_Terminal_01x08, J3 USB_C_Receptacle_USB2.0_16P, J4 Micro_SD_Card_Det2, J5 GNSS u.FL, J6 COMM u.FL, J7 Conn_01x03_Pin, Q1 CSD17318Q2, Q2 CSD17318Q2, Q3 CSD17318Q2, Q4 CSD17318Q2, Q5 CSD17318Q2, Q6 CSD17318Q2, Q7 CSD17318Q2, SW1 BOOTSEL, SW2 USER, U1 RP2350_80QFN, U10 USBLC6-2SC6, U11 TCAN3404-Q1, U12 INA232, U13 NCV68061, U14 NCV68061, U15 TPS561246, U16 ICM-42688-P, U17 ADS7138-Q1, U2 W25Q32RVXHJQ, U3 MAX-M10S, U4 MCP2518FD-xQBB, U5 BMI088, U6 MS5611-01BA, U7 LIS2MDL, U8 SHT4x, U9 Ai-Thinker-Ra-01H, Y1 ABM8-272-T3, Y2 ASE-40.000MHz

Commit message: schematic + prelim layout nearly complete
Parts:
- added C38: 0.1u, Capacitor_SMD:C_0603_1608Metric, F.Cu at (117.4, 121.7)
- added C39: 0.1u, Capacitor_SMD:C_0603_1608Metric, F.Cu at (100.4, 98.9)
- added C40: 10n, Capacitor_SMD:C_0603_1608Metric, F.Cu at (99.7, 96.7)
- added R20: 10K, Resistor_SMD:R_0603_1608Metric, F.Cu at (138.1, 108.5)
- added R21: 3.32K, Resistor_SMD:R_0603_1608Metric, F.Cu at (135.8, 109.3)
- added R22: 10K, Resistor_SMD:R_0603_1608Metric, F.Cu at (138.1, 118.1)
- added R23: 3.32K, Resistor_SMD:R_0603_1608Metric, F.Cu at (135.8, 119.5)
- added R24: 100K, Resistor_SMD:R_0603_1608Metric, F.Cu at (132.8, 105.8)
- added R25: 100K, Resistor_SMD:R_0603_1608Metric, F.Cu at (132.8, 108.8)
- added R26: 100K, Resistor_SMD:R_0603_1608Metric, F.Cu at (132.8, 116.0)
- added R27: 100K, Resistor_SMD:R_0603_1608Metric, F.Cu at (132.8, 119.0)
- added R28: 10K, Resistor_SMD:R_0603_1608Metric, F.Cu at (150.5, 55.0)
- added R29: 1K, Resistor_SMD:R_0603_1608Metric, F.Cu at (132.8, 104.3)
- added R30: 1K, Resistor_SMD:R_0603_1608Metric, F.Cu at (132.8, 107.3)
- added R31: 1K, Resistor_SMD:R_0603_1608Metric, F.Cu at (132.8, 114.5)
- added R32: 1K, Resistor_SMD:R_0603_1608Metric, F.Cu at (132.8, 117.5)
- added R33: 100, Resistor_SMD:R_0603_1608Metric, F.Cu at (98.9, 94.4)
- added R34: 100, Resistor_SMD:R_0603_1608Metric, F.Cu at (100.5, 94.4)
- J1: value Screw_Terminal_01x08 -> LEFT_BANK
- J2: value Screw_Terminal_01x08 -> RIGHT_BANK
- R16: value R_Shunt -> 10m
- TP1: value TestPoint -> RUN
- Y2: value ASE-40.000MHz -> SG-210STF 40M; footprint Oscillator:Oscillator_SMD_Abracon_ASE-4Pin_3.2x2.5mm -> Crystal:Crystal_SMD_2520-4Pin_2.5x2.0mm
- moved C24 92.2 mm to (163.2, 80.9), turned to 180 degrees
- moved C23 91.3 mm to (163.5, 67.7)
- moved C22 90.9 mm to (162.3, 72.9)
- moved R13 87.1 mm to (163.2, 98.5)
- moved C26 76.7 mm to (148.1, 81.9), turned to 90 degrees
- moved C25 75.5 mm to (146.5, 81.9), turned to 90 degrees
- moved C29 72.4 mm to (144.2, 83.9)
- moved C2 62.0 mm to (142.8, 62.4), turned to 180 degrees
- moved U4 55.9 mm to (110.9, 124.0), turned to 180 degrees
- moved Y2 52.5 mm to (114.9, 121.6), turned to 180 degrees
- moved R3 51.9 mm to (114.9, 57.9)
- moved C11 37.9 mm to (114.9, 52.0)
- moved C8 37.9 mm to (114.9, 49.5)
- moved U11 32.5 mm to (133.2, 124.5), turned to 0 degrees
- moved C10 24.4 mm to (114.8, 54.5)
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Connections:
- net Net-(R4-Pad2) renamed /Compute/USER_BTN
- J1 pad 1: unconnected-(J1-Pin_1-Pad1) -> +PBP
- J1 pad 2: unconnected-(J1-Pin_2-Pad2) -> GND
- J1 pad 3: unconnected-(J1-Pin_3-Pad3) -> +PBP
- J1 pad 4: unconnected-(J1-Pin_4-Pad4) -> GND
- J1 pad 5: unconnected-(J1-Pin_5-Pad5) -> /SERVO1_CTL
- J1 pad 6: unconnected-(J1-Pin_6-Pad6) -> /SERVO2_CTL
- J1 pad 7: unconnected-(J1-Pin_7-Pad7) -> /SERVO3_CTL
- J1 pad 8: unconnected-(J1-Pin_8-Pad8) -> /SERVO4_CTL
- J2 pad 1: unconnected-(J2-Pin_1-Pad1) -> /GPIO40_ADC0
- J2 pad 2: unconnected-(J2-Pin_2-Pad2) -> GND
- J2 pad 3: unconnected-(J2-Pin_3-Pad3) -> /CANL
- J2 pad 4: unconnected-(J2-Pin_4-Pad4) -> /CANH
- J2 pad 5: unconnected-(J2-Pin_5-Pad5) -> /PYRO2_DRAIN
- J2 pad 6: unconnected-(J2-Pin_6-Pad6) -> +PBP
- J2 pad 7: unconnected-(J2-Pin_7-Pad7) -> /PYRO1_DRAIN
- J2 pad 8: unconnected-(J2-Pin_8-Pad8) -> +PBP
- Q1 pad 3: unconnected-(Q1-G-Pad3) -> Net-(Q1-G)
- Q2 pad 3: unconnected-(Q2-G-Pad3) -> Net-(Q2-G)
- Q3 pad 3: unconnected-(Q3-G-Pad3) -> Net-(Q3-G)
- Q4 pad 3: unconnected-(Q4-G-Pad3) -> Net-(Q4-G)
- R16 pad 2: unconnected-(R16-Pad2) -> Net-(R16-Pad2)
- R16 pad 3: unconnected-(R16-Pad3) -> Net-(R16-Pad3)
- U12 pad 1: unconnected-(U12-IN+-Pad1) -> /Power & USB/PMON_IN+
- U12 pad 2: unconnected-(U12-IN--Pad2) -> /Power & USB/PMON_IN-
- U12 pad 5: unconnected-(U12-SCL-Pad5) -> /Power & USB/I2C0_SCL
- U12 pad 6: unconnected-(U12-SDA-Pad6) -> /Power & USB/I2C0_SDA
- U16 pad 1: unconnected-(U16-AP_SDO/AP_AD0-Pad1) -> /Sensors/SPI0_MISO
- U16 pad 12: unconnected-(U16-AP_CS-Pad12) -> /Sensors/CS_IMU_MAIN
- U16 pad 13: unconnected-(U16-AP_SCL/AP_SCLK-Pad13) -> /Sensors/SPI0_SCK
- U16 pad 14: unconnected-(U16-AP_SDA/AP_SDIO/AP_SDI-Pad14) -> /Sensors/SPI0_MOSI
- U16 pad 4: unconnected-(U16-INT1/INT-Pad4) -> /Sensors/IMU_MAIN_INT
- U17 pad 1: unconnected-(U17-AIN2/GPIO2-Pad1) -> /Servos & Pyros/PYRO1_PRSNT
- U17 pad 15: unconnected-(U17-AIN0/GPIO0-Pad15) -> /Servos & Pyros/PYRO1_ARM
- U17 pad 16: unconnected-(U17-AIN1/GPIO1-Pad16) -> /Servos & Pyros/PYRO1_FIRE
- U17 pad 3: unconnected-(U17-AIN4/GPIO4-Pad3) -> /Servos & Pyros/PYRO2_ARM
- U17 pad 4: unconnected-(U17-AIN5/GPIO5-Pad4) -> /Servos & Pyros/PYRO2_FIRE
- U17 pad 5: unconnected-(U17-AIN6/GPIO6-Pad5) -> /Servos & Pyros/PYRO2_PRSNT
- U4 pad 10: unconnected-(U4-SCK-Pad10) -> /Connectivity/CS_CANXC
- U4 pad 11: unconnected-(U4-SDI-Pad11) -> /Connectivity/SPI0_MOSI
- U4 pad 12: unconnected-(U4-SDO-Pad12) -> /Connectivity/SPI0_MISO
- U4 pad 13: unconnected-(U4-~{CS}-Pad13) -> /Connectivity/SPI0_SCK
- U9 pad 12: unconnected-(U9-SCK-Pad12) -> /Connectivity/SPI0_SCK
- U9 pad 13: unconnected-(U9-MISO-Pad13) -> /Connectivity/SPI0_MISO
- U9 pad 14: unconnected-(U9-MOSI-Pad14) -> /Connectivity/SPI0_MOSI
- U9 pad 15: unconnected-(U9-~{NSS}-Pad15) -> /Connectivity/CS_RADIO
- U9 pad 4: unconnected-(U9-~{RESET}-Pad4) -> Net-(U9-~{RESET})

Commit message: Schematic tentatively complete
Parts:
- added C41: 100p, Capacitor_SMD:C_0603_1608Metric, F.Cu at (98.4, 64.5)
- added D1: Green 5mA, LED_SMD:LED_0603_1608Metric, F.Cu at (109.9, 66.9)
- added D2: Red 5mA, LED_SMD:LED_0603_1608Metric, F.Cu at (114.9, 76.9)
- added L2: 3.3uH, Inductor_SMD:L_Murata_DFE201610P, F.Cu at (192.2, 110.1)
- added R35: 59, Resistor_SMD:R_0603_1608Metric, F.Cu at (98.4, 67.0)
- added R36: 59, Resistor_SMD:R_0603_1608Metric, F.Cu at (98.4, 69.5)
- added R37: 634, Resistor_SMD:R_0603_1608Metric, F.Cu at (109.9, 65.4)
- added R38: 634, Resistor_SMD:R_0603_1608Metric, F.Cu at (113.4, 76.9)
- added TP2: 3V3, TestPoint:TestPoint_Pad_D1.0mm, F.Cu at (201.5, 102.6)
- BZ1: value PKLCS1212E -> AST1109; footprint Buzzer_Beeper:Buzzer_Murata_PKLCS1212E -> Buzzer_Beeper:Buzzer_Mallory_AST1109MLTRQ
- C10, C35, C6, C7, C9: footprint Capacitor_SMD:C_0805_2012Metric -> Capacitor_SMD:C_0402_1005Metric
- R3: footprint Resistor_SMD:R_0603_1608Metric -> Resistor_SMD:R_0402_1005Metric
- moved R17 91.9 mm to (197.9, 103.3), turned to 90 degrees
- moved R18 91.3 mm to (197.9, 106.2)
- moved C5 89.8 mm to (194.0, 108.2), turned to -90 degrees
- moved C1 88.1 mm to (175.8, 105.0)
- moved U13 88.1 mm to (180.3, 108.2)
- moved U14 88.1 mm to (180.3, 104.7)
- moved C30 88.1 mm to (189.4, 108.5)
- moved C31 88.1 mm to (177.4, 105.0)
- moved FB1 88.1 mm to (176.6, 107.2)
- moved Q5 88.1 mm to (183.7, 108.0)
- moved Q6 88.1 mm to (183.7, 104.5)
- moved R33 88.1 mm to (185.9, 108.5)
- moved R34 88.1 mm to (187.5, 108.5)
- moved U15 88.1 mm to (192.2, 107.7), turned to 90 degrees
- moved C40 88.1 mm to (186.7, 110.8)
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Connections:
- J1 pad 1: +PBP -> +BATT
- U1 pad 64: +1V1 -> +3V3
- U17 pad 1: /Servos & Pyros/PYRO1_PRSNT -> /Servos & Pyros/PYRO2_FIRE
- U17 pad 15: /Servos & Pyros/PYRO1_ARM -> unconnected-(U17-AIN0/GPIO0-Pad15)
- U17 pad 16: /Servos & Pyros/PYRO1_FIRE -> /Servos & Pyros/PYRO2_PRSNT
- U17 pad 2: unconnected-(U17-AIN3/GPIO3-Pad2) -> /Servos & Pyros/PYRO2_ARM
- U17 pad 3: /Servos & Pyros/PYRO2_ARM -> unconnected-(U17-AIN4/GPIO4-Pad3)
- U17 pad 4: /Servos & Pyros/PYRO2_FIRE -> /Servos & Pyros/PYRO1_PRSNT
- U17 pad 5: /Servos & Pyros/PYRO2_PRSNT -> /Servos & Pyros/PYRO1_FIRE
- U17 pad 6: unconnected-(U17-AIN7/GPIO7-Pad6) -> /Servos & Pyros/PYRO1_ARM

Commit message: schematic tentatively finished
Parts:
- moved C41 70.8 mm to (137.8, 123.3), turned to 180 degrees
- moved D1 66.7 mm to (176.5, 71.2)
- moved R37 66.7 mm to (176.5, 69.7)
- moved R36 66.5 mm to (135.4, 124.8), turned to -90 degrees
- moved R35 66.1 mm to (135.4, 121.8), turned to -90 degrees
- moved R12 31.4 mm to (100.5, 87.2), turned to 0 degrees
- moved R11 28.4 mm to (100.5, 84.7), turned to 0 degrees
- moved U11 3.22 mm to (131.2, 123.4)
Connections:
- net /Servos & Pyros/BUZZER renamed /Servos & Pyros/BUZZER_CTL
- net Net-(U11-RXD) renamed /Connectivity/TXCAN
- net Net-(U11-TXD) renamed /Connectivity/RXCAN
- net Net-(U9-~{RESET}) renamed /Connectivity/RADIO_nRST
- R11 pad 2: /Sensors/I2C0_SCL -> /Compute/I2C0_SDA
- R12 pad 2: /Sensors/I2C0_SDA -> /Compute/I2C0_SCL
- R35 pad 1: /Connectivity/CANH -> /CANH
- R36 pad 2: /Connectivity/CANL -> /CANL
- U10 pad 4: /Power & USB/USB_D+ -> /Compute/USB_D+
- U10 pad 6: /Power & USB/USB_D- -> /Compute/USB_D-
- U11 pad 6: /Connectivity/CANL -> /CANL
- U11 pad 7: /Connectivity/CANH -> /CANH
- U12 pad 5: /Power & USB/I2C0_SCL -> /Compute/I2C0_SCL
- U12 pad 6: /Power & USB/I2C0_SDA -> /Compute/I2C0_SDA
- U17 pad 13: /Servos & Pyros/I2C0_SCL -> /Compute/I2C0_SCL
- U17 pad 14: /Servos & Pyros/I2C0_SDA -> /Compute/I2C0_SDA
- U3 pad 16: /Connectivity/I2C0_SDA -> /Compute/I2C0_SDA
- U3 pad 17: /Connectivity/I2C0_SCL -> /Compute/I2C0_SCL
- U5 pad 8: /Sensors/I2C0_SCL -> /Compute/I2C0_SCL
- U5 pad 9: /Sensors/I2C0_SDA -> /Compute/I2C0_SDA
- U6 pad 7: /Sensors/I2C0_SDA -> /Compute/I2C0_SDA
- U6 pad 8: /Sensors/I2C0_SCL -> /Compute/I2C0_SCL
- U7 pad 1: /Sensors/I2C0_SCL -> /Compute/I2C0_SCL
- U7 pad 4: /Sensors/I2C0_SDA -> /Compute/I2C0_SDA
- U8 pad 1: /Sensors/I2C0_SDA -> /Compute/I2C0_SDA
- U8 pad 2: /Sensors/I2C0_SCL -> /Compute/I2C0_SCL
