File: flight-computer-one.kicad_pcb (KiCad board)
At the start: 4 copper layers, 50 x 100 mm, 127 parts, among them J1 LEFT_BANK, J2 RIGHT_BANK, J3 USB_C_Receptacle_USB2.0_16P, J4 Micro_SD_Card_Det2, J5 GNSS u.FL, J6 COMM u.FL, J7 Conn_01x03_Pin, Q1 CSD17318Q2, Q2 CSD17318Q2, Q3 CSD17318Q2, Q4 CSD17318Q2, Q5 CSD17318Q2, Q6 CSD17318Q2, Q7 CSD17318Q2, SW1 BOOTSEL, SW2 USER, U1 RP2350_80QFN, U10 USBLC6-2SC6, U11 TCAN3404-Q1, U12 INA232, U13 NCV68061, U14 NCV68061, U15 TPS561246, U16 ICM-42688-P, U17 ADS7138-Q1, U2 W25Q32RVXHJQ, U3 MAX-M10S, U4 MCP2518FD-xQBB, U5 BMI088, U6 MS5611-01BA, U7 LIS2MDL, U8 SHT4x, U9 Ai-Thinker-Ra-01H, Y1 ABM8-272-T3, Y2 SG-210STF 40M

Commit message: swapped POR chip for TPS2121
Parts:
- removed Q5, Q6: CSD17318Q2, Package_SON:Texas_DQK
- removed U13, U14: NCV68061, Package_TO_SOT_SMD:SOT-23-6
- added C42: 0.1u, Capacitor_SMD:C_0603_1608Metric, F.Cu at (124.5, 68.2)
- added C43: 0.1u, Capacitor_SMD:C_0603_1608Metric, F.Cu at (128.0, 123.3)
- added C44: 10n, Capacitor_SMD:C_0603_1608Metric, F.Cu at (159.0, 105.7)
- added R39: 100K, Capacitor_SMD:C_0603_1608Metric, F.Cu at (157.4, 105.7)
- added U18: TPS2121, Package_DFN_QFN:Texas_VQFN-HR-12_2x2.5mm_P0.5mm_ThermalVias, F.Cu at (158.2, 102.4)
- moved TP2 46.7 mm to (158.0, 119.6), turned to 90 degrees
- moved C31 43.4 mm to (153.8, 68.5), turned to 0 degrees
- moved FB1 43.1 mm to (156.1, 69.3), turned to 90 degrees
- moved R38 41.5 mm to (154.8, 74.2)
- moved C1 41.2 mm to (153.8, 70.1), turned to 0 degrees
- moved C19 38.6 mm to (156.9, 117.2)
- moved D2 38.4 mm to (153.2, 74.2)
- moved R18 38.2 mm to (160.1, 112.0), turned to 180 degrees
- moved L2 36.2 mm to (156.3, 114.8)
- moved R17 35.7 mm to (163.3, 112.0), turned to 0 degrees
- moved C5 34.2 mm to (160.8, 116.3)
- moved U15 34.1 mm to (158.7, 114.1), turned to 0 degrees
- moved C30 33.0 mm to (156.6, 112.0), turned to 180 degrees
- moved R16 30.0 mm to (157.0, 109.2), turned to 0 degrees
- moved R19 29.6 mm to (161.5, 113.9), turned to 180 degrees
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Connections:
- net /Connectivity/CS_CANXC renamed /Compute/CS_CANXC
- net /Connectivity/CS_RADIO renamed /Compute/CS_RADIO
- net /Connectivity/TCAN_STB renamed /Compute/TCAN_STB
- net /Sensors/CS_IMU_MAIN renamed /Compute/CS_IMU_MAIN
- net /Servos & Pyros/BUZZER_CTL renamed /Compute/BUZZER_CTL
- net Net-(U15-EN) renamed /Power & USB/TPS_EN
- U1 pad 42: /Compute/GPIO33 -> /Compute/USER_LED
- U1 pad 45: /Compute/GPIO36 -> /SERVO1_CTL
- U1 pad 46: /Compute/GPIO37 -> /SERVO2_CTL
- U1 pad 47: /Compute/GPIO38 -> /SERVO3_CTL
- U1 pad 48: /Compute/GPIO39 -> /SERVO4_CTL
- U1 pad 49: /Compute/GPIO40_ADC0 -> /GPIO40_ADC0
- U16 pad 1: /Sensors/SPI0_MISO -> /Compute/SPI0_MISO
- U16 pad 13: /Sensors/SPI0_SCK -> /Compute/SPI0_SCK
- U16 pad 14: /Sensors/SPI0_MOSI -> /Compute/SPI0_MOSI
- U4 pad 11: /Connectivity/SPI0_MOSI -> /Compute/SPI0_MOSI
- U4 pad 12: /Connectivity/SPI0_MISO -> /Compute/SPI0_MISO
- U4 pad 13: /Connectivity/SPI0_SCK -> /Compute/SPI0_SCK
- U9 pad 12: /Connectivity/SPI0_SCK -> /Compute/SPI0_SCK
- U9 pad 13: /Connectivity/SPI0_MISO -> /Compute/SPI0_MISO
- U9 pad 14: /Connectivity/SPI0_MOSI -> /Compute/SPI0_MOSI
Routing:
- net /SERVO4_CTL: track 0.00 -> 37.9 mm
- net /GPIO40_ADC0: track 0.00 -> 37.1 mm
- net GND: track 0.00 -> 37.0 mm, vias 0 -> 25
- net /SERVO3_CTL: track 0.00 -> 32.8 mm
- net /SERVO2_CTL: track 0.00 -> 27.7 mm
- net +PBP: track 0.00 -> 24.6 mm, vias 0 -> 1
- net /SERVO1_CTL: track 0.00 -> 22.4 mm
- net /Connectivity/TXCAN: track 0.00 -> 21.6 mm, vias 0 -> 1
- net /Servos & Pyros/PYRO2_PRSNT: track 0.00 -> 17.8 mm
- net /Compute/I2C0_SCL: track 0.00 -> 16.9 mm
- net /Compute/I2C0_SDA: track 0.00 -> 16.5 mm
- net /Servos & Pyros/PYRO2_ARM: track 0.00 -> 15.6 mm
- net /Servos & Pyros/PYRO2_FIRE: track 0.00 -> 13.3 mm
- net /Servos & Pyros/PYRO1_ARM: track 0.00 -> 12.8 mm
- net /Connectivity/RXCAN: track 0.00 -> 10.7 mm, vias 0 -> 1
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- added copper zone on In2.Cu, net +3V3
- removed copper zone on In2.Cu, net GND
Other:
- rule pad_to_mask_clearance: 0 -> 0.0762

Commit message: added pictures to readme
Parts:
- C40: value 10n -> 0.1u
Changed lines of the file:
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@@
 			)
 		)
-		(property "Value" "10n"
+		(property "Value" "0.1u"
 			(at 0 1.43 90)
 			(layer "F.Fab")

Commit message: preliminary change to SAME51
Parts:
- removed TP1: RUN, TestPoint:TestPoint_Pad_D1.0mm
- added D3: Red 5mA, LED_SMD:LED_0603_1608Metric, F.Cu at (160.5, 120.5)
- added R40: 634, Resistor_SMD:R_0603_1608Metric, F.Cu at (162.1, 120.5)
- C6, C7: footprint Capacitor_SMD:C_0402_1005Metric -> Capacitor_SMD:C_0603_1608Metric
- D1: value Green 5mA -> Red 5mA
- D2: value Red 5mA -> Green 5mA
- R7, R8: footprint Resistor_SMD:R_0603_1608Metric -> Resistor_SMD:R_0402_1005Metric
- moved C10 63.6 mm to (147.0, 81.2), turned to -90 degrees
- moved C11 63.2 mm to (152.9, 73.0)
- moved C12 57.2 mm to (141.1, 67.3), turned to 180 degrees
- moved R3 52.8 mm to (151.5, 64.3), turned to -90 degrees
- moved C6 48.7 mm to (149.1, 67.3)
- moved L1 48.5 mm to (149.2, 64.0)
- moved C9 47.8 mm to (151.5, 66.5), turned to -90 degrees
- moved C7 46.4 mm to (149.1, 65.8)
- moved R12 29.4 mm to (129.8, 85.4), turned to 90 degrees
- moved R11 27.7 mm to (128.2, 85.4), turned to 90 degrees
- moved R37 16.7 mm to (159.9, 78.8), turned to 180 degrees
- moved J7 15.2 mm to (148.5, 89.0), turned to 180 degrees
- moved D1 15.1 mm to (159.9, 77.2), turned to 180 degrees
- moved R10 9.07 mm to (149.3, 84.5), turned to 90 degrees
- moved R9 8.88 mm to (147.7, 84.5), turned to 90 degrees
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Connections:
- Q1 pad 1: /Servos & Pyros/PYRO1_DRAIN -> /PYRO1_DRAIN
- Q1 pad 2: /Servos & Pyros/PYRO1_DRAIN -> /PYRO1_DRAIN
- Q1 pad 5: /Servos & Pyros/PYRO1_DRAIN -> /PYRO1_DRAIN
- Q1 pad 6: /Servos & Pyros/PYRO1_DRAIN -> /PYRO1_DRAIN
- Q1 pad 8: /Servos & Pyros/PYRO1_DRAIN -> /PYRO1_DRAIN
- Q3 pad 1: /Servos & Pyros/PYRO2_DRAIN -> /PYRO2_DRAIN
- Q3 pad 2: /Servos & Pyros/PYRO2_DRAIN -> /PYRO2_DRAIN
- Q3 pad 5: /Servos & Pyros/PYRO2_DRAIN -> /PYRO2_DRAIN
- Q3 pad 6: /Servos & Pyros/PYRO2_DRAIN -> /PYRO2_DRAIN
- Q3 pad 8: /Servos & Pyros/PYRO2_DRAIN -> /PYRO2_DRAIN
Routing:
- net /Connectivity/RXCAN: track 10.7 -> 53.2 mm, vias 1 -> 2
- net /Connectivity/TXCAN: track 21.6 -> 58.2 mm, vias 1 -> 2
- net /GPIO40_ADC0: track 37.1 -> 69.8 mm, vias 0 -> 1
- net /SERVO4_CTL: track 37.9 -> 66.7 mm, vias 0 -> 1
- net /SERVO3_CTL: track 32.8 -> 60.4 mm, vias 0 -> 1
- net /SERVO2_CTL: track 27.7 -> 54.2 mm, vias 0 -> 1
- net /SERVO1_CTL: track 22.4 -> 48.1 mm, vias 0 -> 1
- net +3V3: track 7.89 -> 33.2 mm, vias 1 -> 20
- net /Compute/SPI0_MOSI: track 0.00 -> 17.3 mm, vias 0 -> 3
- net GND: track 37.0 -> 53.9 mm, vias 25 -> 60
- net /Compute/SPI0_SCK: track 0.00 -> 16.9 mm, vias 0 -> 4
- net /Compute/SPI0_MISO: track 0.00 -> 16.1 mm, vias 0 -> 3
- net /Compute/CS_CANXC: track 0.00 -> 14.8 mm, vias 0 -> 2
- net /Connectivity/ANT_GNSS: track 0.00 -> 10.8 mm
- net /Compute/QSPI_SS: track 0.00 -> 10.1 mm
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- added copper zone on F.Cu, net +3V3
- added copper zone on F.Cu, net /Power & USB/TPS_SW
Other:
- board text added: "3V3"
- board text added: "5V0"
- board text added: "USR"

Commit message: same51 wired, near completion
Parts:
- removed the C17 at (84.9, 68.8)
- removed the C18 at (84.9, 71.3)
- removed the C2 at (142.9, 62.0)
- removed the C20 at (84.9, 73.7)
- removed the C21 at (84.9, 76.2)
- removed the C3 at (140.8, 81.8)
- removed C38, C42, C43: 0.1u, Capacitor_SMD:C_0603_1608Metric
- removed the C4 at (143.2, 85.3)
- removed the C6 at (149.1, 67.3)
- removed the C7 at (149.1, 65.8)
- removed the C8 at (108.2, 25.9)
- removed the J7 at (148.5, 89.0)
- removed the L1 at (149.2, 64.0)
- removed the R10 at (149.3, 84.5)
- removed the R2 at (145.8, 81.8)
- removed the R3 at (151.5, 64.3)
- removed the R7 at (145.8, 64.6)
- removed the R8 at (146.9, 64.6)
- removed the U2 at (142.3, 64.0)
- removed the U4 at (126.5, 71.4)
- removed Y2: SG-210STF 40M, Crystal:Crystal_SMD_2520-4Pin_2.5x2.0mm
- added G***: LOGO, LRI_partlib:gnd-symbol, B.Cu at (133.9, 130.5)
- added J4: SWD, Connector_PinHeader_1.27mm:PinHeader_2x05_P1.27mm_Vertical_SMD, F.Cu at (145.1, 57.6)
- C10, C9: value 4.7u -> 0.1u; footprint Capacitor_SMD:C_0402_1005Metric -> Capacitor_SMD:C_0603_1608Metric
- C11: value 0.1u -> 10u
- C20: renamed from C35; footprint Capacitor_SMD:C_0402_1005Metric -> Capacitor_SMD:C_0603_1608Metric
- R14: renamed from R9; value 100 -> 1K
- R15: renamed from R1; value 1K -> 10K
- SW1: value BOOTSEL -> RESET
- U1: value RP2350_80QFN -> ATSAME51J19A-M; footprint Package_DFN_QFN:QFN-80-1EP_10x10mm_P0.4mm_EP3.4x3.4mm_ThermalVias -> Package_DFN_QFN:QFN-64-1EP_9x9mm_P0.5mm_EP4.7x4.7mm
- U10: renamed from U8; value SHT4x -> SHT40
- Y1: value ABM8-272-T3 -> SiT8008BI-11-33N-20.000000; footprint Crystal:Crystal_SMD_3225-4Pin_3.2x2.5mm -> Oscillator:Oscillator_SMD_SiT_PQFN-4Pin_2.5x2.0mm
- moved C13 69.0 mm to (151.5, 77.0), turned to -90 degrees
- moved C14 67.7 mm to (152.1, 69.3)
- moved C16 60.4 mm to (143.7, 80.0), turned to -90 degrees
- moved C15 54.7 mm to (138.8, 73.0), turned to 180 degrees
- moved SW2 36.3 mm to (146.2, 89.9), turned to 180 degrees
- moved R17 31.9 mm to (149.9, 89.6), turned to 90 degrees
- moved C10 22.7 mm to (152.8, 59.2), turned to 0 degrees
- moved R14 22.7 mm to (143.1, 62.3), turned to 180 degrees
- moved C9 16.5 mm to (149.6, 82.9), turned to 0 degrees
- moved U8 9.93 mm to (140.6, 84.2)
- moved C23 9.93 mm to (142.9, 84.0)
- moved C24 9.93 mm to (138.4, 84.0)
- moved C25 9.93 mm to (140.4, 87.8)
- moved C26 9.93 mm to (140.4, 86.2)
- moved SW1 8.66 mm to (153.1, 55.5), turned to -90 degrees
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- renumbered C44 to C1, C24 to C17, C22 to C18, C23 to C19, C1 to C2, C36 to C21, C37 to C22, C27 to C23, C29 to C24, C26 to C25, C25 to C26, C28 to C27, C41 to C28, C32 to C29, C31 to C3, C33 to C30, C34 to C31, C30 to C4, C40 to C5, C5 to C6, C39 to C7, C19 to C8, D3 to D2, D2 to D3, J4 to J5, J5 to J7, L2 to L1, Q7 to Q5, R11 to R1, R33 to R10, R34 to R11, R17 to R12, R18 to R13, R13 to R16, R4 to R17, R38 to R18, R28 to R19, R12 to R2, R35 to R20, R36 to R21, R29 to R22, R30 to R23, R31 to R24, R32 to R25, R24 to R26, R26 to R27, R25 to R28, R27 to R29, R6 to R3, R20 to R30, R22 to R31, R21 to R32, R23 to R33, R15 to R34, R14 to R35, R5 to R4, R39 to R5, R37 to R6, R40 to R7, R16 to R8, R19 to R9, TP2 to TP1, U9 to U12, U3 to U13, U17 to U14, U10 to U2, U18 to U3, U15 to U4, U12 to U5, U5 to U6, U6 to U7, U7 to U8, U16 to U9
Connections:
- net Net-(J3-CC1) renamed /Power & USB/USB_CC1
- net Net-(J3-CC2) renamed /Power & USB/USB_CC2
- C10 pad 1: +1V1 -> /Compute/~{RESET}
- C11 pad 1: +1V1 -> GND
- C11 pad 2: GND -> Net-(U1-VDDCORE)
- C9 pad 1: /Compute/VREG_AVDD -> +3V3
- R14 pad 1: /Compute/SWCLK -> +3V3
- R14 pad 2: Net-(U1-SWCLK) -> /Compute/SWCLK
- R15 pad 1: /Compute/QSPI_SS -> +3V3
- R15 pad 2: /Compute/~{USB_BOOT} -> /Compute/~{RESET}
- SW1 pad 2: /Compute/~{USB_BOOT} -> /Compute/~{RESET}
- U1 pad 1: /Compute/GPIO4 -> unconnected-(U1-PA00-Pad1)
- U1 pad 10: +1V1 -> unconnected-(U1-PB07-Pad10)
- U1 pad 11: /Compute/GPIO12 -> unconnected-(U1-PB08-Pad11)
- U1 pad 12: /Compute/GPIO13 -> unconnected-(U1-PB09-Pad12)
- U1 pad 13: /Compute/GPIO14 -> unconnected-(U1-PA04-Pad13)
- U1 pad 14: /Compute/GPIO15 -> unconnected-(U1-PA05-Pad14)
- U1 pad 15: +3V3 -> unconnected-(U1-PA06-Pad15)
- U1 pad 16: /Compute/GPIO16 -> unconnected-(U1-PA07-Pad16)
- U1 pad 17: /Compute/GPIO17 -> unconnected-(U1-PA08-Pad17)
- U1 pad 18: /Compute/GPIO18 -> /Compute/BUZZER_CTL
- U1 pad 19: /Compute/GPIO19 -> /GPIO40_ADC0
- U1 pad 2: /Compute/GPIO5 -> unconnected-(U1-PA01-Pad2)
- U1 pad 20: /Compute/GPIO20 -> unconnected-(U1-PA11-Pad20)
- U1 pad 21: /Compute/GPIO21 -> +3V3
- U1 pad 22: /Compute/GPIO22 -> GND
- U1 pad 23: /Compute/GPIO23 -> unconnected-(U1-PB10-Pad23)
- U1 pad 24: +3V3 -> /Compute/USER_BTN
- U1 pad 25: /Compute/GPIO24 -> /SERVO4_CTL
- U1 pad 26: /Compute/GPIO25 -> /SERVO3_CTL
- U1 pad 27: /Compute/GPIO26 -> /SERVO2_CTL
- U1 pad 28: /Compute/GPIO27 -> /SERVO1_CTL
- U1 pad 29: +3V3 -> unconnected-(U1-PA12-Pad29)
- U1 pad 3: /Compute/GPIO6 -> unconnected-(U1-PA02-Pad3)
- U1 pad 30: /Compute/XIN -> unconnected-(U1-PA13-Pad30)
- U1 pad 31: /Compute/XOUT -> /Compute/XIN
- U1 pad 32: +1V1 -> /Compute/XOUT
- U1 pad 33: Net-(U1-SWCLK) -> GND
- U1 pad 34: Net-(U1-SWD) -> +3V3
- U1 pad 35: /Compute/RUN -> /Compute/DAT0/MISO
- U1 pad 36: /Compute/GPIO28 -> /Compute/SD_CLK
- U1 pad 37: /Compute/GPIO29 -> /Compute/DAT3/CS
- U1 pad 38: /Compute/GPIO30 -> /Compute/CMD/MOSI
- U1 pad 39: /Compute/GPIO31 -> /Compute/USER_LED
- U1 pad 4: /Compute/GPIO7 -> unconnected-(U1-PA03-Pad4)
- U1 pad 40: /Compute/GPIO32 -> /Compute/CARD_DET
- U1 pad 41: +3V3 -> unconnected-(U1-PA20-Pad41)
- U1 pad 42: /Compute/USER_LED -> unconnected-(U1-PA21-Pad42)
- U1 pad 43: /Compute/GPIO34 -> /Compute/TXCAN
- U1 pad 44: /Compute/GPIO35 -> /Compute/RXCAN
- U1 pad 45: /SERVO1_CTL -> /Compute/USB_D-
- U1 pad 46: /SERVO2_CTL -> /Compute/USB_D+
- U1 pad 47: /SERVO3_CTL -> GND
- U1 pad 48: /SERVO4_CTL -> +3V3
- U1 pad 49: /GPIO40_ADC0 -> unconnected-(U1-PB22-Pad49)
- U1 pad 5: +3V3 -> unconnected-(U1-PB04-Pad5)
- U1 pad 50: +3V3 -> unconnected-(U1-PB23-Pad50)
- U1 pad 51: +1V1 -> unconnected-(U1-PA27-Pad51)
- U1 pad 52: /Compute/GPIO41_ADC1 -> /Compute/~{RESET}
- U1 pad 53: /Compute/GPIO42_ADC2 -> Net-(U1-VDDCORE)
- U1 pad 54: /Compute/GPIO43_ADC3 -> GND
- U1 pad 55: /Compute/GPIO44_ADC4 -> unconnected-(U1-VSW-Pad55)
- U1 pad 56: /Compute/GPIO45_ADC5 -> +3V3
- U1 pad 57: /Compute/GPIO46_ADC6 -> /Compute/SWCLK
- U1 pad 58: /Compute/GPIO47_ADC7 -> /Compute/SWDIO
- U1 pad 59: +3V3 -> /Compute/SWO
- U1 pad 6: /Compute/GPIO8 -> unconnected-(U1-PB05-Pad6)
- U1 pad 60: +3V3 -> unconnected-(U1-PB31-Pad60)
- U1 pad 61: /Compute/VREG_AVDD -> unconnected-(U1-PB00-Pad61)
- U1 pad 62: GND -> unconnected-(U1-PB01-Pad62)
- U1 pad 63: /Compute/VREG_LX -> unconnected-(U1-PB02-Pad63)
- U1 pad 64: +3V3 -> unconnected-(U1-PB03-Pad64)
- U1 pad 65: +1V1 -> GND
- U1 pad 7: /Compute/GPIO9 -> GND
- U1 pad 8: /Compute/GPIO10 -> +3V3
- U1 pad 9: /Compute/GPIO11 -> unconnected-(U1-PB06-Pad9)
- U11 pad 1: /Connectivity/RXCAN -> /Compute/RXCAN
- U11 pad 4: /Connectivity/TXCAN -> /Compute/TXCAN
- Y1 pad 1: /Compute/XIN -> unconnected-(Y1-NC-Pad1)
- Y1 pad 3: Net-(C4-Pad1) -> /Compute/XIN
- Y1 pad 4: GND -> +3V3
Routing:
- net /Compute/TXCAN: track 0.00 -> 76.6 mm, vias 0 -> 2
- net /Compute/RXCAN: track 0.00 -> 72.6 mm, vias 0 -> 2
- net /Compute/TCAN_STB: track 0.00 -> 64.7 mm, vias 0 -> 2
- net /Connectivity/TXCAN: track 58.2 -> 0.00 mm, vias 2 -> 0
- net /Connectivity/RXCAN: track 53.2 -> 0.00 mm, vias 2 -> 0
- net /Compute/CARD_DET: track 1.87 -> 36.0 mm
- net +3V3: track 33.2 -> 65.3 mm, vias 20 -> 37
- net VBUS: track 0.00 -> 31.7 mm, vias 0 -> 1
- net /Compute/DAT0/MISO: track 0.00 -> 22.2 mm
- net /Compute/BUZZER_CTL: track 0.00 -> 21.1 mm
- net /Compute/SD_CLK: track 0.00 -> 21.0 mm
- net /Compute/CMD/MOSI: track 0.00 -> 20.0 mm
- net /Compute/~{RESET}: track 0.00 -> 18.7 mm
- net /Compute/DAT3/CS: track 0.00 -> 18.2 mm
- net /Compute/I2C0_SCL: track 10.2 -> 27.8 mm
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- added copper zone on F.Cu, net +PBP
Other:
- board text added: "+"
- board text added: "-"
- board text added: "1"
- board text added: "2"
- board text added: "3"
- board text added: "4"
- board text added: "AA CTL"
- board text added: "ADC"
- board text added: "BATT IN"
- board text added: "CAN FD"
- board text added: "D"
- board text added: "EXT PWR"
- board text added: "H"
- board text added: "L"
- board text added: "PYRO 1"
- board text added: "PYRO 2"

Commit message: completed layout for Rev.A
Parts:
- added REF**: ESD-Logo_6.6x6mm_SilkScreen, Symbol:ESD-Logo_6.6x6mm_SilkScreen, F.Cu at (146.5, 48.7)
- moved C27 2.41 mm to (125.3, 76.5)
- moved U10 2.41 mm to (125.3, 78.5)
Connections:
- U1 pad 1: unconnected-(U1-PA00-Pad1) -> /Compute/CS_RADIO
- U1 pad 11: unconnected-(U1-PB08-Pad11) -> /Compute/I2C0_SCL
- U1 pad 12: unconnected-(U1-PB09-Pad12) -> /Compute/I2C0_SDA
- U1 pad 15: unconnected-(U1-PA06-Pad15) -> /Compute/TCAN_STB
- U1 pad 61: unconnected-(U1-PB00-Pad61) -> /Compute/CS_IMU_MAIN
- U1 pad 62: unconnected-(U1-PB01-Pad62) -> /Compute/SPI0_MISO
- U1 pad 63: unconnected-(U1-PB02-Pad63) -> /Compute/SPI0_MOSI
- U1 pad 64: unconnected-(U1-PB03-Pad64) -> /Compute/SPI0_SCK
Routing:
- net /Compute/I2C0_SDA: track 25.7 -> 126.8 mm, vias 0 -> 5
- net /Compute/I2C0_SCL: track 27.8 -> 128.8 mm, vias 0 -> 2
- net /Compute/SPI0_MISO: track 6.23 -> 23.2 mm
- net /Compute/SPI0_SCK: track 0.25 -> 16.5 mm, vias 0 -> 3
- net /Compute/SPI0_MOSI: track 6.89 -> 20.6 mm
- net /Compute/CS_IMU_MAIN: track 0.00 -> 13.4 mm, vias 0 -> 2
- net GND: track 53.4 -> 66.6 mm, vias 72 -> 191
- net /Compute/CS_RADIO: track 0.00 -> 7.95 mm
- net +3V3: track 65.3 -> 67.9 mm, vias 37 -> 40
- net /Compute/TCAN_STB: track 64.7 -> 63.2 mm
- net VBUS: vias 1 -> 2

Commit message: new routing
Parts:
- removed C29, C30, C31: 1u, Capacitor_SMD:C_0603_1608Metric
- removed C9: 0.1u, Capacitor_SMD:C_0603_1608Metric
- removed U14: ADS7138-Q1, Package_DFN_QFN:WQFN-16-1EP_3x3mm_P0.5mm_EP1.68x1.68mm_ThermalVias
- removed Y1: SiT8008BI-11-33N-20.000000, Oscillator:Oscillator_SMD_SiT_PQFN-4Pin_2.5x2.0mm
- added R36: 1K, Resistor_SMD:R_0603_1608Metric, F.Cu at (167.6, 103.7)
- added R37: 1K, Resistor_SMD:R_0603_1608Metric, F.Cu at (164.2, 103.7)
- moved U7 11.3 mm to (134.7, 85.5), turned to 90 degrees
- moved C17 9.00 mm to (134.7, 88.1), turned to 180 degrees
- moved C19 8.10 mm to (125.5, 86.4), turned to -90 degrees
- moved SW2 6.42 mm to (146.8, 83.5), turned to -90 degrees
- moved R34 6.32 mm to (144.8, 90.3), turned to -90 degrees
- moved C27 5.70 mm to (127.9, 81.5), turned to -90 degrees
- moved U10 5.50 mm to (129.9, 81.5), turned to 180 degrees
- moved U6 4.88 mm to (128.1, 86.6), turned to 90 degrees
- moved R35 4.17 mm to (142.4, 89.7), turned to 180 degrees
- moved R17 4.11 mm to (146.6, 87.2), turned to 180 degrees
- moved C18 3.11 mm to (130.7, 86.9), turned to 90 degrees
- moved C21 3.01 mm to (128.8, 72.3)
- moved C20 3.01 mm to (133.1, 69.5)
- moved C22 3.01 mm to (131.6, 69.5)
- moved U9 3.01 mm to (128.5, 69.5)
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Connections:
- net /Compute/CS_IMU_MAIN renamed /Compute/CS_ICM
- J5 pad 1: /Compute/DAT2 -> unconnected-(J5-DAT2-Pad1)
- J5 pad 2: /Compute/DAT3/CS -> /Compute/SD_CS
- J5 pad 3: /Compute/CMD/MOSI -> /Compute/SD_MOSI
- J5 pad 5: /Compute/SD_CLK -> /Compute/SD_SCK
- J5 pad 7: /Compute/DAT0/MISO -> /Compute/SD_MISO
- J5 pad 8: /Compute/DAT1 -> unconnected-(J5-DAT1-Pad8)
- R22 pad 1: /Servos & Pyros/PYRO1_ARM -> /Compute/PYRO1_ARM
- R23 pad 1: /Servos & Pyros/PYRO1_FIRE -> /Compute/PYRO1_FIRE
- R24 pad 1: /Servos & Pyros/PYRO2_ARM -> /Compute/PYRO2_ARM
- R25 pad 1: /Servos & Pyros/PYRO2_FIRE -> /Compute/PYRO2_FIRE
- R30 pad 2: /Servos & Pyros/PYRO1_PRSNT -> /Compute/PYRO1_PRESENT
- R31 pad 2: /Servos & Pyros/PYRO2_PRSNT -> /Compute/PYRO2_PRESENT
- R32 pad 1: /Servos & Pyros/PYRO1_PRSNT -> /Compute/PYRO1_PRESENT
- R33 pad 1: /Servos & Pyros/PYRO2_PRSNT -> /Compute/PYRO2_PRESENT
- U1 pad 1: /Compute/CS_RADIO -> /Compute/PYRO2_PRESENT
- U1 pad 11: /Compute/I2C0_SCL -> /Compute/I2C0_SDA
- U1 pad 12: /Compute/I2C0_SDA -> /Compute/I2C0_SCL
- U1 pad 2: unconnected-(U1-PA01-Pad2) -> /Compute/PYRO2_FIRE
- U1 pad 29: unconnected-(U1-PA12-Pad29) -> /Compute/I2C1_SDA
- U1 pad 3: unconnected-(U1-PA02-Pad3) -> /Compute/PYRO2_ARM
- U1 pad 30: unconnected-(U1-PA13-Pad30) -> /Compute/I2C1_SCL
- U1 pad 31: /Compute/XIN -> unconnected-(U1-PA14-Pad31)
- U1 pad 32: /Compute/XOUT -> unconnected-(U1-PA15-Pad32)
- U1 pad 35: /Compute/DAT0/MISO -> /Compute/SD_SCK
- U1 pad 36: /Compute/SD_CLK -> /Compute/SD_MOSI
- U1 pad 37: /Compute/DAT3/CS -> /Compute/SD_MISO
- U1 pad 38: /Compute/CMD/MOSI -> /Compute/SD_CS
- U1 pad 4: unconnected-(U1-PA03-Pad4) -> /Compute/PYRO1_PRESENT
- U1 pad 5: unconnected-(U1-PB04-Pad5) -> /Compute/PYRO1_FIRE
- U1 pad 6: unconnected-(U1-PB05-Pad6) -> /Compute/PYRO1_ARM
- U1 pad 60: unconnected-(U1-PB31-Pad60) -> /Compute/CS_RADIO
- U13 pad 16: /Compute/I2C0_SDA -> /Compute/I2C1_SDA
- U13 pad 17: /Compute/I2C0_SCL -> /Compute/I2C1_SCL
- U5 pad 5: /Compute/I2C0_SCL -> /Compute/I2C1_SCL
- U5 pad 6: /Compute/I2C0_SDA -> /Compute/I2C1_SDA
Routing:
- net /Compute/I2C0_SCL: track 128.8 -> 29.6 mm
- net /Compute/I2C0_SDA: track 126.8 -> 30.9 mm, vias 5 -> 2
- net /Compute/PYRO2_PRESENT: track 0.00 -> 67.4 mm, vias 0 -> 2
- net /Compute/I2C1_SDA: track 0.00 -> 66.9 mm, vias 0 -> 4
- net /Compute/I2C1_SCL: track 0.00 -> 65.6 mm, vias 0 -> 4
- net /Compute/PYRO2_ARM: track 0.00 -> 61.9 mm, vias 0 -> 2
- net /Compute/PYRO2_FIRE: track 0.00 -> 61.8 mm, vias 0 -> 2
- net /Compute/PYRO1_PRESENT: track 0.00 -> 54.3 mm, vias 0 -> 2
- net /Compute/PYRO1_ARM: track 0.00 -> 52.0 mm, vias 0 -> 2
- net /Compute/PYRO1_FIRE: track 0.00 -> 50.7 mm, vias 0 -> 2
- net /Compute/SD_MISO: track 0.00 -> 24.8 mm
- net /Compute/DAT0/MISO: track 22.2 -> 0.00 mm
- net /Compute/SD_CLK: track 21.0 -> 0.00 mm
- net /Compute/CMD/MOSI: track 20.0 -> 0.00 mm
- net /Compute/SD_SCK: track 0.00 -> 19.9 mm
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
Commit message: routing done
Routing:
- net GND: track 67.2 -> 87.7 mm, vias 159 -> 123
- net /Compute/SPI0_MOSI: track 21.3 -> 22.2 mm
- net /Compute/SPI0_MISO: track 23.3 -> 23.9 mm
- net VBUS: vias 2 -> 1

Commit message: final production files
Parts:
- U11: footprint Package_SON:VSON-8-1EP_3x3mm_P0.65mm_EP1.65x2.4mm -> Package_TO_SOT_SMD:SOT-23-8
Connections:
- U5 pad 7: unconnected-(U5-A0-Pad7) -> GND
Routing:
- net /Compute/SPI0_SCK: track 17.3 -> 20.4 mm
- net /Compute/I2C0_SDA: track 30.9 -> 32.8 mm
- net /Compute/PYRO2_ARM: track 61.9 -> 63.6 mm
- net /Compute/CS_RADIO: track 10.9 -> 12.0 mm
- net /Compute/PYRO2_FIRE: track 61.8 -> 62.7 mm
- net /Compute/PYRO2_PRESENT: track 67.4 -> 68.1 mm
- net Net-(BZ1--): track 7.78 -> 8.45 mm
- net /Compute/I2C1_SCL: track 65.4 -> 66.1 mm
- net GND: track 87.7 -> 87.2 mm, vias 123 -> 134
