File: flight-computer-one.kicad_pcb (KiCad board)
At the start: 4 copper layers, 50 x 100 mm, 105 parts, among them J1 LEFT_BANK, J2 RIGHT_BANK, J3 USB_C_Receptacle_USB2.0_16P, J4 SWD, J5 Micro_SD_Card_Det2, J6 COMM u.FL, J7 GNSS u.FL, Q1 CSD17318Q2, Q2 CSD17318Q2, Q3 CSD17318Q2, Q4 CSD17318Q2, Q5 CSD17318Q2, SW1 RESET, SW2 USER, U1 ATSAME51J19A-M, U10 SHT40, U11 TCAN3404-Q1, U12 Ai-Thinker-Ra-01H, U13 MAX-M10S, U2 USBLC6-2SC6, U3 TPS2121, U4 TPS561246, U5 INA232, U6 BMI088, U7 MS5611-01BA, U8 LIS2MDL, U9 ICM-42688-P

Commit message: oopsies fixed I2C
Connections:
- U1 pad 11: /Compute/I2C0_SDA -> unconnected-(U1-PB08-Pad11)
- U1 pad 12: /Compute/I2C0_SCL -> unconnected-(U1-PB09-Pad12)
- U1 pad 17: unconnected-(U1-PA08-Pad17) -> /Compute/I2C0_SDA
- U1 pad 18: /Compute/BUZZER_CTL -> /Compute/I2C0_SCL
- U1 pad 20: unconnected-(U1-PA11-Pad20) -> /Compute/BUZZER_CTL
Routing:
- net /Compute/I2C0_SCL: track 29.7 -> 25.7 mm
- net /Compute/BUZZER_CTL: track 13.2 -> 16.2 mm, vias 0 -> 2
- net /Compute/I2C0_SDA: track 32.8 -> 31.6 mm
Changed lines of the file:
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@@
 	(net 49 "Net-(BZ1--)")
 	(net 50 "Net-(Q1-S-Pad4)")
-	(net 51 "unconnected-(U1-PA08-Pad17)")
+	(net 51 "unconnected-(U1-PB09-Pad12)")
 	(net 52 "Net-(Q3-S-Pad4)")
 	(net 53 "unconnected-(U1-PA07-Pad16)")
@@
 	(net 61 "unconnected-(U1-PB07-Pad10)")
 	(net 62 "unconnected-(U1-PB10-Pad23)")
-	(net 63 "unconnected-(U1-PA11-Pad20)")
+	(net 63 "unconnected-(U1-PB08-Pad11)")
 	(net 64 "unconnected-(U1-PB06-Pad9)")
 	(net 65 "unconnected-(U1-PA14-Pad31)")
@@
 			(layers "F.Cu" "F.Mask" "F.Paste")
 			(roundrect_rratio 0.25)
-			(net 8 "/Compute/I2C0_SDA")
+			(net 63 "unconnected-(U1-PB08-Pad11)")
 			(pinfunction "PB08")
-			(pintype "bidirectional")
+			(pintype "bidirectional+no_connect")
 		)
 		(pad "12" smd roundrect
@@
 			(layers "F.Cu" "F.Mask" "F.Paste")
 			(roundrect_rratio 0.25)
-			(net 9 "/Compute/I2C0_SCL")
+			(net 51 "unconnected-(U1-PB09-Pad12)")
 			(pinfunction "PB09")
-			(pintype "bidirectional")
+			(pintype "bidirectional+no_connect")
 		)
 		(pad "13" smd roundrect
@@
 			(layers "F.Cu" "F.Mask" "F.Paste")
 			(roundrect_rratio 0.25)
-			(net 51 "unconnected-(U1-PA08-Pad17)")
+			(net 8 "/Compute/I2C0_SDA")
 			(pinfunction "PA08")
-			(pintype "bidirectional+no_connect")
+			(pintype "bidirectional")
 		)
 		(pad "18" smd roundrect
@@
 			(layers "F.Cu" "F.Mask" "F.Paste")
 			(roundrect_rratio 0.25)
-			(net 13 "/Compute/BUZZER_CTL")
+			(net 9 "/Compute/I2C0_SCL")
 			(pinfunction "PA09")
 			(pintype "bidirectional")
@@
 			(layers "F.Cu" "F.Mask" "F.Paste")
 			(roundrect_rratio 0.25)
-			(net 63 "unconnected-(U1-PA11-Pad20)")
+			(net 13 "/Compute/BUZZER_CTL")
 			(pinfunction "PA11")
-			(pintype "bidirectional+no_connect")
+			(pintype "bidirectional")
 		)
 		(pad "21" smd roundrect
@@
 	)
 	(segment
-		(start 139.44 74.5625)
-		(end 141.0375 74.5625)
-		(width 0.1)
-		(layer "F.Cu")
-		(net 8)
-	)
-	(segment
 		(start 129.38 85.14)
 		(end 129.45 85.21)
@@
 	)
 	(segment
-		(start 139.1575 74.5625)
-		(end 139.44 74.5625)
-		(width 0.1)
-		(layer "F.Cu")
-		(net 8)
-	)
-	(segment
-		(start 134.89 78.83)
-		(end 139.1575 74.5625)
-		(width 0.1)
-		(layer "F.Cu")
-		(net 8)
-	)
-	(segment
-		(start 133.66 78.83)
-		(end 134.89 78.83)
+		(start 136.19 82.26)
+		(end 134.0675 84.3825)
 		(width 0.1)
 		(layer "F.Cu")
@@
 	)
 	(segment
-		(start 136.19 82.26)
-		(end 134.0675 84.3825)
+		(start 141.7 78.67)
+		(end 141.7 77.725)
 		(width 0.1)
 		(layer "F.Cu")
@@
 	)
 	(segment
-		(start 132.97 78.83)
-		(end 132.77 79.03)
-		(width 0.1)
-		(layer "F.Cu")
-		(net 8)
-	)
-	(segment
 		(start 131.44 83.1)
 		(end 131.44 82.585)
@@
 	)
 	(segment
-		(start 133.66 78.83)
-		(end 132.97 78.83)
+		(start 141.61 79.11)
+		(end 141.61 78.76)
 		(width 0.1)
 		(layer "F.Cu")
@@
 	)
 	(segment
+		(start 141.61 78.76)
+		(end 141.7 78.67)
+		(width 0.1)
+		(layer "F.Cu")
+		(net 8)
+	)
+	(segment
 		(start 130.5925 81.95)
 		(end 131.925 81.95)
@@
 	)
 	(via
-		(at 131.44 83.1)
+		(at 141.61 79.11)
 		(size 0.7)
 		(drill 0.3)
@@
 	)
 	(via
-		(at 132.77 79.03)
-		(size 0.6)
-		(drill 0.2)
+		(at 131.44 83.1)
+		(size 0.7)
+		(drill 0.3)
 		(layers "F.Cu" "B.Cu")
 		(net 8)
 	)
 	(segment
-		(start 132.77 79.03)
-		(end 132.77 81.77)
+		(start 132.73 81.81)
+		(end 133.4 81.14)
 		(width 0.1)
 		(layer "B.Cu")
@@
 	)
 	(segment
-		(start 132.77 81.77)
+		(start 141.61 79.443669)
+		(end 141.61 79.11)
+		(width 0.1)
+		(layer "B.Cu")
+		(net 8)
+	)
+	(segment
+		(start 139.913669 81.14)
+		(end 141.61 79.443669)
+		(width 0.1)
+		(layer "B.Cu")
+		(net 8)
+	)
+	(segment
+		(start 133.4 81.14)
+		(end 139.913669 81.14)
+		(width 0.1)
+		(layer "B.Cu")
+		(net 8)
+	)
+	(segment
+		(start 132.73 81.81)
 		(end 131.44 83.1)
 		(width 0.1)
@@
 	)
 	(segment
-		(start 130.5925 81.15)
-		(end 132.725 81.15)
+		(start 132.77 81.77)
+		(end 132.73 81.81)
 		(width 0.1)
-		(layer "F.Cu")
-		(net 9)
+		(layer "B.Cu")
+		(net 8)
 	)
 	(segment
-		(start 141.0375 75.0625)
-		(end 140.5625 75.0625)
+		(start 130.5925 81.15)
+		(end 132.725 81.15)
 		(width 0.1)
 		(layer "F.Cu")
@@
 	)
 	(segment
-		(start 132.675 84.24)
-		(end 132.8175 84.3825)
+		(start 142.2 77.725)
+		(end 142.2 80.02)
 		(width 0.1)
 		(layer "F.Cu")
@@
 	)
 	(segment
-		(start 140.5625 75.0625)
-		(end 133.6 82.025)
+		(start 132.675 84.24)
+		(end 132.8175 84.3825)
 		(width 0.1)
 		(layer "F.Cu")
@@
 	)
 	(segment
+		(start 142.2 80.02)
+		(end 141.3 80.92)
+		(width 0.1)
+		(layer "F.Cu")
+		(net 9)
+	)
+	(segment
 		(start 140.225 82.025)
+		(end 139.93 82.025)
+		(width 0.1)
+		(layer "F.Cu")
+		(net 9)
+	)
+	(segment
+		(start 139.93 82.025)
 		(end 133.6 82.025)
 		(width 0.1)
@@
 	)
 	(segment
+		(start 140.195 82.025)
+		(end 139.93 82.025)
+		(width 0.1)
+		(layer "F.Cu")
+		(net 9)
+	)
+	(segment
 		(start 132.725 81.15)
 		(end 133.6 82.025)
@@
 	)
 	(segment
+		(start 141.3 80.92)
+		(end 141.3 83.3875)
+		(width 0.1)
+		(layer "F.Cu")
+		(net 9)
+	)
+	(segment
 		(start 141.3 83.1)
 		(end 140.225 82.025)
@@
 	)
 	(segment
-		(start 143.78 81.93)
-		(end 143.14 81.93)
+		(start 144.7775 82.9275)
+		(end 143.84 81.99)
 		(width 0.15)
 		(layer "F.Cu")
@@
 	)
 	(segment
-		(start 143.14 81.93)
-		(end 142.2 80.99)
+		(start 143.1 76.85)
+		(end 143.2 76.95)
 		(width 0.15)
 		(layer "F.Cu")
@@
 	)
 	(segment
-		(start 142.2 80.99)
-		(end 142.2 77.725)
+		(start 143.2 76.95)
+		(end 143.2 77.725)
 		(width 0.15)
 		(layer "F.Cu")
@@
 	)
 	(segment
-		(start 144.7775 82.9275)
-		(end 143.78 81.93)
+		(start 143.84 81.99)
+		(end 143.17 81.99)
 		(width 0.15)
 		(layer "F.Cu")
 		(net 13)
 	)
+	(segment
+		(start 143.1 76.41)
+		(end 143.1 76.85)
+		(width 0.15)
+		(layer "F.Cu")
+		(net 13)
+	)
+	(via
+		(at 143.1 76.41)
+		(size 0.7)
+		(drill 0.3)
+		(layers "F.Cu" "B.Cu")
+		(net 13)
+	)
+	(via
+		(at 143.17 81.99)
+		(size 0.7)
+		(drill 0.3)
+		(layers "F.Cu" "B.Cu")
+		(net 13)
+	)
+	(segment
+		(start 142.234 77.276)
+		(end 143.1 76.41)
+		(width 0.15)
+		(layer "B.Cu")
+		(net 13)
+	)
+	(segment
+		(start 143.17 81.99)
+		(end 142.234 81.054)
+		(width 0.15)
+		(layer "B.Cu")
+		(net 13)
+	)
+	(segment
+		(start 142.234 81.054)
+		(end 142.234 77.276)
+		(width 0.15)
+		(layer "B.Cu")
+		(net 13)
+	)

Commit message: Final production files (again)
Parts:
- R8: footprint Resistor_SMD:R_Shunt_Vishay_WSKW0612 -> LRI_Partlib:L4CA0612L0M50FNR
- moved C1 5.16 mm to (161.0, 100.9), turned to 0 degrees
- moved R5 4.79 mm to (161.0, 102.5), turned to 0 degrees
- moved R8 3.34 mm to (157.8, 106.0), turned to -90 degrees
- moved C5 2.32 mm to (164.3, 107.4)
- moved R11 2.32 mm to (162.0, 106.6)
- moved R10 2.32 mm to (162.0, 108.2)
- moved C7 1.30 mm to (169.4, 107.2)
- moved U5 1.30 mm to (166.8, 106.7)
- moved U3 0.80 mm to (157.8, 101.7), turned to -90 degrees
Connections:
- R8 pad 1: PWROR -> Net-(R11-Pad1)
- R8 pad 2: Net-(R11-Pad1) -> PWROR
- R8 pad 3: Net-(R10-Pad1) -> +PBP
- R8 pad 4: +PBP -> Net-(R10-Pad1)
Routing:
- net PWROR: track 7.82 -> 3.83 mm
- net +PBP: track 16.8 -> 20.4 mm
- net Net-(R11-Pad1): track 1.50 -> 3.44 mm
- net Net-(R10-Pad1): track 1.51 -> 3.09 mm
- net /Compute/I2C1_SDA: track 67.2 -> 68.4 mm
- net /Power & USB/PMON_IN+: track 3.24 -> 4.27 mm
- net GND: track 87.2 -> 88.2 mm, vias 134 -> 132
- net VBUS: track 31.7 -> 30.9 mm
- net /Power & USB/PMON_IN-: track 5.08 -> 5.59 mm
