File: connectivity.kicad_sch (KiCad schematic)
At the start: 5 parts, among them J2 Conn_Coaxial, J5 Conn_Coaxial, U11 Ai-Thinker-Ra-01, U4 MCP2518FD-xQBB, U6 MAX-M10S

Commit message: created project lib
Parts:
- renumbered J2 to J6
Other:
- note added: "TCAN1472-Q1 MISSING"
Changed lines of the file:
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@@
 	(generator_version "9.0")
 	(paper "A4")
+	(text "TCAN1472-Q1 MISSING"
+		(exclude_from_sim no)
+		(at 201.168 46.228 0)
+		(effects
+			(font
+				(size 3.81 3.81)
+			)
+		)
+	)
 	(wire
 		(pts
@@
 		(dnp no)
 		(fields_autoplaced yes)
-		(property "Reference" "J2"
+		(property "Reference" "J6"
 			(at 163.83 114.5931 0)
 			(effects
@@
 			(project "flight-computer-one"
 				(path "/2b49a1e7-3a95-411d-8c49-438ba0d49dde/34ffb04f-a567-4939-915a-72e6afee4bc4"
-					(reference "J2")
+					(reference "J6")
 					(unit 1)
 				)

Commit message: added gitignore
Parts:
- added U11: TCAN3404-Q1, Package_SON:VSON-8-1EP_3x3mm_P0.65mm_EP1.65x2.4mm, symbol Interface_CAN_LIN:TCAN334G
- U9: renamed from U11; value Ai-Thinker-Ra-01 -> Ai-Thinker-Ra-01H
- renumbered U6 to U3
Connections:
- net GND: now also U11.2 (GND)
- new net +3V3: U11.3 (VCC)
Other:
- note removed: "TCAN1472-Q1 MISSING"
- moved on the sheet: U4

Commit message: Fixed BMI088 footprint and readme
Connections:
- net GND: now also U11.9 (EP)
Changed lines of the file:
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@@
 	(generator_version "9.0")
 	(paper "A4")
+	(junction
+		(at 115.57 82.55)
+		(diameter 0)
+		(color 0 0 0 0)
+	)
+	(wire
+		(pts
+			(xy 113.03 82.55) (xy 115.57 82.55)
+		)
+		(stroke
+			(width 0)
+			(type default)
+		)
+	)
 	(wire
 		(pts
@@
 	(wire
 		(pts
-			(xy 115.57 57.15) (xy 115.57 60.96)
+			(xy 115.57 58.42) (xy 115.57 60.96)
 		)
 		(stroke
@@
 		(pts
 			(xy 115.57 81.28) (xy 115.57 82.55)
+		)
+		(stroke
+			(width 0)
+			(type default)
+		)
+	)
+	(wire
+		(pts
+			(xy 115.57 82.55) (xy 115.57 83.82)
+		)
+		(stroke
+			(width 0)
+			(type default)
+		)
+	)
+	(wire
+		(pts
+			(xy 113.03 81.28) (xy 113.03 82.55)
 		)
 		(stroke
@@
 	(symbol
 		(lib_id "power:GND")
-		(at 115.57 82.55 0)
+		(at 115.57 83.82 0)
 		(unit 1)
 		(exclude_from_sim no)
@@
 		(fields_autoplaced yes)
 		(property "Reference" "#PWR023"
+			(at 115.57 90.17 0)
+			(effects
+				(font
+					(size 1.27 1.27)
+				)
+				(hide yes)
+			)
+		)
+		(property "Value" "GND"
 			(at 115.57 88.9 0)
 			(effects
@@
 					(size 1.27 1.27)
 				)
-				(hide yes)
-			)
-		)
-		(property "Value" "GND"
-			(at 115.57 87.63 0)
-			(effects
-				(font
-					(size 1.27 1.27)
-				)
 			)
 		)
 		(property "Footprint" ""
-			(at 115.57 82.55 0)
+			(at 115.57 83.82 0)
 			(effects
 				(font
@@
 		)
 		(property "Datasheet" ""
-			(at 115.57 82.55 0)
+			(at 115.57 83.82 0)
 			(effects
 				(font
@@
 		)
 		(property "Description" "Power symbol creates a global label with name \"GND\" , ground"
-			(at 115.57 82.55 0)
+			(at 115.57 83.82 0)
 			(effects
 				(font
@@
 	(symbol
 		(lib_id "power:+3V3")
-		(at 115.57 57.15 0)
+		(at 115.57 58.42 0)
 		(unit 1)
 		(exclude_from_sim no)
@@
 		(fields_autoplaced yes)
 		(property "Reference" "#PWR024"
-			(at 115.57 60.96 0)
+			(at 115.57 62.23 0)
 			(effects
 				(font
@@
 		)
 		(property "Value" "+3V3"
-			(at 115.57 52.07 0)
+			(at 115.57 53.34 0)
 			(effects
 				(font
@@
 		)
 		(property "Footprint" ""
-			(at 115.57 57.15 0)
+			(at 115.57 58.42 0)
 			(effects
 				(font
@@
 		)
 		(property "Datasheet" ""
-			(at 115.57 57.15 0)
+			(at 115.57 58.42 0)
 			(effects
 				(font
@@
 		)
 		(property "Description" "Power symbol creates a global label with name \"+3V3\""
-			(at 115.57 57.15 0)
+			(at 115.57 58.42 0)
 			(effects
 				(font
@@
 		(pin "3"
 		)
-		(instances
+		(pin "9"
+		)
+		(instances

Commit message: nearly completed schematic, partial layout
Parts:
- added Y2: ASE-40.000MHz, Oscillator:Oscillator_SMD_Abracon_ASE-4Pin_3.2x2.5mm, symbol Oscillator:ASE-xxxMHz
- J5: value Conn_Coaxial -> GNSS u.FL
- J6: value Conn_Coaxial -> COMM u.FL
Connections:
- net +3V3: now also U3.7 (VCC_IO), U3.8 (VCC), U4.14 (VDD), U9.3 (VDD), Y2.4 (Vdd)
- net GND: now also U3.1 (GND), U3.10 (GND), U3.12 (GND), U4.15 (VSS), U4.7 (VSS), U9.16 (GND), U9.2 (GND), U9.9 (GND), Y2.2 (GND)
- net ANT_COMM: now reaches J6.1 (In), U9.1 (ANT)
- net at U4.1 (TXCAN): now also U11.1 (TXD)
- net at U4.2 (RXCAN): now also U11.4 (RXD)
- net at U4.6 (OSC1): now also Y2.3 (OUT)
- net ANT_GNSS: now reaches J5.1 (In), U3.11 (RF_IN)
- net I2C0_SDA: now reaches U3.16 (SDA)
- net I2C0_SCL: now reaches U3.17 (SCL)
- net CANL: now reaches U11.6 (CANL)
- net CANH: now reaches U11.7 (CANH)
- net TCAN_STB: now reaches U11.8 (STB)
- no-connect marks 0 -> 12
Other:
- note added: "GNSS Receiver I2C Addr: 0x42"
- moved on the sheet: J5, J6, U11, U3, U9

Commit message: schematic + prelim layout nearly complete
Parts:
- removed Y2: ASE-40.000MHz, Oscillator:Oscillator_SMD_Abracon_ASE-4Pin_3.2x2.5mm, symbol Oscillator:ASE-xxxMHz
- added C38: 0.1u, Capacitor_SMD:C_0603_1608Metric, symbol Device:C
- added R28: 10K, Resistor_SMD:R_0603_1608Metric, symbol Device:R
- added Y2: SG-210STF 40M, Crystal:Crystal_SMD_2520-4Pin_2.5x2.0mm, symbol Oscillator:SG-210STF
Connections:
- net +3V3: now also C38.2, R28.1, Y2.4 (Vcc)
- net GND: now also C38.1, Y2.2 (GND)
- net SPI0_SCK: now reaches U9.12 (SCK)
- net SPI0_SCK: now also U4.13 (~{CS})
- net SPI0_MISO: now reaches U9.13 (MISO)
- net SPI0_MISO: now also U4.12 (SDO)
- net SPI0_MOSI: now reaches U9.14 (MOSI)
- net SPI0_MOSI: now also U4.11 (SDI)
- net CS_RADIO: now reaches U9.15 (~{NSS})
- net at U9.4 (~{RESET}): now also R28.2
- net at U4.6 (OSC1): now also Y2.3 (OUT)
- net CS_CANXC: now reaches U4.10 (SCK)
- no-connect marks 12 -> 19
Other:
- note added: "COMM radio transceiver SPI, active w CS_RADIO"
- note added: "MISSING CAN TERMINATION"
- moved on the sheet: U11, U4

Commit message: Schematic tentatively complete
Parts:
- added C41: 100p, Capacitor_SMD:C_0603_1608Metric, symbol Device:C
- added R35, R36: 59, Resistor_SMD:R_0603_1608Metric, symbol Device:R
Connections:
- net CANH: now also R35.1
- net CANL: now also R36.2
- net GND: now also C41.1
- new net: C41.2, R35.2, R36.1
- no-connect marks 19 -> 23
Other:
- note added: "SPI to 8Mbps CAN FD w/ split termination"
- note removed: "MISSING CAN TERMINATION"
- moved on the sheet: J5, J6, R28, U3, U9

Commit message: schematic tentatively finished
Connections:
- net RADIO_nRST: now reaches R28.2, U9.4 (~{RESET})
- net RXCAN: now reaches U11.1 (TXD), U4.1 (TXCAN)
- net TXCAN: now reaches U11.4 (RXD), U4.2 (RXCAN)
Other:
- moved on the sheet: U4

Commit message: swapped POR chip for TPS2121
Parts:
- added C42, C43: 0.1u, Capacitor_SMD:C_0603_1608Metric, symbol Device:C
Connections:
- net +3V3: now also C42.2, C43.2
- net GND: now also C42.1, C43.1
