File: connectivity.kicad_sch (KiCad schematic)
At the start: 14 parts, among them J5 GNSS u.FL, J6 COMM u.FL, U11 TCAN3404-Q1, U3 MAX-M10S, U4 MCP2518FD-xQBB, U9 Ai-Thinker-Ra-01H, Y2 SG-210STF 40M

Commit message: same51 wired, near completion
Parts:
- removed C38, C42, C43: 0.1u, Capacitor_SMD:C_0603_1608Metric, symbol Device:C
- removed U4: MCP2518FD-xQBB, Package_DFN_QFN:DFN-14-1EP_3x4.5mm_P0.65mm_EP1.65x4.25mm, symbol Interface_CAN_LIN:MCP2518FD-xQBB
- removed Y2: SG-210STF 40M, Crystal:Crystal_SMD_2520-4Pin_2.5x2.0mm, symbol Oscillator:SG-210STF
- renumbered C41 to C28, J5 to J7, R28 to R19, R35 to R20, R36 to R21, U9 to U12, U3 to U13
Connections:
- net RXCAN: now also U11.4 (RXD); no longer U11.1 (TXD)
- net TXCAN: now also U11.1 (TXD); no longer U11.4 (RXD)
- no-connect marks 23 -> 17
Other:
- note added: "8Mbps CAN FD w/ split termination"
- note removed: "SPI to 8Mbps CAN FD w/ split termination"
- moved on the sheet: C28, J7, R20, R21, U11, U13

Commit message: new routing
Connections:
- net I2C0_SCL renamed I2C1_SCL
- net I2C0_SDA renamed I2C1_SDA
Changed lines of the file:
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@@
 		)
 	)
-	(hierarchical_label "I2C0_SCL"
+	(hierarchical_label "I2C1_SCL"
 		(shape input)
 		(at 176.53 64.77 180)
@@
 		)
 	)
-	(hierarchical_label "I2C0_SDA"
+	(hierarchical_label "I2C1_SDA"
 		(shape bidirectional)
 		(at 176.53 62.23 180)

Commit message: final production files
Parts:
- U11: footprint Package_SON:VSON-8-1EP_3x3mm_P0.65mm_EP1.65x2.4mm -> Package_TO_SOT_SMD:SOT-23-8
- U13: DK Part (none) -> https://www.digikey.com/en/products/detail/u-blox/MAX-M10S-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
Changed lines of the file:
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@@
+			)
+		)
+		(property "DK Part" "https://www.digikey.com/en/products/detail/u-blox/MAX-M10S-00B/15712906"
+			(at 195.58 64.77 0)
+			(effects
+				(font
+					(size 1.27 1.27)
+				)
+				(hide yes)
 			)
 		)
@@
 			)
 		)
-		(property "Footprint" "Package_SON:VSON-8-1EP_3x3mm_P0.65mm_EP1.65x2.4mm"
+		(property "Footprint" "Package_TO_SOT_SMD:SOT-23-8"
 			(at 69.85 69.85 0)
 			(effects
