File: power_usb.kicad_sch (KiCad schematic)
At the start: 8 parts, among them J3 USB_C_Receptacle_USB2.0_16P, U10 USBLC6-2SC6, U2 NCP1117-3.3_SOT223

Commit message: added gitignore
Parts:
- removed C19, C5: 10u, Capacitor_SMD:C_0805_2012Metric, symbol Device:C
- removed U2: NCP1117-3.3_SOT223, Package_TO_SOT_SMD:SOT-223-3_TabPin2, symbol Regulator_Linear:NCP1117-3.3_SOT223
- added D1: PMEG4005CT, Package_TO_SOT_SMD:SOT-23, symbol Device:D_Dual_CommonCathode_AAK_Parallel
- R5: value 5k1 -> 5.1K
- R6: renamed from R13; value 5k1 -> 5.1K; footprint Capacitor_SMD:C_0603_1608Metric -> Resistor_SMD:R_0603_1608Metric
Connections:
- net +5V is gone; now on net VBUS: C1.1
- net +BATT: now also D1.2 (A)
- net VBUS: now also D1.1 (A)
- new net +VSYS: D1.3 (K)
Other:
- note added: "18V to 3.3V buck"
- note added: "INA232 power monitor on VSYS"
- note added: "Power OR (and technically RPP too)"
- note removed: "5V power-OR"
- note removed: "Buck to 5V"
- moved on the sheet: C1

Commit message: Fixed BMI088 footprint and readme
Parts:
- removed D1: PMEG4005CT, Package_TO_SOT_SMD:SOT-23, symbol Device:D_Dual_CommonCathode_AAK_Parallel
Other:
- note added: "13V to 3.3V buck"
- note added: "Power muxing"
- note added: "TPS2121, INA232, BUCK MISSING"
- note removed: "18V to 3.3V buck"
- note removed: "Power OR (and technically RPP too)"
Changed lines of the file:
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@@
 	(generator_version "9.0")
 	(paper "A4")
-	(text "18V to 3.3V buck"
+	(text "13V to 3.3V buck"
 		(exclude_from_sim no)
 		(at 206.502 116.84 0)
@@
 		)
 	)
+	(text "TPS2121, INA232, BUCK MISSING"
+		(exclude_from_sim no)
+		(at 106.172 142.494 0)
+		(effects
+			(font
+				(size 3.81 3.81)
+			)
+		)
+	)
 	(text "INA232 power monitor on VSYS"
 		(exclude_from_sim no)
@@
 		)
 	)
-	(text "Power OR (and technically RPP too)"
+	(text "Power muxing"
 		(exclude_from_sim no)
 		(at 204.47 39.37 0)
@@
 			)
 		)
-		(property "Value" "+VSYS"
+		(property "Value" "VSYS"
 			(at 228.6 44.45 0)
 			(effects
@@
 			)
 		)
-		(property "Value" "+VSYS"
+		(property "Value" "VSYS"
 			(at 180.34 105.41 0)
 			(effects
@@
 					(unit 1)
 				)
-			)
-		)
-	)
-	(symbol
-		(lib_id "Device:D_Dual_CommonCathode_AAK_Parallel")
-		(at 208.28 55.88 0)
-		(unit 1)
-		(exclude_from_sim no)
-		(in_bom yes)
-		(on_board yes)
-		(dnp no)
-		(fields_autoplaced yes)
-		(property "Reference" "D1"
-			(at 208.2165 46.99 0)
-			(effects
-				(font
-					(size 1.27 1.27)
-				)
-			)
-		)
-		(property "Value" "PMEG4005CT"
-			(at 208.2165 49.53 0)
-			(effects
-				(font
-					(size 1.27 1.27)
-				)
-			)
-		)
-		(property "Footprint" "Package_TO_SOT_SMD:SOT-23"
-			(at 209.55 55.88 0)
-			(effects
-				(font
-					(size 1.27 1.27)
-				)
-				(hide yes)
-			)
-		)
-		(property "Datasheet" "https://assets.nexperia.com/documents/data-sheet/PMEG4005CT.pdf"
-			(at 209.55 55.88 0)
-			(effects
-				(font
-					(size 1.27 1.27)
-				)
-				(hide yes)
-			)
-		)
-		(property "Description" "Dual diode, common cathode on pin 3"
-			(at 208.28 55.88 0)
-			(effects
-				(font
-					(size 1.27 1.27)
-				)
-				(hide yes)
-			)
-		)
-		(pin "1"
-		)
-		(pin "3"
-		)
-		(pin "2"
-		)
-		(instances
-			(project ""
-				(path "/2b49a1e7-3a95-411d-8c49-438ba0d49dde/420394b1-4c9b-4d8d-83f2-b66955e186e4"
-					(reference "D1")
-					(unit 1)
-				)

Commit message: progress, particularly on power
Parts:
- added C19: 22u, Capacitor_SMD:C_0805_2012Metric, symbol Device:C
- added C30: 10u, Capacitor_SMD:C_0805_2012Metric, symbol Device:C
- added C31: 100n, Capacitor_SMD:C_0603_1608Metric, symbol Device:C
- added C5: 0.1u, Capacitor_SMD:C_0603_1608Metric, symbol Device:C
- added FB1: 220R@100MHz, Inductor_SMD:L_0603_1608Metric, symbol Device:FerriteBead
- added L2: 3.3u, symbol Device:L
- added Q5, Q6: CSD17318Q2, Package_SON:Texas_DQK, symbol Transistor_FET:CSD17313Q2
- added R16: R_Shunt, Resistor_SMD:R_Shunt_Vishay_WSKW0612, symbol Device:R_Shunt
- added R17, R19: 100K, Resistor_SMD:R_0603_1608Metric, symbol Device:R
- added R18: 22.1K, Resistor_SMD:R_0603_1608Metric, symbol Device:R
- added U12: INA232, LRI_partlib:TSOT-23-8, symbol LRI_partlib:INA232
- added U13, U14: NCV68061, Package_TO_SOT_SMD:SOT-23-6, symbol LRI_partlib:NCV68061
- added U15: TPS561246, Package_TO_SOT_SMD:SOT-563, symbol LRI_partlib:TPS561246
- C1: value 10u -> 10n; footprint Capacitor_SMD:C_0805_2012Metric -> Capacitor_SMD:C_0603_1608Metric
Connections:
- net +3V3: now also C19.1, L2.2, R17.2
- net +BATT: now also Q5.4 (S), Q5.7 (S), U13.3 (EN), U13.6 (S)
- net GND: now also C1.1, C19.2, C30.2, C31.1, R18.2, U12.3 (GND), U13.2 (GND), U14.2 (GND), U15.3 (GND); no longer C1.2
- net VBUS: now also C31.2, FB1.2, Q6.4 (S), Q6.7 (S), U14.3 (EN), U14.6 (S); no longer C1.1, J3.A4 (VBUS), J3.A9 (VBUS), J3.B4 (VBUS), J3.B9 (VBUS)
- new net: C5.1, U15.4 (BST)
- new net: R19.2, U15.5 (EN)
- new net: Q5.3 (G), U13.5 (G)
- new net: Q6.3 (G), U14.5 (G)
- new net +PBP: C30.1, R16.4, R19.1, U15.1 (VIN)
- new net PWROR: Q5.1 (D), Q5.2 (D), Q5.5 (D), Q5.6 (D), Q5.8 (D), Q6.1 (D), Q6.2 (D), Q6.5 (D), Q6.6 (D), Q6.8 (D), R16.1, U13.4 (D), U14.4 (D)
- new net TPS_FB: R17.1, R18.1, U15.6 (FB)
- new net TPS_SW: C5.2, L2.1, U15.2 (SW)
- new net VBUS_RAW: C1.2, FB1.1, J3.A4 (VBUS), J3.A9 (VBUS), J3.B4 (VBUS), J3.B9 (VBUS)
- no-connect marks 2 -> 4
Other:
- note added: "PBP = Protected Battery Power"
- note added: "Powering the pyros from +PBP instead of +BATT ensures that the pyro MOSFETs get RPP too, but it also theoretically allows you to light e-matches when the board is only powered from the USB port. Don't actually light e-matches with your laptop! Use a high-value resistor for testing instead."
- note removed: "13V to 3.3V buck"
- note removed: "INA232 power monitor on VSYS"
- note removed: "Power muxing"
- note removed: "TPS2121, INA232, BUCK MISSING"
- moved on the sheet: C1, U10

Commit message: nearly completed schematic, partial layout
Parts:
- C31: value 100n -> 0.1u
- L2: value 3.3u -> 3.3uH
Connections:
- net +3V3: now also U12.4 (VS)
- net CONN_D+: now also J3.A6 (D+), J3.B6 (D+), U10.3 (I/O2); no longer J3.A7 (D-), J3.B7 (D-), U10.1 (I/O1)
- net CONN_D-: now also J3.A7 (D-), J3.B7 (D-), U10.1 (I/O1); no longer J3.A6 (D+), J3.B6 (D+), U10.3 (I/O2)
- net USB_D+: now also U10.4 (I/O2); no longer U10.6 (I/O1)
- net USB_D-: now also U10.6 (I/O1); no longer U10.4 (I/O2)
- net VBUS: no longer U10.5 (VBUS)
- net VBUS_RAW: now also U10.5 (VBUS)
- no-connect marks 4 -> 6
Changed lines of the file:
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@@
 	)
 	(no_connect
+		(at 226.06 66.04)
+	)
+	(no_connect
 		(at 63.5 156.21)
 	)
@@
 		(at 52.07 59.69)
 	)
+	(no_connect
+		(at 226.06 68.58)
+	)
 	(wire
 		(pts
@@
 	(wire
 		(pts
+			(xy 74.93 44.45) (xy 74.93 43.18)
+		)
+		(stroke
+			(width 0)
+			(type default)
+		)
+	)
+	(wire
+		(pts
 			(xy 53.34 44.45) (xy 53.34 41.91)
 		)
@@
 	(wire
 		(pts
+			(xy 66.04 46.99) (xy 66.04 45.72)
+		)
+		(stroke
+			(width 0)
+			(type default)
+		)
+	)
+	(wire
+		(pts
 			(xy 179.07 124.46) (xy 176.53 124.46)
 		)
@@
 	(wire
 		(pts
+			(xy 215.9 52.07) (xy 215.9 53.34)
+		)
+		(stroke
+			(width 0)
+			(type default)
+		)
+	)
+	(wire
+		(pts
 			(xy 53.34 49.53) (xy 53.34 46.99)
 		)
@@
 		)
 	)
-	(label "USB_D+"
+	(label "USB_D-"
 		(at 113.03 60.96 180)
 		(effects
@@
 		)
 	)
-	(label "CONN_D+"
+	(label "CONN_D-"
 		(at 76.2 60.96 180)
 		(effects
@@
 		)
 	)
-	(label "USB_D-"
+	(label "USB_D+"
 		(at 113.03 63.5 180)
 		(effects
@@
 		)
 	)
-	(label "CONN_D-"
+	(label "CONN_D+"
 		(at 76.2 63.5 180)
 		(effects
@@
 			)
 		)
-		(property "Value" "VBUS"
+		(property "Value" "VBUS_RAW"
 			(at 86.741 48.9458 0)
 			(effects
@@
 			)
 		)
-		(property "Value" "3.3u"
+		(property "Value" "3.3uH"
 			(at 228.6 116.84 90)
 			(effects
@@
 	(symbol
 		(lib_id "power:GND")
-		(at 74.93 43.18 0)
+		(at 74.93 44.45 0)
 		(unit 1)
 		(exclude_from_sim no)
@@
 		(dnp no)
 		(property "Reference" "#PWR046"
-			(at 74.93 49.53 0)
+			(at 74.93 50.8 0)
 			(effects
 				(font
@@
 		)
 		(property "Value" "GND"
-			(at 75.057 47.5742 0)
+			(at 75.057 48.8442 0)
 			(effects
 				(font
@@
 		)
 		(property "Footprint" ""
-			(at 74.93 43.18 0)
+			(at 74.93 44.45 0)
 			(effects
 				(font
@@
 		)
 		(property "Datasheet" ""
-			(at 74.93 43.18 0)
+			(at 74.93 44.45 0)
 			(effects
 				(font
@@
 		)
 		(property "Description" ""
-			(at 74.93 43.18 0)
+			(at 74.93 44.45 0)
 			(effects
 				(font
@@
 	)
 	(symbol
+		(lib_id "power:+3V3")
+		(at 215.9 52.07 0)
+		(unit 1)
+		(exclude_from_sim no)
+		(in_bom yes)
+		(on_board yes)
+		(dnp no)
+		(property "Reference" "#PWR077"
+			(at 215.9 55.88 0)
+			(effects
+				(font
+					(size 1.27 1.27)
+				)
+				(hide yes)
+			)
+		)
+		(property "Value" "+3V3"
+			(at 216.281 47.6758 0)
+			(effects
+				(font
+					(size 1.27 1.27)
+				)
+			)
+		)
+		(property "Footprint" ""
+			(at 215.9 52.07 0)
+			(effects
+				(font
+					(size 1.27 1.27)
+				)
+				(hide yes)
+			)
+		)
+		(property "Datasheet" ""
+			(at 215.9 52.07 0)
+			(effects
+				(font
+					(size 1.27 1.27)
+				)
+				(hide yes)
+			)
+		)
+		(property "Description" ""
+			(at 215.9 52.07 0)
+			(effects
+				(font
+					(size 1.27 1.27)
+				)
+				(hide yes)
+			)
+		)
+		(pin "1"
+		)
+		(instances
+			(project "flight-computer-one"
+				(path "/2b49a1e7-3a95-411d-8c49-438ba0d49dde/420394b1-4c9b-4d8d-83f2-b66955e186e4"
+					(reference "#PWR077")
+					(unit 1)
+				)
+			)
+		)
+	)
+	(symbol
 		(lib_id "Device:R")
 		(at 66.04 41.91 0)
@@
 	(symbol
 		(lib_id "power:GND")
-		(at 66.04 45.72 0)
+		(at 66.04 46.99 0)
 		(unit 1)
 		(exclude_from_sim no)
@@
 		(dnp no)
 		(property "Reference" "#PWR062"
-			(at 66.04 52.07 0)
+			(at 66.04 53.34 0)
 			(effects
 				(font
@@
 		)
 		(property "Value" "GND"
-			(at 66.04 50.038 0)
+			(at 66.04 51.308 0)
 			(effects
 				(font
@@
 		)
 		(property "Footprint" ""
-			(at 66.04 45.72 0)
+			(at 66.04 46.99 0)
 			(effects
 				(font
@@
 		)
 		(property "Datasheet" ""
-			(at 66.04 45.72 0)
+			(at 66.04 46.99 0)
 			(effects
 				(font
@@
 		)
 		(property "Description" ""
-			(at 66.04 45.72 0)
+			(at 66.04 46.99 0)
 			(effects
 				(font
@@
 			)
 		)
-		(property "Value" "100n"
+		(property "Value" "0.1u"
 			(at 102.489 33.147 0)
 			(effects

Commit message: schematic + prelim layout nearly complete
Parts:
- added C39: 0.1u, Capacitor_SMD:C_0603_1608Metric, symbol Device:C
- added C40: 10n, Capacitor_SMD:C_0603_1608Metric, symbol Device:C
- added R33, R34: 100, Resistor_SMD:R_0603_1608Metric, symbol Device:R
- R16: value R_Shunt -> 10m
Connections:
- net +3V3: now also C39.1
- net GND: now also C39.2
- net PMON_IN+: now reaches U12.1 (IN+)
- net PMON_IN+: now also C40.2, R34.2
- net PMON_IN-: now reaches U12.2 (IN-)
- net PMON_IN-: now also C40.1, R33.2
- net I2C0_SCL: now reaches U12.5 (SCL)
- net I2C0_SDA: now reaches U12.6 (SDA)
- net at R16.2: now also R34.1
- net at R16.3: now also R33.1
Other:
- note added: "3.3V buck converter"
- note added: "Power OR and RVP"
- note added: "Power monitoring"
- note added: "You can use ADCRANGE=1."
- moved on the sheet: C19, C30, C5, L2, R16, R17, R18, R19, U12, U15

Commit message: Schematic tentatively complete
Parts:
- added D1: Green 5mA, LED_SMD:LED_0603_1608Metric, symbol Device:LED
- added R37: 634, Resistor_SMD:R_0603_1608Metric, symbol Device:R
- added TP2: 3V3, TestPoint:TestPoint_Pad_D1.0mm, symbol Connector:TestPoint
- L2: footprint (none) -> Inductor_SMD:L_Murata_DFE201610P
Connections:
- net +3V3: now also TP2.1
- net GND: now also R37.2
- net VBUS: now also D1.2 (A)
- new net: D1.1 (K), R37.1
Other:
- moved on the sheet: C39, C40, R16, R33, R34, U12

Commit message: schematic tentatively finished
Connections:
- net TPS_EN: now reaches R19.2, U15.5 (EN)
Changed lines of the file:
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@@
 	(wire
 		(pts
-			(xy 91.44 60.96) (xy 113.03 60.96)
-		)
-		(stroke
-			(width 0)
-			(type default)
-		)
-	)
-	(wire
-		(pts
-			(xy 233.68 134.62) (xy 245.11 134.62)
+			(xy 91.44 60.96) (xy 106.68 60.96)
+		)
+		(stroke
+			(width 0)
+			(type default)
+		)
+	)
+	(wire
+		(pts
+			(xy 233.68 134.62) (xy 241.3 134.62)
 		)
 		(stroke
@@
 	(wire
 		(pts
-			(xy 91.44 63.5) (xy 113.03 63.5)
+			(xy 91.44 63.5) (xy 106.68 63.5)
 		)
 		(stroke
@@
 	(wire
 		(pts
-			(xy 233.68 137.16) (xy 245.11 137.16)
+			(xy 233.68 137.16) (xy 241.3 137.16)
 		)
 		(stroke
@@
 		)
 	)
-	(label "USB_D-"
-		(at 113.03 60.96 180)
-		(effects
-			(font
-				(size 1.27 1.27)
-			)
-			(justify right bottom)
-		)
-	)
 	(label "CONN_D-"
 		(at 76.2 60.96 180)
@@
 		)
 	)
-	(label "I2C0_SCL"
-		(at 245.11 137.16 180)
-		(effects
-			(font
-				(size 1.27 1.27)
-			)
-			(justify right bottom)
-		)
-	)
-	(label "I2C0_SDA"
-		(at 245.11 134.62 180)
-		(effects
-			(font
-				(size 1.27 1.27)
-			)
-			(justify right bottom)
-		)
-	)
-	(label "USB_D+"
-		(at 113.03 63.5 180)
-		(effects
-			(font
-				(size 1.27 1.27)
-			)
-			(justify right bottom)
+	(label "TPS_EN"
+		(at 184.15 71.12 0)
+		(effects
+			(font
+				(size 1.27 1.27)
+			)
+			(justify left bottom)
 		)
 	)
@@
 		)
 	)
+	(hierarchical_label "I2C0_SCL"
+		(shape input)
+		(at 241.3 137.16 0)
+		(effects
+			(font
+				(size 1.27 1.27)
+			)
+			(justify left)
+		)
+	)
+	(hierarchical_label "I2C0_SDA"
+		(shape bidirectional)
+		(at 241.3 134.62 0)
+		(effects
+			(font
+				(size 1.27 1.27)
+			)
+			(justify left)
+		)
+	)
+	(hierarchical_label "USB_D-"
+		(shape bidirectional)
+		(at 106.68 60.96 0)
+		(effects
+			(font
+				(size 1.27 1.27)
+			)
+			(justify left)
+		)
+	)
+	(hierarchical_label "USB_D+"
+		(shape bidirectional)
+		(at 106.68 63.5 0)
+		(effects
+			(font
+				(size 1.27 1.27)
+			)
+			(justify left)
+		)
+	)

Commit message: swapped POR chip for TPS2121
Parts:
- removed Q5, Q6: CSD17318Q2, Package_SON:Texas_DQK, symbol Transistor_FET:CSD17313Q2
- removed U13, U14: NCV68061, Package_TO_SOT_SMD:SOT-23-6, symbol LRI_partlib:NCV68061
- added C44: 10n, Capacitor_SMD:C_0603_1608Metric, symbol Device:C
- added R39: 100K, Capacitor_SMD:C_0603_1608Metric, symbol Device:R
- added U18: TPS2121, Package_DFN_QFN:Texas_VQFN-HR-12_2x2.5mm_P0.5mm_ThermalVias, symbol LRI_partlib:TPS2121
Connections:
- net +BATT: now also U18.7 (IN1)
- net GND: now also C44.2, R39.2, U18.12 (GND), U18.3 (CP2), U18.4 (OV2), U18.5 (OV1), U18.6 (PR1), U18.9 (ST)
- net PWROR: now also U18.1 (OUT), U18.8 (OUT)
- net VBUS: now also U18.2 (IN2)
- new net: R39.1, U18.10 (ILM)
- new net: C44.1, U18.11 (SS)
- no-connect marks 6 -> 4
Other:
- moved on the sheet: C40, D1, R16, R33, R34, R37
