File: power_usb.kicad_sch (KiCad schematic)
At the start: 27 parts, among them J3 USB_C_Receptacle_USB2.0_16P, U10 USBLC6-2SC6, U12 INA232, U15 TPS561246, U18 TPS2121

Commit message: added pictures to readme
Parts:
- C40: value 10n -> 0.1u
Changed lines of the file:
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@@
 			)
 		)
-		(property "Value" "10n"
+		(property "Value" "0.1u"
 			(at 179.832 140.97 0)
 			(effects

Commit message: preliminary change to SAME51
Parts:
- added D3: Red 5mA, LED_SMD:LED_0603_1608Metric, symbol Device:LED
- added R40: 634, Resistor_SMD:R_0603_1608Metric, symbol Device:R
- D1: value Green 5mA -> Red 5mA
- renumbered L2 to L1
Connections:
- net +3V3: now also D3.2 (A)
- net GND: now also R40.2
- new net: D3.1 (K), R40.1
Other:
- moved on the sheet: D1, R37

Commit message: same51 wired, near completion
Parts:
- renumbered C44 to C1, C1 to C2, C31 to C3, C30 to C4, C40 to C5, C5 to C6, C39 to C7, C19 to C8, D3 to D2, R33 to R10, R34 to R11, R17 to R12, R18 to R13, R6 to R3, R5 to R4, R39 to R5, R37 to R6, R40 to R7, R16 to R8, R19 to R9, TP2 to TP1, U10 to U2, U18 to U3, U15 to U4, U12 to U5
Connections:
- net USB_CC2: now reaches J3.B5 (CC2), R3.1
- net USB_CC1: now reaches J3.A5 (CC1), R4.1
Other:
- note removed: "PBP = Protected Battery Power"
- note removed: "Powering the pyros from +PBP instead of +BATT ensures that the pyro MOSFETs get RPP too, but it also theoretically allows you to light e-matches when the board is only powered from the USB port. Don't actually light e-matches with your laptop! Use a high-value resistor for testing instead."
- moved on the sheet: C4, C6, C8, L1, R12, R13, R9, TP1, U4

Commit message: Moved power monitor to seperate I2C bus for easier routing
Connections:
- net I2C0_SCL renamed I2C1_SCL
- net I2C0_SDA renamed I2C1_SDA
Changed lines of the file:
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@@
 		)
 	)
-	(hierarchical_label "I2C0_SCL"
+	(hierarchical_label "I2C1_SCL"
 		(shape input)
 		(at 241.3 137.16 0)
@@
 		)
 	)
-	(hierarchical_label "I2C0_SDA"
+	(hierarchical_label "I2C1_SDA"
 		(shape bidirectional)
 		(at 241.3 134.62 0)

Commit message: final production files
Parts:
- R8: DK Part (none) -> https://www.digikey.com/en/products/detail/littelfuse-inc/L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
Connections:
- net GND: now also U5.7 (A0)
- no-connect marks 4 -> 3
Changed lines of the file:
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@@
 		(at 52.07 59.69)
 	)
-	(no_connect
-		(at 233.68 144.78)
-	)
 	(wire
 		(pts
@@
 	(wire
 		(pts
+			(xy 236.22 146.05) (xy 236.22 144.78)
+		)
+		(stroke
+			(width 0)
+			(type default)
+		)
+	)
+	(wire
+		(pts
 			(xy 52.07 29.21) (xy 64.77 29.21)
 		)
@@
 	(wire
 		(pts
+			(xy 236.22 144.78) (xy 233.68 144.78)
+		)
+		(stroke
+			(width 0)
+			(type default)
+		)
+	)
+	(wire
+		(pts
 			(xy 218.44 49.53) (xy 231.14 49.53)
 		)
@@
 			)
 		)
+		(property "DK Part" "https://www.digikey.com/en/products/detail/littelfuse-inc/L4CA0612LR010FNR/18795242"
+			(at 166.37 128.27 90)
+			(effects
+				(font
+					(size 1.27 1.27)
+				)
+				(hide yes)
+			)
+		)
 		(pin "4"
 		)
@@
 					(unit 1)
 				)
+			)
+		)
+	)
+	(symbol
+		(lib_name "GND_4")
+		(lib_id "power:GND")
+		(at 236.22 146.05 0)
+		(unit 1)
+		(exclude_from_sim no)
+		(in_bom yes)
+		(on_board yes)
+		(dnp no)
+		(fields_autoplaced yes)
+		(property "Reference" "#PWR041"
+			(at 236.22 152.4 0)
+			(effects
+				(font
+					(size 1.27 1.27)
+				)
+				(hide yes)
+			)
+		)
+		(property "Value" "GND"
+			(at 236.22 151.13 0)
+			(effects
+				(font
+					(size 1.27 1.27)
+				)
+			)
+		)
+		(property "Footprint" ""
+			(at 236.22 146.05 0)
+			(effects
+				(font
+					(size 1.27 1.27)
+				)
+				(hide yes)
+			)
+		)
+		(property "Datasheet" ""
+			(at 236.22 146.05 0)
+			(effects
+				(font
+					(size 1.27 1.27)
+				)
+				(hide yes)
+			)
+		)
+		(property "Description" "Power symbol creates a global label with name \"GND\" , ground"
+			(at 236.22 146.05 0)
+			(effects
+				(font
+					(size 1.27 1.27)
+				)
+				(hide yes)
+			)
+		)
+		(pin "1"
+		)
+		(instances
+			(project ""
+				(path "/2b49a1e7-3a95-411d-8c49-438ba0d49dde/420394b1-4c9b-4d8d-83f2-b66955e186e4"
+					(reference "#PWR041")
+					(unit 1)
+				)

Commit message: Final production files (again)
Parts:
- R8: footprint Resistor_SMD:R_Shunt_Vishay_WSKW0612 -> LRI_Partlib:L4CA0612L0M50FNR
Connections:
- net +PBP: now also R8.3; no longer R8.4
- net PWROR: now also R8.2; no longer R8.1
- net at R10.1: now also R8.4; no longer R8.3
- net at R11.1: now also R8.1; no longer R8.2
Changed lines of the file:
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@@
 	(wire
 		(pts
+			(xy 156.21 132.08) (xy 163.83 132.08)
+		)
+		(stroke
+			(width 0)
+			(type default)
+		)
+	)
+	(wire
+		(pts
 			(xy 59.69 60.96) (xy 81.28 60.96)
 		)
@@
 	(wire
 		(pts
+			(xy 160.02 144.78) (xy 176.53 144.78)
+		)
+		(stroke
+			(width 0)
+			(type default)
+		)
+	)
+	(wire
+		(pts
 			(xy 90.17 156.21) (xy 90.17 161.29)
 		)
@@
 	(wire
 		(pts
-			(xy 156.21 128.27) (xy 161.29 128.27)
+			(xy 172.72 128.27) (xy 172.72 134.62)
 		)
 		(stroke
@@
 	(wire
 		(pts
-			(xy 90.17 38.1) (xy 90.17 39.37)
+			(xy 161.29 128.27) (xy 160.02 128.27)
 		)
 		(stroke
@@
 	(wire
 		(pts
-			(xy 86.36 53.34) (xy 86.36 55.88)
+			(xy 90.17 38.1) (xy 90.17 39.37)
 		)
 		(stroke
@@
 	(wire
 		(pts
-			(xy 187.96 52.07) (xy 175.26 52.07)
+			(xy 86.36 53.34) (xy 86.36 55.88)
 		)
 		(stroke
@@
 	(wire
 		(pts
-			(xy 57.15 63.5) (xy 57.15 46.99)
+			(xy 187.96 52.07) (xy 175.26 52.07)
 		)
 		(stroke
@@
 	(wire
 		(pts
-			(xy 91.44 60.96) (xy 106.68 60.96)
+			(xy 57.15 63.5) (xy 57.15 46.99)
 		)
 		(stroke
@@
 	(wire
 		(pts
-			(xy 233.68 134.62) (xy 241.3 134.62)
+			(xy 91.44 60.96) (xy 106.68 60.96)
 		)
 		(stroke
@@
 	(wire
 		(pts
-			(xy 163.83 132.08) (xy 163.83 144.78)
+			(xy 233.68 134.62) (xy 241.3 134.62)
 		)
 		(stroke
@@
 	(wire
 		(pts
-			(xy 156.21 124.46) (xy 156.21 128.27)
+			(xy 156.21 124.46) (xy 156.21 132.08)
 		)
 		(stroke
@@
 	(wire
 		(pts
-			(xy 168.91 134.62) (xy 176.53 134.62)
+			(xy 125.73 93.98) (xy 129.54 93.98)
 		)
 		(stroke
@@
 	(wire
 		(pts
-			(xy 125.73 93.98) (xy 129.54 93.98)
+			(xy 125.73 90.17) (xy 125.73 93.98)
 		)
 		(stroke
@@
 	(wire
 		(pts
-			(xy 125.73 90.17) (xy 125.73 93.98)
+			(xy 116.84 104.14) (xy 116.84 105.41)
 		)
 		(stroke
@@
 	(wire
 		(pts
-			(xy 116.84 104.14) (xy 116.84 105.41)
+			(xy 172.72 134.62) (xy 176.53 134.62)
 		)
 		(stroke
@@
 	(wire
 		(pts
-			(xy 176.53 124.46) (xy 176.53 128.27)
+			(xy 176.53 124.46) (xy 176.53 132.08)
 		)
 		(stroke
@@
 	(wire
 		(pts
+			(xy 171.45 128.27) (xy 172.72 128.27)
+		)
+		(stroke
+			(width 0)
+			(type default)
+		)
+	)
+	(wire
+		(pts
 			(xy 74.93 44.45) (xy 74.93 43.18)
 		)
@@
 	(wire
 		(pts
-			(xy 171.45 128.27) (xy 176.53 128.27)
+			(xy 53.34 41.91) (xy 52.07 41.91)
 		)
 		(stroke
@@
 	(wire
 		(pts
-			(xy 53.34 41.91) (xy 52.07 41.91)
+			(xy 168.91 132.08) (xy 176.53 132.08)
 		)
 		(stroke
@@
 	(wire
 		(pts
-			(xy 163.83 144.78) (xy 176.53 144.78)
+			(xy 55.88 147.32) (xy 55.88 157.48)
 		)
 		(stroke
@@
 	(wire
 		(pts
-			(xy 55.88 147.32) (xy 55.88 157.48)
+			(xy 255.27 60.96) (xy 255.27 62.23)
 		)
 		(stroke
@@
 	(wire
 		(pts
-			(xy 255.27 60.96) (xy 255.27 62.23)
+			(xy 105.41 38.1) (xy 105.41 39.37)
 		)
 		(stroke
@@
 	(wire
 		(pts
-			(xy 105.41 38.1) (xy 105.41 39.37)
+			(xy 80.01 139.7) (xy 95.25 139.7)
 		)
 		(stroke
@@
 	(wire
 		(pts
-			(xy 80.01 139.7) (xy 95.25 139.7)
+			(xy 175.26 41.91) (xy 175.26 43.18)
 		)
 		(stroke
@@
 	(wire
 		(pts
-			(xy 175.26 41.91) (xy 175.26 43.18)
+			(xy 160.02 128.27) (xy 160.02 144.78)
 		)
 		(stroke
@@
 	(wire
 		(pts
-			(xy 168.91 132.08) (xy 168.91 134.62)
-		)
-		(stroke
-			(width 0)
-			(type default)
-		)
-	)
-	(wire
-		(pts
 			(xy 118.11 29.21) (xy 105.41 29.21)
 		)
@@
 			)
 		)
-		(property "Footprint" "Resistor_SMD:R_Shunt_Vishay_WSKW0612"
+		(property "Footprint" "LRI_Partlib:L4CA0612L0M50FNR"
 			(at 166.37 126.492 90)
 			(effects
