File: flight-computer-one.kicad_sch (KiCad schematic)
At the start: 4 parts

Commit message: the beginnings of a footprint
Parts:
- added J3, J4: Screw_Terminal_01x08, TerminalBlock_Phoenix:TerminalBlock_Phoenix_MKDS-1,5-8_1x08_P5.00mm_Horizontal, symbol Connector:Screw_Terminal_01x08
Other:
- sheet Networking renamed Connectivity
- sheet Connectivity: file networking.kicad_sch -> connectivity.kicad_sch
Changed lines of the file:
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@@
+		)
+	)
+	(symbol
+		(lib_id "Connector:Screw_Terminal_01x08")
+		(at 185.42 170.18 0)
+		(unit 1)
+		(exclude_from_sim no)
+		(in_bom yes)
+		(on_board yes)
+		(dnp no)
+		(fields_autoplaced yes)
+		(property "Reference" "J3"
+			(at 187.96 170.1799 0)
+			(effects
+				(font
+					(size 1.27 1.27)
+				)
+				(justify left)
+			)
+		)
+		(property "Value" "Screw_Terminal_01x08"
+			(at 187.96 172.7199 0)
+			(effects
+				(font
+					(size 1.27 1.27)
+				)
+				(justify left)
+			)
+		)
+		(property "Footprint" "TerminalBlock_Phoenix:TerminalBlock_Phoenix_MKDS-1,5-8_1x08_P5.00mm_Horizontal"
+			(at 185.42 170.18 0)
+			(effects
+				(font
+					(size 1.27 1.27)
+				)
+				(hide yes)
+			)
+		)
+		(property "Datasheet" "~"
+			(at 185.42 170.18 0)
+			(effects
+				(font
+					(size 1.27 1.27)
+				)
+				(hide yes)
+			)
+		)
+		(property "Description" "Generic screw terminal, single row, 01x08, script generated (kicad-library-utils/schlib/autogen/connector/)"
+			(at 185.42 170.18 0)
+			(effects
+				(font
+					(size 1.27 1.27)
+				)
+				(hide yes)
+			)
+		)
+		(pin "2"
+		)
+		(pin "5"
+		)
+		(pin "4"
+		)
+		(pin "1"
+		)
+		(pin "3"
+		)
+		(pin "6"
+		)
+		(pin "7"
+		)
+		(pin "8"
+		)
+		(instances
+			(project ""
+				(path "/2b49a1e7-3a95-411d-8c49-438ba0d49dde"
+					(reference "J3")
+					(unit 1)
+				)
+			)
+		)
+	)
+	(symbol
+		(lib_id "Connector:Screw_Terminal_01x08")
+		(at 237.49 170.18 0)
+		(mirror y)
+		(unit 1)
+		(exclude_from_sim no)
+		(in_bom yes)
+		(on_board yes)
+		(dnp no)
+		(fields_autoplaced yes)
+		(property "Reference" "J4"
+			(at 234.95 170.1799 0)
+			(effects
+				(font
+					(size 1.27 1.27)
+				)
+				(justify left)
+			)
+		)
+		(property "Value" "Screw_Terminal_01x08"
+			(at 234.95 172.7199 0)
+			(effects
+				(font
+					(size 1.27 1.27)
+				)
+				(justify left)
+			)
+		)
+		(property "Footprint" "TerminalBlock_Phoenix:TerminalBlock_Phoenix_MKDS-1,5-8_1x08_P5.00mm_Horizontal"
+			(at 237.49 170.18 0)
+			(effects
+				(font
+					(size 1.27 1.27)
+				)
+				(hide yes)
+			)
+		)
+		(property "Datasheet" "~"
+			(at 237.49 170.18 0)
+			(effects
+				(font
+					(size 1.27 1.27)
+				)
+				(hide yes)
+			)
+		)
+		(property "Description" "Generic screw terminal, single row, 01x08, script generated (kicad-library-utils/schlib/autogen/connector/)"
+			(at 237.49 170.18 0)
+			(effects
+				(font
+					(size 1.27 1.27)
+				)
+				(hide yes)
+			)
+		)
+		(pin "2"
+		)
+		(pin "5"
+		)
+		(pin "4"
+		)
+		(pin "1"
+		)
+		(pin "3"
+		)
+		(pin "6"
+		)
+		(pin "7"
+		)
+		(pin "8"
+		)
+		(instances
+			(project "flight-computer-one"
+				(path "/2b49a1e7-3a95-411d-8c49-438ba0d49dde"
+					(reference "J4")
+					(unit 1)
+				)
+			)
 		)
 	)
@@
 			(color 0 0 0 0.0000)
 		)
-		(property "Sheetname" "Networking"
+		(property "Sheetname" "Connectivity"
 			(at 180.34 31.0384 0)
 			(effects
@@
 			)
 		)
-		(property "Sheetfile" "networking.kicad_sch"
+		(property "Sheetfile" "connectivity.kicad_sch"
 			(at 180.34 98.3746 0)
 			(effects

Commit message: created project lib
Parts:
- renumbered J3 to J1, J4 to J2
Other:
- sheet Servos and Pyros renamed Servos & Pyros
- added sheet Power & USB (power_usb.kicad_sch)
- moved on the sheet: H1, H2, H3, H4, J1, J2
Changed lines of the file:
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@@
 	(generator "eeschema")
 	(generator_version "9.0")
-	(paper "A3")
+	(paper "A4")
 	(symbol
 		(lib_id "Mechanical:MountingHole")
-		(at 322.58 195.58 0)
+		(at 26.67 255.27 0)
 		(unit 1)
 		(exclude_from_sim no)
@@
 		(dnp no)
 		(property "Reference" "H1"
-			(at 325.12 194.4116 0)
+			(at 29.21 254.1016 0)
 			(effects
 				(font
@@
 		)
 		(property "Value" "MountingHole"
-			(at 325.12 196.723 0)
+			(at 29.21 256.413 0)
 			(effects
 				(font
@@
 		)
 		(property "Footprint" "MountingHole:MountingHole_3.2mm_M3"
-			(at 322.58 195.58 0)
+			(at 26.67 255.27 0)
 			(effects
 				(font
@@
 		)
 		(property "Datasheet" "~"
-			(at 322.58 195.58 0)
+			(at 26.67 255.27 0)
 			(effects
 				(font
@@
 		)
 		(property "Description" ""
-			(at 322.58 195.58 0)
+			(at 26.67 255.27 0)
 			(effects
 				(font
@@
 	(symbol
 		(lib_id "Mechanical:MountingHole")
-		(at 322.58 200.66 0)
+		(at 26.67 260.35 0)
 		(unit 1)
 		(exclude_from_sim no)
@@
 		(dnp no)
 		(property "Reference" "H2"
-			(at 325.12 199.4916 0)
+			(at 29.21 259.1816 0)
 			(effects
 				(font
@@
 		)
 		(property "Value" "MountingHole"
-			(at 325.12 201.803 0)
+			(at 29.21 261.493 0)
 			(effects
 				(font
@@
 		)
 		(property "Footprint" "MountingHole:MountingHole_3.2mm_M3"
-			(at 322.58 200.66 0)
+			(at 26.67 260.35 0)
 			(effects
 				(font
@@
 		)
 		(property "Datasheet" "~"
-			(at 322.58 200.66 0)
+			(at 26.67 260.35 0)
 			(effects
 				(font
@@
 		)
 		(property "Description" ""
-			(at 322.58 200.66 0)
+			(at 26.67 260.35 0)
 			(effects
 				(font
@@
 	(symbol
 		(lib_id "Mechanical:MountingHole")
-		(at 322.58 205.74 0)
+		(at 26.67 265.43 0)
 		(unit 1)
 		(exclude_from_sim no)
@@
 		(dnp no)
 		(property "Reference" "H3"
-			(at 325.12 204.5716 0)
+			(at 29.21 264.2616 0)
 			(effects
 				(font
@@
 		)
 		(property "Value" "MountingHole"
-			(at 325.12 206.883 0)
+			(at 29.21 266.573 0)
 			(effects
 				(font
@@
 		)
 		(property "Footprint" "MountingHole:MountingHole_3.2mm_M3"
-			(at 322.58 205.74 0)
+			(at 26.67 265.43 0)
 			(effects
 				(font
@@
 		)
 		(property "Datasheet" "~"
-			(at 322.58 205.74 0)
+			(at 26.67 265.43 0)
 			(effects
 				(font
@@
 		)
 		(property "Description" ""
-			(at 322.58 205.74 0)
+			(at 26.67 265.43 0)
 			(effects
 				(font
@@
 	(symbol
 		(lib_id "Mechanical:MountingHole")
-		(at 322.58 210.82 0)
+		(at 26.67 270.51 0)
 		(unit 1)
 		(exclude_from_sim no)
@@
 		(dnp no)
 		(property "Reference" "H4"
-			(at 325.12 209.55 0)
+			(at 29.21 269.24 0)
 			(effects
 				(font
@@
 		)
 		(property "Value" "MountingHole"
-			(at 325.12 211.963 0)
+			(at 29.21 271.653 0)
 			(effects
 				(font
@@
 		)
 		(property "Footprint" "MountingHole:MountingHole_3.2mm_M3"
-			(at 322.58 210.82 0)
+			(at 26.67 270.51 0)
 			(effects
 				(font
@@
 		)
 		(property "Datasheet" "~"
-			(at 322.58 210.82 0)
+			(at 26.67 270.51 0)
 			(effects
 				(font
@@
 		)
 		(property "Description" ""
-			(at 322.58 210.82 0)
+			(at 26.67 270.51 0)
 			(effects
 				(font
@@
 	(symbol
 		(lib_id "Connector:Screw_Terminal_01x08")
-		(at 185.42 170.18 0)
+		(at 86.36 166.37 0)
 		(unit 1)
 		(exclude_from_sim no)
@@
 		(dnp no)
 		(fields_autoplaced yes)
-		(property "Reference" "J3"
-			(at 187.96 170.1799 0)
+		(property "Reference" "J1"
+			(at 88.9 166.3699 0)
 			(effects
 				(font
@@
 		)
 		(property "Value" "Screw_Terminal_01x08"
-			(at 187.96 172.7199 0)
+			(at 88.9 168.9099 0)
 			(effects
 				(font
@@
 		)
 		(property "Footprint" "TerminalBlock_Phoenix:TerminalBlock_Phoenix_MKDS-1,5-8_1x08_P5.00mm_Horizontal"
-			(at 185.42 170.18 0)
+			(at 86.36 166.37 0)
 			(effects
 				(font
@@
 		)
 		(property "Datasheet" "~"
-			(at 185.42 170.18 0)
+			(at 86.36 166.37 0)
 			(effects
 				(font
@@
 		)
 		(property "Description" "Generic screw terminal, single row, 01x08, script generated (kicad-library-utils/schlib/autogen/connector/)"
-			(at 185.42 170.18 0)
+			(at 86.36 166.37 0)
 			(effects
 				(font
@@
 			(project ""
 				(path "/2b49a1e7-3a95-411d-8c49-438ba0d49dde"
-					(reference "J3")
+					(reference "J1")
 					(unit 1)
 				)
@@
 	(symbol
 		(lib_id "Connector:Screw_Terminal_01x08")
-		(at 237.49 170.18 0)
+		(at 140.97 166.37 0)
 		(mirror y)
 		(unit 1)
@@
 		(dnp no)
 		(fields_autoplaced yes)
-		(property "Reference" "J4"
-			(at 234.95 170.1799 0)
+		(property "Reference" "J2"
+			(at 138.43 166.3699 0)
 			(effects
 				(font
@@
 		)
 		(property "Value" "Screw_Terminal_01x08"
-			(at 234.95 172.7199 0)
+			(at 138.43 168.9099 0)
 			(effects
 				(font
@@
 		)
 		(property "Footprint" "TerminalBlock_Phoenix:TerminalBlock_Phoenix_MKDS-1,5-8_1x08_P5.00mm_Horizontal"
-			(at 237.49 170.18 0)
+			(at 140.97 166.37 0)
 			(effects
 				(font
@@
 		)
 		(property "Datasheet" "~"
-			(at 237.49 170.18 0)
+			(at 140.97 166.37 0)
 			(effects
 				(font
@@
 		)
 		(property "Description" "Generic screw terminal, single row, 01x08, script generated (kicad-library-utils/schlib/autogen/connector/)"
-			(at 237.49 170.18 0)
+			(at 140.97 166.37 0)
 			(effects
 				(font
@@
 			(project "flight-computer-one"
 				(path "/2b49a1e7-3a95-411d-8c49-438ba0d49dde"
-					(reference "J4")
+					(reference "J2")
 					(unit 1)
 				)
@@
 	(sheet
 		(at 34.29 30.48)
-		(size 60.96 67.31)
+		(size 41.91 66.04)
 		(exclude_from_sim no)
 		(in_bom yes)
@@
 		)
 		(property "Sheetfile" "compute.kicad_sch"
-			(at 34.29 98.3746 0)
+			(at 34.29 97.1046 0)
 			(effects
 				(font
@@
 			(project "flight-computer-one"
 				(path "/2b49a1e7-3a95-411d-8c49-438ba0d49dde"
-					(page "2")
+					(page "3")
 				)
 			)
@@
 	)
 	(sheet
-		(at 180.34 31.75)
-		(size 60.96 66.04)
+		(at 139.7 99.06)
+		(size 38.1 30.48)
 		(exclude_from_sim no)
 		(in_bom yes)
@@
 		)
 		(property "Sheetname" "Connectivity"
-			(at 180.34 31.0384 0)
+			(at 139.7 98.3484 0)
 			(effects
 				(font
@@
 		)
 		(property "Sheetfile" "connectivity.kicad_sch"
-			(at 180.34 98.3746 0)
+			(at 139.7 130.1246 0)
 			(effects
 				(font
@@
 			(project "flight-computer-one"
 				(path "/2b49a1e7-3a95-411d-8c49-438ba0d49dde"
-					(page "4")
+					(page "5")
 				)
 			)
@@
 	)
 	(sheet
-		(at 255.27 31.75)
-		(size 55.88 66.04)
+		(at 107.95 30.48)
+		(size 49.53 36.83)
 		(exclude_from_sim no)
 		(in_bom yes)
@@
 			(color 0 0 0 0.0000)
 		)
-		(property "Sheetname" "Servos and Pyros"
-			(at 255.27 31.0384 0)
+		(property "Sheetname" "Power & USB"
+			(at 107.95 29.7684 0)
 			(effects
 				(font
@@
 			)
 		)
-		(property "Sheetfile" "servo_pyro.kicad_sch"
-			(at 255.27 98.3746 0)
+		(property "Sheetfile" "power_usb.kicad_sch"
+			(at 107.95 67.8946 0)
 			(effects
 				(font
@@
 			(project "flight-computer-one"
 				(path "/2b49a1e7-3a95-411d-8c49-438ba0d49dde"
-					(page "5")
+					(page "2")
 				)
 			)
@@
 	)
 	(sheet
-		(at 107.95 30.48)
-		(size 58.42 67.31)
+		(at 210.82 53.34)
+		(size 38.1 35.56)
 		(exclude_from_sim no)
 		(in_bom yes)
@@
 			(color 0 0 0 0.0000)
 		)
+		(property "Sheetname" "Servos & Pyros"
+			(at 210.82 52.6284 0)
+			(effects
+				(font
+					(size 1.27 1.27)
+				)
+				(justify left bottom)
+			)
+		)
+		(property "Sheetfile" "servo_pyro.kicad_sch"
+			(at 210.82 89.4846 0)
+			(effects
+				(font
+					(size 1.27 1.27)
+				)
+				(justify left top)
+			)
+		)
+		(instances
+			(project "flight-computer-one"
+				(path "/2b49a1e7-3a95-411d-8c49-438ba0d49dde"
+					(page "6")
+				)
+			)
+		)
+	)
+	(sheet
+		(at 83.82 97.79)
+		(size 44.45 43.18)
+		(exclude_from_sim no)
+		(in_bom yes)
+		(on_board yes)
+		(dnp no)
+		(fields_autoplaced yes)
+		(stroke
+			(width 0.1524)
+			(type solid)
+		)
+		(fill
+			(color 0 0 0 0.0000)
+		)
 		(property "Sheetname" "Sensors"
-			(at 107.95 29.7684 0)
+			(at 83.82 97.0784 0)
 			(effects
 				(font
@@
 		)
 		(property "Sheetfile" "sensors.kicad_sch"
-			(at 107.95 98.3746 0)
+			(at 83.82 141.5546 0)
 			(effects
 				(font
@@
 			(project "flight-computer-one"
 				(path "/2b49a1e7-3a95-411d-8c49-438ba0d49dde"
-					(page "3")
-				)
-			)
+					(page "4")
+				)
+			)

Commit message: nearly completed schematic, partial layout
Other:
- moved on the sheet: H1, H2, H3, H4
Changed lines of the file:
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@@
 	(symbol
 		(lib_id "Mechanical:MountingHole")
-		(at 26.67 255.27 0)
+		(at 24.13 173.99 0)
 		(unit 1)
 		(exclude_from_sim no)
@@
 		(dnp no)
 		(property "Reference" "H1"
-			(at 29.21 254.1016 0)
-			(effects
-				(font
-					(size 1.27 1.27)
-				)
-				(justify left)
-			)
-		)
-		(property "Value" "MountingHole"
-			(at 29.21 256.413 0)
-			(effects
-				(font
-					(size 1.27 1.27)
-				)
-				(justify left)
-			)
-		)
-		(property "Footprint" "MountingHole:MountingHole_3.2mm_M3"
-			(at 26.67 255.27 0)
-			(effects
-				(font
-					(size 1.27 1.27)
-				)
-				(hide yes)
-			)
-		)
-		(property "Datasheet" "~"
-			(at 26.67 255.27 0)
-			(effects
-				(font
-					(size 1.27 1.27)
-				)
-				(hide yes)
-			)
-		)
-		(property "Description" ""
-			(at 26.67 255.27 0)
+			(at 26.67 172.8216 0)
+			(effects
+				(font
+					(size 1.27 1.27)
+				)
+				(justify left)
+			)
+		)
+		(property "Value" "MountingHole"
+			(at 26.67 175.133 0)
+			(effects
+				(font
+					(size 1.27 1.27)
+				)
+				(justify left)
+			)
+		)
+		(property "Footprint" "MountingHole:MountingHole_3.2mm_M3"
+			(at 24.13 173.99 0)
+			(effects
+				(font
+					(size 1.27 1.27)
+				)
+				(hide yes)
+			)
+		)
+		(property "Datasheet" "~"
+			(at 24.13 173.99 0)
+			(effects
+				(font
+					(size 1.27 1.27)
+				)
+				(hide yes)
+			)
+		)
+		(property "Description" ""
+			(at 24.13 173.99 0)
 			(effects
 				(font
@@
 	(symbol
 		(lib_id "Mechanical:MountingHole")
-		(at 26.67 260.35 0)
+		(at 24.13 179.07 0)
 		(unit 1)
 		(exclude_from_sim no)
@@
 		(dnp no)
 		(property "Reference" "H2"
-			(at 29.21 259.1816 0)
-			(effects
-				(font
-					(size 1.27 1.27)
-				)
-				(justify left)
-			)
-		)
-		(property "Value" "MountingHole"
-			(at 29.21 261.493 0)
-			(effects
-				(font
-					(size 1.27 1.27)
-				)
-				(justify left)
-			)
-		)
-		(property "Footprint" "MountingHole:MountingHole_3.2mm_M3"
-			(at 26.67 260.35 0)
-			(effects
-				(font
-					(size 1.27 1.27)
-				)
-				(hide yes)
-			)
-		)
-		(property "Datasheet" "~"
-			(at 26.67 260.35 0)
-			(effects
-				(font
-					(size 1.27 1.27)
-				)
-				(hide yes)
-			)
-		)
-		(property "Description" ""
-			(at 26.67 260.35 0)
+			(at 26.67 177.9016 0)
+			(effects
+				(font
+					(size 1.27 1.27)
+				)
+				(justify left)
+			)
+		)
+		(property "Value" "MountingHole"
+			(at 26.67 180.213 0)
+			(effects
+				(font
+					(size 1.27 1.27)
+				)
+				(justify left)
+			)
+		)
+		(property "Footprint" "MountingHole:MountingHole_3.2mm_M3"
+			(at 24.13 179.07 0)
+			(effects
+				(font
+					(size 1.27 1.27)
+				)
+				(hide yes)
+			)
+		)
+		(property "Datasheet" "~"
+			(at 24.13 179.07 0)
+			(effects
+				(font
+					(size 1.27 1.27)
+				)
+				(hide yes)
+			)
+		)
+		(property "Description" ""
+			(at 24.13 179.07 0)
 			(effects
 				(font
@@
 	(symbol
 		(lib_id "Mechanical:MountingHole")
-		(at 26.67 265.43 0)
+		(at 24.13 184.15 0)
 		(unit 1)
 		(exclude_from_sim no)
@@
 		(dnp no)
 		(property "Reference" "H3"
-			(at 29.21 264.2616 0)
-			(effects
-				(font
-					(size 1.27 1.27)
-				)
-				(justify left)
-			)
-		)
-		(property "Value" "MountingHole"
-			(at 29.21 266.573 0)
-			(effects
-				(font
-					(size 1.27 1.27)
-				)
-				(justify left)
-			)
-		)
-		(property "Footprint" "MountingHole:MountingHole_3.2mm_M3"
-			(at 26.67 265.43 0)
-			(effects
-				(font
-					(size 1.27 1.27)
-				)
-				(hide yes)
-			)
-		)
-		(property "Datasheet" "~"
-			(at 26.67 265.43 0)
-			(effects
-				(font
-					(size 1.27 1.27)
-				)
-				(hide yes)
-			)
-		)
-		(property "Description" ""
-			(at 26.67 265.43 0)
+			(at 26.67 182.9816 0)
+			(effects
+				(font
+					(size 1.27 1.27)
+				)
+				(justify left)
+			)
+		)
+		(property "Value" "MountingHole"
+			(at 26.67 185.293 0)
+			(effects
+				(font
+					(size 1.27 1.27)
+				)
+				(justify left)
+			)
+		)
+		(property "Footprint" "MountingHole:MountingHole_3.2mm_M3"
+			(at 24.13 184.15 0)
+			(effects
+				(font
+					(size 1.27 1.27)
+				)
+				(hide yes)
+			)
+		)
+		(property "Datasheet" "~"
+			(at 24.13 184.15 0)
+			(effects
+				(font
+					(size 1.27 1.27)
+				)
+				(hide yes)
+			)
+		)
+		(property "Description" ""
+			(at 24.13 184.15 0)
 			(effects
 				(font
@@
 	(symbol
 		(lib_id "Mechanical:MountingHole")
-		(at 26.67 270.51 0)
+		(at 24.13 189.23 0)
 		(unit 1)
 		(exclude_from_sim no)
@@
 		(dnp no)
 		(property "Reference" "H4"
-			(at 29.21 269.24 0)
-			(effects
-				(font
-					(size 1.27 1.27)
-				)
-				(justify left)
-			)
-		)
-		(property "Value" "MountingHole"
-			(at 29.21 271.653 0)
-			(effects
-				(font
-					(size 1.27 1.27)
-				)
-				(justify left)
-			)
-		)
-		(property "Footprint" "MountingHole:MountingHole_3.2mm_M3"
-			(at 26.67 270.51 0)
-			(effects
-				(font
-					(size 1.27 1.27)
-				)
-				(hide yes)
-			)
-		)
-		(property "Datasheet" "~"
-			(at 26.67 270.51 0)
-			(effects
-				(font
-					(size 1.27 1.27)
-				)
-				(hide yes)
-			)
-		)
-		(property "Description" ""
-			(at 26.67 270.51 0)
-			(effects
-				(font
+			(at 26.67 187.96 0)
+			(effects
+				(font
+					(size 1.27 1.27)
+				)
+				(justify left)
+			)
+		)
+		(property "Value" "MountingHole"
+			(at 26.67 190.373 0)
+			(effects
+				(font
+					(size 1.27 1.27)
+				)
+				(justify left)
+			)
+		)
+		(property "Footprint" "MountingHole:MountingHole_3.2mm_M3"
+			(at 24.13 189.23 0)
+			(effects
+				(font
+					(size 1.27 1.27)
+				)
+				(hide yes)
+			)
+		)
+		(property "Datasheet" "~"
+			(at 24.13 189.23 0)
+			(effects
+				(font
+					(size 1.27 1.27)
+				)
+				(hide yes)
+			)
+		)
+		(property "Description" ""
+			(at 24.13 189.23 0)
+			(effects
+				(font

Commit message: schematic + prelim layout nearly complete
Parts:
- J1: value Screw_Terminal_01x08 -> LEFT_BANK
- J2: value Screw_Terminal_01x08 -> RIGHT_BANK
Connections:
- net +PBP: now reaches J1.1 (Pin_1)
- net +PBP: now also J1.3 (Pin_3), J2.6 (Pin_6), J2.8 (Pin_8)
- net GND: now reaches J1.2 (Pin_2)
- net GND: now also J1.4 (Pin_4), J2.2 (Pin_2)
- net SERVO1_CTL: now reaches J1.5 (Pin_5)
- net SERVO2_CTL: now reaches J1.6 (Pin_6)
- net SERVO3_CTL: now reaches J1.7 (Pin_7)
- net SERVO4_CTL: now reaches J1.8 (Pin_8)
- net GPIO40_ADC0: now reaches J2.1 (Pin_1)
- net CANL: now reaches J2.3 (Pin_3)
- net CANH: now reaches J2.4 (Pin_4)
- net PYRO2_DRAIN: now reaches J2.5 (Pin_5)
- net PYRO1_DRAIN: now reaches J2.7 (Pin_7)
Other:
- moved on the sheet: J2

Commit message: Schematic tentatively complete
Connections:
- net +PBP: no longer J1.1 (Pin_1)
- new net +BATT: J1.1 (Pin_1)
Changed lines of the file:
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@@
 	(paper "A4")
-	(junction
-		(at 60.96 158.75)
-		(diameter 0)
-		(color 0 0 0 0)
-	)
 	(junction
 		(at 142.24 158.75)
@@
 	(wire
 		(pts
-			(xy 60.96 163.83) (xy 60.96 158.75)
-		)
-		(stroke
-			(width 0)
-			(type default)
-		)
-	)
-	(wire
-		(pts
 			(xy 121.92 163.83) (xy 142.24 163.83)
 		)
@@
 	(wire
 		(pts
-			(xy 144.78 173.99) (xy 121.92 173.99)
+			(xy 142.24 173.99) (xy 121.92 173.99)
 		)
 		(stroke
@@
 	(wire
 		(pts
-			(xy 81.28 163.83) (xy 60.96 163.83)
-		)
-		(stroke
-			(width 0)
-			(type default)
-		)
-	)
-	(wire
-		(pts
 			(xy 66.04 171.45) (xy 81.28 171.45)
 		)
@@
 	(wire
 		(pts
-			(xy 144.78 179.07) (xy 144.78 173.99)
+			(xy 142.24 179.07) (xy 142.24 173.99)
 		)
 		(stroke
@@
 	(wire
 		(pts
+			(xy 52.07 163.83) (xy 81.28 163.83)
+		)
+		(stroke
+			(width 0)
+			(type default)
+		)
+	)
+	(wire
+		(pts
 			(xy 121.92 166.37) (xy 137.16 166.37)
 		)
@@
 		(pts
 			(xy 81.28 168.91) (xy 66.04 168.91)
+		)
+		(stroke
+			(width 0)
+			(type default)
+		)
+	)
+	(wire
+		(pts
+			(xy 52.07 154.94) (xy 52.07 163.83)
 		)
 		(stroke
@@
 	)
 	(symbol
+		(lib_id "power:+BATT")
+		(at 60.96 154.94 0)
+		(unit 1)
+		(exclude_from_sim no)
+		(in_bom yes)
+		(on_board yes)
+		(dnp no)
+		(fields_autoplaced yes)
+		(property "Reference" "#PWR0103"
+			(at 60.96 158.75 0)
+			(effects
+				(font
+					(size 1.27 1.27)
+				)
+				(hide yes)
+			)
+		)
+		(property "Value" "+BATT"
+			(at 60.96 149.86 0)
+			(effects
+				(font
+					(size 1.27 1.27)
+				)
+			)
+		)
+		(property "Footprint" ""
+			(at 60.96 154.94 0)
+			(effects
+				(font
+					(size 1.27 1.27)
+				)
+				(hide yes)
+			)
+		)
+		(property "Datasheet" ""
+			(at 60.96 154.94 0)
+			(effects
+				(font
+					(size 1.27 1.27)
+				)
+				(hide yes)
+			)
+		)
+		(property "Description" "Power symbol creates a global label with name \"+BATT\""
+			(at 60.96 154.94 0)
+			(effects
+				(font
+					(size 1.27 1.27)
+				)
+				(hide yes)
+			)
+		)
+		(pin "1"
+		)
+		(instances
+			(project "flight-computer-one"
+				(path "/2b49a1e7-3a95-411d-8c49-438ba0d49dde"
+					(reference "#PWR0103")
+					(unit 1)
+				)
+			)
+		)
+	)
+	(symbol
 		(lib_id "power:+VSW")
-		(at 60.96 154.94 0)
+		(at 52.07 154.94 0)
 		(mirror y)
 		(unit 1)
@@
 		(fields_autoplaced yes)
 		(property "Reference" "#PWR096"
-			(at 60.96 158.75 0)
+			(at 52.07 158.75 0)
 			(effects
 				(font
@@
 		)
 		(property "Value" "+PBP"
-			(at 60.96 149.86 0)
+			(at 52.07 149.86 0)
 			(effects
 				(font
@@
 		)
 		(property "Footprint" ""
-			(at 60.96 154.94 0)
+			(at 52.07 154.94 0)
 			(effects
 				(font
@@
 		)
 		(property "Datasheet" ""
-			(at 60.96 154.94 0)
+			(at 52.07 154.94 0)
 			(effects
 				(font
@@
 		)
 		(property "Description" "Power symbol creates a global label with name \"+VSW\""
-			(at 60.96 154.94 0)
+			(at 52.07 154.94 0)
 			(effects
 				(font
@@
 	(symbol
 		(lib_id "power:GND")
-		(at 144.78 179.07 0)
+		(at 142.24 179.07 0)
 		(unit 1)
 		(exclude_from_sim no)
@@
 		(fields_autoplaced yes)
 		(property "Reference" "#PWR094"
-			(at 144.78 185.42 0)
+			(at 142.24 185.42 0)
 			(effects
 				(font
@@
 		)
 		(property "Value" "GND"
-			(at 144.78 184.15 0)
+			(at 142.24 184.15 0)
 			(effects
 				(font
@@
 		)
 		(property "Footprint" ""
-			(at 144.78 179.07 0)
+			(at 142.24 179.07 0)
 			(effects
 				(font
@@
 		)
 		(property "Datasheet" ""
-			(at 144.78 179.07 0)
+			(at 142.24 179.07 0)
 			(effects
 				(font
@@
 		)
 		(property "Description" "Power symbol creates a global label with name \"GND\" , ground"
-			(at 144.78 179.07 0)
-			(effects
-				(font
+			(at 142.24 179.07 0)
+			(effects
+				(font

Commit message: schematic tentatively finished
Parts:
- added R11, R12: 1K, Resistor_SMD:R_0603_1608Metric, symbol Device:R
Connections:
- new net +3V3: R11.1, R12.1
- new net Compute/I2C0_SCL: R12.2
- new net Compute/I2C0_SDA: R11.2
Other:
- sheet Compute ports: added BUZZER_CTL, CS_CANXC, CS_IMU_MAIN, CS_RADIO, GPIO40_ADC0, I2C0_SCL, I2C0_SDA, SERVO1_CTL, SERVO2_CTL, SERVO3_CTL, SERVO4_CTL, SPI0_MISO, SPI0_MOSI, SPI0_SCK, TCAN_STB, USB_D+, USB_D-; removed none
- sheet Connectivity ports: added CANH, CANL, CS_CANXC, CS_RADIO, I2C0_SCL, I2C0_SDA, SPI0_MISO, SPI0_MOSI, SPI0_SCK, TCAN_STB; removed none
- sheet Power & USB ports: added I2C0_SCL, I2C0_SDA, USB_D+, USB_D-; removed none
- sheet Sensors ports: added CS_IMU_MAIN, I2C0_SCL, I2C0_SDA, SPI0_MISO, SPI0_MOSI, SPI0_SCK; removed none
- sheet Servos & Pyros ports: added BUZZER_CTL, I2C0_SCL, I2C0_SDA; removed none
