File: flight-computer-one.kicad_sch (KiCad schematic)
At the start: 8 parts, among them J1 LEFT_BANK, J2 RIGHT_BANK

Commit message: Moved ICM to I2C
Other:
- sheet Compute ports: added none; removed CS_IMU_MAIN
- sheet Sensors ports: added none; removed CS_IMU_MAIN, SPI0_MISO, SPI0_MOSI, SPI0_SCK
Changed lines of the file:
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@@
-	)
-	(junction
-		(at 200.66 60.96)
-		(diameter 0)
-		(color 0 0 0 0)
 	)
 	(junction
@@
 	)
 	(junction
-		(at 198.12 63.5)
-		(diameter 0)
-		(color 0 0 0 0)
-	)
-	(junction
 		(at 63.5 147.32)
 		(diameter 0)
@@
 	)
 	(junction
-		(at 195.58 66.04)
-		(diameter 0)
-		(color 0 0 0 0)
-	)
-	(junction
 		(at 210.82 91.44)
 		(diameter 0)
@@
 	(wire
 		(pts
-			(xy 195.58 66.04) (xy 233.68 66.04)
-		)
-		(stroke
-			(width 0)
-			(type default)
-		)
-	)
-	(wire
-		(pts
-			(xy 200.66 60.96) (xy 233.68 60.96)
-		)
-		(stroke
-			(width 0)
-			(type default)
-		)
-	)
-	(wire
-		(pts
 			(xy 173.99 43.18) (xy 173.99 46.99)
 		)
@@
 	(wire
 		(pts
-			(xy 198.12 63.5) (xy 233.68 63.5)
-		)
-		(stroke
-			(width 0)
-			(type default)
-		)
-	)
-	(wire
-		(pts
 			(xy 186.69 121.92) (xy 186.69 100.33)
 		)
@@
 		(pts
 			(xy 63.5 142.24) (xy 63.5 147.32)
-		)
-		(stroke
-			(width 0)
-			(type default)
-		)
-	)
-	(wire
-		(pts
-			(xy 139.7 69.85) (xy 233.68 69.85)
 		)
 		(stroke
@@
 			)
 		)
-		(pin "CS_IMU_MAIN" output
-			(at 139.7 69.85 0)
-			(effects
-				(font
-					(size 1.27 1.27)
-				)
-				(justify right)
-			)
-		)
 		(pin "CS_RADIO" output
 			(at 139.7 72.39 0)
@@
 			(effects
 				(font
-					(size 1.27 1.27)
-				)
-				(justify left)
-			)
-		)
-		(pin "CS_IMU_MAIN" input
-			(at 233.68 69.85 180)
-			(effects
-				(font
-					(size 1.27 1.27)
-				)
-				(justify left)
-			)
-		)
-		(pin "SPI0_MISO" output
-			(at 233.68 66.04 180)
-			(effects
-				(font
-					(size 1.27 1.27)
-				)
-				(justify left)
-			)
-		)
-		(pin "SPI0_MOSI" input
-			(at 233.68 63.5 180)
-			(effects
-				(font
-					(size 1.27 1.27)
-				)
-				(justify left)
-			)
-		)
-		(pin "SPI0_SCK" input
-			(at 233.68 60.96 180)
-			(effects
-				(font

Commit message: Final schematic changes
Other:
- sheet Servos & Pyros renamed Pyros
- sheet Compute ports: added CS_ICM, PYRO1_ARM, PYRO1_FIRE, PYRO1_PRESENT, PYRO2_ARM, PYRO2_FIRE, PYRO2_PRESENT; removed none
- sheet Pyros ports: added PYRO1_ARM, PYRO1_FIRE, PYRO1_PRESENT, PYRO2_ARM, PYRO2_FIRE, PYRO2_PRESENT; removed I2C0_SCL, I2C0_SDA
- sheet Sensors ports: added CS_ICM, SPI0_MISO, SPI0_MOSI, SPI0_SCK; removed none

Commit message: Moved power monitor to seperate I2C bus for easier routing
Parts:
- added R36, R37: 1K, Resistor_SMD:R_0603_1608Metric, symbol Device:R
Connections:
- net +3V3: now also R36.2, R37.1
- new net Compute/I2C1_SCL: R36.1
- new net Compute/I2C1_SDA: R37.2
Other:
- sheet Compute ports: added I2C1_SCL, I2C1_SDA; removed none
- sheet Power & USB ports: added I2C1_SCL, I2C1_SDA; removed I2C0_SCL, I2C0_SDA

Commit message: new routing
Other:
- sheet Connectivity ports: added I2C1_SCL, I2C1_SDA; removed I2C0_SCL, I2C0_SDA
- moved on the sheet: R1, R2, R36, R37

Commit message: final production files
Parts:
- J1, J2: DK Part (none) -> https://www.digikey.com/en/products/detail/amphenol-anytek/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
Changed lines of the file:
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@@
+			)
+		)
+		(property "DK Part" "https://www.digikey.com/en/products/detail/amphenol-anytek/VI0801550000G/2261365"
+			(at 91.44 147.32 0)
+			(effects
+				(font
+					(size 1.27 1.27)
+				)
+				(hide yes)
 			)
 		)
@@
 			(at 121.92 149.86 0)
 			(effects
+				(font
+					(size 1.27 1.27)
+				)
+				(hide yes)
+			)
+		)
+		(property "DK Part" "https://www.digikey.com/en/products/detail/amphenol-anytek/VI0801550000G/2261365"
+			(at 121.92 149.86 0)
+			(effects
